Commit message: updated the gazebo with table model

File: iiwa_description/urdf/iiwa14.urdf.xacro (robot description, xacro)
@@ -18,4 +18,5 @@
     <child
       link="frame" />
+    <axis xyz="0 0 1"/>
   </joint>
   <link
@@ -60,5 +61,5 @@
   </link>
   <!--iiwa-->
-  <xacro:iiwa14 hardware_interface="$(arg hardware_interface)" robot_name="$(arg robot_name)" parent="frame">
+  <xacro:iiwa14 hardware_interface="$(arg hardware_interface)" robot_name="$(arg robot_name)" parent="world">
     <origin xyz="$(arg origin_xyz)" rpy="$(arg origin_rpy)" />
   </xacro:iiwa14>

File: iiwa_description/urdf/iiwa14.xacro (robot description, xacro)
@@ -19,4 +19,5 @@
       <parent link="${parent}"/>
       <child link="${robot_name}_link_0"/>
+      <axis xyz="0 0 1"/>
     </joint>
     <link name="${robot_name}_link_0">
