Commit message: Stable Robot before making .world

File: iiwa_description/urdf/gripper_eoat.xacro (robot description, xacro)
@@ -4,6 +4,6 @@
   <xacro:property name="PIhalf" value="1.570796" />
   <xacro:property name="PI" value="3.141592" />
-  <xacro:property name="joint_friction" value="0.1" />
-  <xacro:property name="joint_damping" value="0.1" />
+  <xacro:property name="joint_friction" value="0.0001" />
+  <xacro:property name="joint_damping" value="0.0001" />
   <link
     name="gripper_base_link">
@@ -48,5 +48,5 @@
   <joint
     name="gripper_base_joint"
-    type="continuous">
+    type="revolute">
     <origin
       xyz="0 0 0.045"
@@ -59,4 +59,6 @@
       xyz="0 0 1" />
     <limit
+      lower="0"
+      upper="0"
       effort="2000"
       velocity="13" />
