Commit message: Python script for controlling robot added, and PID gains are correct. Need to correct sine wave input to surface

File: iiwa_description/urdf/iiwa.transmission.xacro (robot description, xacro)
@@ -149,5 +149,5 @@
     </transmission>
 <transmission name="pulsating_surface_tran_1">
-      <robotNamespace>/pulsating_surface</robotNamespace>
+      <robotNamespace>/${robot_name}</robotNamespace>
       <type>transmission_interface/SimpleTransmission</type>
       <joint name="prismatic_joint">

File: iiwa_description/urdf/pulsating_surface.urdf.xacro (robot description, xacro)
@@ -37,5 +37,5 @@
       <parent link="post"/>
       <child link="surface"/>
-      <origin xyz="0 0 0.5" rpy="0 0 1.5707"/>
+      <origin xyz="0 0 0.3" rpy="0 0 1.5707"/>
       <axis xyz="0 0 1"/>
       <limit lower="-0.1" upper="0.3"
