Commit message: Stable robot with effort interfce position controllers. Not all PID gains are tuned

File: iiwa_description/urdf/iiwa14.xacro (robot description, xacro)
@@ -17,5 +17,5 @@
   <xacro:property name="joint_friction" value="0.4"/>
   <xacro:property name="max_effort" value="5000"/>
-  <xacro:property name="max_velocity" value="10"/>
+  <xacro:property name="max_velocity" value="100"/>
   <xacro:macro name="iiwa14" params="parent hardware_interface robot_name *origin">
     <!--joint between {parent} and link_0-->
@@ -61,8 +61,4 @@
       <limit lower="${-170 * PI / 180}" upper="${170 * PI / 180}"
              effort="${max_effort}" velocity="${max_velocity}" />
-      <safety_controller soft_lower_limit="${-168 * PI / 180}"
-                         soft_upper_limit="${168 * PI / 180}"
-                         k_position="${safety_controller_k_pos}"
-                         k_velocity="${safety_controller_k_vel}"/>
       <dynamics damping="${joint_damping}" friction="${joint_friction}"/>
     </joint>
@@ -96,8 +92,4 @@
       <limit lower="${-120 * PI / 180}" upper="${120 * PI / 180}"
              effort="${max_effort}" velocity="${max_velocity}" />
-      <safety_controller soft_lower_limit="${-118 * PI / 180}"
-                         soft_upper_limit="${118 * PI / 180}"
-                         k_position="${safety_controller_k_pos}"
-                         k_velocity="${safety_controller_k_vel}"/>
       <dynamics damping="${joint_damping}" friction="${joint_friction}"/>
     </joint>
@@ -131,8 +123,4 @@
       <limit lower="${-170 * PI / 180}" upper="${170 * PI / 180}"
              effort="${max_effort}" velocity="${max_velocity}" />
-      <safety_controller soft_lower_limit="${-168 * PI / 180}"
-                         soft_upper_limit="${168 * PI / 180}"
-                         k_position="${safety_controller_k_pos}"
-                         k_velocity="${safety_controller_k_vel}"/>
       <dynamics damping="${joint_damping}" friction="${joint_friction}"/>
     </joint>
@@ -166,8 +154,4 @@
       <limit lower="${-120 * PI / 180}" upper="${120 * PI / 180}"
              effort="${max_effort}" velocity="${max_velocity}" />
-      <safety_controller soft_lower_limit="${-118 * PI / 180}"
-                         soft_upper_limit="${118 * PI / 180}"
-                         k_position="${safety_controller_k_pos}"
-                         k_velocity="${safety_controller_k_vel}"/>
       <dynamics damping="${joint_damping}" friction="${joint_friction}"/>
     </joint>
@@ -201,8 +185,4 @@
       <limit lower="${-170 * PI / 180}" upper="${170 * PI / 180}"
              effort="${max_effort}" velocity="${max_velocity}" />
-      <safety_controller soft_lower_limit="${-168 * PI / 180}"
-                         soft_upper_limit="${168 * PI / 180}"
-                         k_position="${safety_controller_k_pos}"
-                         k_velocity="${safety_controller_k_vel}"/>
       <dynamics damping="${joint_damping}" friction="${joint_friction}"/>
     </joint>
@@ -236,8 +216,4 @@
       <limit lower="${-120 * PI / 180}" upper="${120 * PI / 180}"
              effort="${max_effort}" velocity="${max_velocity}" />
-      <safety_controller soft_lower_limit="${-118 * PI / 180}"
-                         soft_upper_limit="${118 * PI / 180}"
-                         k_position="${safety_controller_k_pos}"
-                         k_velocity="${safety_controller_k_vel}"/>
       <dynamics damping="${joint_damping}" friction="${joint_friction}"/>
     </joint>
@@ -271,8 +247,4 @@
       <limit lower="${-175 * PI / 180}" upper="${175 * PI / 180}"
              effort="${max_effort}" velocity="${max_velocity}" />
-      <safety_controller soft_lower_limit="${-173 * PI / 180}"
-                         soft_upper_limit="${173 * PI / 180}"
-                         k_position="${safety_controller_k_pos}"
-                         k_velocity="${safety_controller_k_vel}"/>
       <dynamics damping="${joint_damping}" friction="${joint_friction}"/>
     </joint>
