Commit message: First github commit

File: iiwa_description/urdf/iiwa.gazebo.xacro (robot description, xacro)
@@ -16,5 +16,5 @@
     <!-- Link1 -->
     <gazebo reference="${robot_name}_link_1">
-      <material>Gazebo/Orange</material>
+      <material>Gazebo/White</material>
       <mu1>0.2</mu1>
       <mu2>0.2</mu2>
@@ -22,5 +22,5 @@
     <!-- Link2 -->
     <gazebo reference="${robot_name}_link_2">
-      <material>Gazebo/Orange</material>
+      <material>Gazebo/White</material>
       <mu1>0.2</mu1>
       <mu2>0.2</mu2>
@@ -28,5 +28,5 @@
     <!-- Link3 -->
     <gazebo reference="${robot_name}_link_3">
-      <material>Gazebo/Orange</material>
+      <material>Gazebo/White</material>
       <mu1>0.2</mu1>
       <mu2>0.2</mu2>
@@ -34,5 +34,5 @@
     <!-- Link4 -->
     <gazebo reference="${robot_name}_link_4">
-      <material>Gazebo/Orange</material>
+      <material>Gazebo/White</material>
       <mu1>0.2</mu1>
       <mu2>0.2</mu2>
@@ -40,5 +40,5 @@
     <!-- Link5 -->
     <gazebo reference="${robot_name}_link_5">
-      <material>Gazebo/Orange</material>
+      <material>Gazebo/White</material>
       <mu1>0.2</mu1>
       <mu2>0.2</mu2>
@@ -46,5 +46,5 @@
     <!-- Link6 -->
     <gazebo reference="${robot_name}_link_6">
-      <material>Gazebo/Orange</material>
+      <material>Gazebo/White</material>
       <mu1>0.2</mu1>
       <mu2>0.2</mu2>

File: iiwa_description/urdf/iiwa14.urdf.xacro (robot description, xacro)
@@ -10,7 +10,55 @@
   <xacro:arg name="origin_rpy" default="0 0 0"/>
   <!-- Fix to world just for testing -->
-  <link name="world"/>
+  <link name="world" />
+  <joint
+    name="fixed"
+    type="fixed">
+    <parent
+      link="world" />
+    <child
+      link="frame" />
+  </joint>
+  <link
+    name="frame">
+    <inertial>
+      <origin
+        xyz="1.5 0.25 1.25"
+        rpy="0 0 0" />
+      <mass
+        value="2697" />
+      <inertia
+        ixx="0"
+        ixy="0"
+        ixz="0"
+        iyy="0"
+        iyz="0"
+        izz="0" />
+    </inertial>
+    <visual>
+      <origin
+        xyz="0 0 0"
+        rpy="0 0 0" />
+      <geometry>
+        <mesh
+          filename="package://iiwa_description/meshes/iiwa14/visual/base_link.STL" />
+      </geometry>
+      <material
+        name="">
+        <color
+          rgba="0.64706 0.61961 0.58824 1" />
+      </material>
+    </visual>
+    <collision>
+      <origin
+        xyz="0 0 0"
+        rpy="0 0 0" />
+      <geometry>
+        <mesh
+          filename="package://iiwa_description/meshes/iiwa14/collision/base_link.STL" />
+      </geometry>
+    </collision>
+  </link>
   <!--iiwa-->
-  <xacro:iiwa14 hardware_interface="$(arg hardware_interface)" robot_name="$(arg robot_name)" parent="world">
+  <xacro:iiwa14 hardware_interface="$(arg hardware_interface)" robot_name="$(arg robot_name)" parent="frame">
     <origin xyz="$(arg origin_xyz)" rpy="$(arg origin_rpy)" />
   </xacro:iiwa14>

File: iiwa_description/urdf/iiwa14.xacro (robot description, xacro)
@@ -295,8 +295,48 @@
       <parent link="${robot_name}_link_7"/>
       <child link="${robot_name}_link_ee"/>
-      <origin xyz="0 0 0.045" rpy="0 0 0"/>
-    </joint>
-    <link name="${robot_name}_link_ee">
-    </link>
+      <origin xyz="0 0 0.0525" rpy="1.57 0 0"/>
+    </joint>
+    <!--link name="${robot_name}_link_ee">
+    </link-->
+  <link
+    name="${robot_name}_link_ee">
+    <inertial>
+      <origin
+        xyz="9.5698E-05 0.0082673 2.27179999999949E-06"
+        rpy="0 0 0" />
+      <mass
+        value="0.042407" />
+      <inertia
+        ixx="2.09361562697698E-05"
+        ixy="-1.03008820969214E-10"
+        ixz="7.85583672233988E-16"
+        iyy="1.20677052581546E-05"
+        iyz="1.27817724850131E-09"
+        izz="2.2947402405232E-05" />
+    </inertial>
+    <visual>
+      <origin
+        xyz="0 0 0"
+        rpy="1.5707963267949 0 0" />
+      <geometry>
+        <mesh
+          filename="package://iiwa_description/meshes/iiwa14/collision/flange.STL" />
+      </geometry>
+      <material
+        name="">
+        <color
+          rgba="0.79216 0.81961 0.93333 1" />
+      </material>
+    </visual>
+    <collision>
+      <origin
+        xyz="0 0 0"
+        rpy="1.5707963267949 0 0" />
+      <geometry>
+        <mesh
+          filename="package://iiwa_description/meshes/iiwa14/collision/flange.STL" />
+      </geometry>
+    </collision>
+  </link>
     <!--Extensions -->
     <xacro:iiwa_gazebo robot_name="${robot_name}" />

Commit message: Stable Robot

File: iiwa_description/urdf/iiwa.gazebo.xacro (robot description, xacro)
@@ -8,4 +8,30 @@
       </plugin>
     </gazebo>
+    <gazebo>
+      <plugin name='gazebo_ros_ft_sensor' filename='libgazebo_ros_ft_sensor.so'>
+          <robotNamespace>/${robot_name}</robotNamespace>
+          <topicName>ft_sensor_data</topicName>
+          <jointName>${robot_name}_joint_7</jointName>
+          <updateRate>10</updateRate>
+      </plugin>
+  </gazebo>
+  <gazebo>
+      <plugin name='gazebo_ros_ft_sensor_claw' filename='libgazebo_ros_ft_sensor.so'>
+          <robotNamespace>/${robot_name}</robotNamespace>
+          <topicName>ft_sensor_data_claw</topicName>
+          <jointName>claw_1_joint</jointName>
+          <updateRate>10</updateRate>
+      </plugin>
+  </gazebo>
+    <gazebo>
+      <static>0</static>
+    </gazebo>
+    <!--Frame-->
+    <gazebo reference="frame">
+      <material>Gazebo/White</material>
+      <mu1>0.2</mu1>
+      <mu2>0.2</mu2>
+      <selfCollide>1</selfCollide>
+    </gazebo>
     <!-- Link0 -->
     <gazebo reference="${robot_name}_link_0">
@@ -13,4 +39,5 @@
       <mu1>0.2</mu1>
       <mu2>0.2</mu2>
+      <selfCollide>1</selfCollide>
     </gazebo>
     <!-- Link1 -->
@@ -19,4 +46,5 @@
       <mu1>0.2</mu1>
       <mu2>0.2</mu2>
+      <selfCollide>1</selfCollide>
     </gazebo>
     <!-- Link2 -->
@@ -25,4 +53,5 @@
       <mu1>0.2</mu1>
       <mu2>0.2</mu2>
+      <selfCollide>1</selfCollide>
     </gazebo>
     <!-- Link3 -->
@@ -31,4 +60,5 @@
       <mu1>0.2</mu1>
       <mu2>0.2</mu2>
+      <selfCollide>1</selfCollide>
     </gazebo>
     <!-- Link4 -->
@@ -37,4 +67,5 @@
       <mu1>0.2</mu1>
       <mu2>0.2</mu2>
+      <selfCollide>1</selfCollide>
     </gazebo>
     <!-- Link5 -->
@@ -43,4 +74,5 @@
       <mu1>0.2</mu1>
       <mu2>0.2</mu2>
+      <selfCollide>1</selfCollide>
     </gazebo>
     <!-- Link6 -->
@@ -49,4 +81,5 @@
       <mu1>0.2</mu1>
       <mu2>0.2</mu2>
+      <selfCollide>1</selfCollide>
     </gazebo>
     <!-- Link7 -->
@@ -55,4 +88,73 @@
       <mu1>0.2</mu1>
       <mu2>0.2</mu2>
+      <selfCollide>1</selfCollide>
+    </gazebo>
+    <gazebo reference="${robot_name}_joint_7">
+      <provideFeedback>true</provideFeedback>
+    </gazebo>
+    <!--EOAT-->
+<!--
+    <gazebo reference="rotating_base_link">
+      <material>Gazebo/Grey</material>
+      <mu1>0.2</mu1>
+      <mu2>0.2</mu2>
+      <selfCollide>1</selfCollide>
+    </gazebo>
+    <gazebo reference="rotating_arm_link">
+      <material>Gazebo/Orange</material>
+      <mu1>0.2</mu1>
+      <mu2>0.2</mu2>
+      <selfCollide>1</selfCollide>
+    </gazebo>
+-->
+    <gazebo reference="gripper_base_link">
+      <material>Gazebo/White</material>
+      <mu1>0.2</mu1>
+      <mu2>0.2</mu2>
+      <selfCollide>1</selfCollide>
+    </gazebo>
+    <gazebo reference="claw_1_link">
+      <material>Gazebo/Grey</material>
+      <mu1>0.2</mu1>
+      <mu2>0.2</mu2>
+      <gravity>1</gravity>
+      <selfCollide>1</selfCollide>
+    </gazebo>
+    <gazebo reference="claw_1_joint">
+      <provideFeedback>true</provideFeedback>
+    </gazebo>
+    <gazebo reference="claw_2_link">
+      <material>Gazebo/Orange</material>
+      <mu1>0.2</mu1>
+      <mu2>0.2</mu2>
+      <gravity>1</gravity>
+      <selfCollide>1</selfCollide>
+    </gazebo>
+    <gazebo reference="claw_3_link">
+      <material>Gazebo/Blue</material>
+      <mu1>0.2</mu1>
+      <mu2>0.2</mu2>
+      <gravity>1</gravity>
+      <selfCollide>1</selfCollide>
+    </gazebo>
+    <gazebo reference="claw_4_link">
+      <material>Gazebo/Red</material>
+      <mu1>0.2</mu1>
+      <mu2>0.2</mu2>
+      <gravity>1</gravity>
+      <selfCollide>1</selfCollide>
+    </gazebo>
+    <gazebo reference="post">
+      <material>Gazebo/White</material>
+      <mu1>0.2</mu1>
+      <mu2>0.2</mu2>
+    </gazebo>
+    <gazebo reference="surface">
+      <material>Gazebo/Orange</material>
+      <mu1>0.2</mu1>
+      <mu2>0.2</mu2>
+      <kd>2500</kd>
+      <kp>10000</kp>
+      <selfCollide>1</selfCollide>
     </gazebo>
   </xacro:macro>

File: iiwa_description/urdf/iiwa.transmission.xacro (robot description, xacro)
@@ -79,4 +79,84 @@
       </actuator>
     </transmission>
+    <!--Added for EOAT-->
+<!--
+  <transmission name="eoat_tran1">
+    <robotNamespace>/${robot_name}</robotNamespace>
+    <type>transmission_interface/SimpleTransmission</type>
+    <joint name="rotating_base_joint">
+      <hardwareInterface>${hardware_interface}</hardwareInterface>
+    </joint>
+    <actuator name="motor1">
+      <hardwareInterface>${hardware_interface}</hardwareInterface>
+      <mechanicalReduction>1</mechanicalReduction>
+    </actuator>
+  </transmission>
+  <transmission name="eoat_tran2">
+    <robotNamespace>/${robot_name}</robotNamespace>
+    <type>transmission_interface/SimpleTransmission</type>
+    <joint name="rotating_arm_joint">
+      <hardwareInterface>${hardware_interface}</hardwareInterface>
+    </joint>
+    <actuator name="motor2">
+      <hardwareInterface>${hardware_interface}</hardwareInterface>
+      <mechanicalReduction>1</mechanicalReduction>
+    </actuator>
+  </transmission>
+-->
+<transmission name="claw_1_tran">
+      <robotNamespace>/${robot_name}</robotNamespace>
+      <type>transmission_interface/SimpleTransmission</type>
+      <joint name="claw_1_joint">
+  <hardwareInterface>${hardware_interface}</hardwareInterface>
+      </joint>
+      <actuator name="claw_1_motor">
+  <hardwareInterface>${hardware_interface}</hardwareInterface>
+  <mechanicalReduction>1</mechanicalReduction>
+      </actuator>
+    </transmission>
+    <transmission name="claw_2_tran">
+      <robotNamespace>/${robot_name}</robotNamespace>
+      <type>transmission_interface/SimpleTransmission</type>
+      <joint name="claw_2_joint">
+  <hardwareInterface>${hardware_interface}</hardwareInterface>
+      </joint>
+      <actuator name="claw_2_motor">
+  <hardwareInterface>${hardware_interface}</hardwareInterface>
+  <mechanicalReduction>1</mechanicalReduction>
+      </actuator>
+    </transmission>
+    <transmission name="claw_3_tran">
+      <robotNamespace>/${robot_name}</robotNamespace>
+      <type>transmission_interface/SimpleTransmission</type>
+      <joint name="claw_3_joint">
+  <hardwareInterface>${hardware_interface}</hardwareInterface>
+      </joint>
+      <actuator name="claw_3_motor">
+  <hardwareInterface>${hardware_interface}</hardwareInterface>
+  <mechanicalReduction>1</mechanicalReduction>
+      </actuator>
+    </transmission>
+<transmission name="claw_4_tran">
+      <robotNamespace>/${robot_name}</robotNamespace>
+      <type>transmission_interface/SimpleTransmission</type>
+      <joint name="claw_4_joint">
+  <hardwareInterface>${hardware_interface}</hardwareInterface>
+      </joint>
+      <actuator name="claw_4_motor">
+  <hardwareInterface>${hardware_interface}</hardwareInterface>
+  <mechanicalReduction>1</mechanicalReduction>
+      </actuator>
+    </transmission>
+<transmission name="pulsating_surface_tran_1">
+      <robotNamespace>/pulsating_surface</robotNamespace>
+      <type>transmission_interface/SimpleTransmission</type>
+      <joint name="prismatic_joint">
+  <hardwareInterface>${hardware_interface}</hardwareInterface>
+      </joint>
+      <actuator name="pulsating_surface_motor_1">
+  <hardwareInterface>${hardware_interface}</hardwareInterface>
+  <mechanicalReduction>1</mechanicalReduction>
+      </actuator>
+    </transmission>
   </xacro:macro>
 </robot>

File: iiwa_description/urdf/iiwa14.urdf.xacro (robot description, xacro)
@@ -42,5 +42,5 @@
       <geometry>
         <mesh
-          filename="package://iiwa_description/meshes/iiwa14/visual/base_link.STL" />
+          filename="package://iiwa_description/meshes/iiwa14/visual/base_link.STL"/>
       </geometry>
       <material

File: iiwa_description/urdf/iiwa14.xacro (robot description, xacro)
@@ -7,8 +7,13 @@
   <!-- Include Utilities -->
   <xacro:include filename="$(find iiwa_description)/urdf/utilities.xacro" />
+  <!-- Include EOAT -->
+  <xacro:include filename="$(find iiwa_description)/urdf/juans_eoat.xacro" />
+  <xacro:include filename="$(find iiwa_description)/urdf/gripper_eoat.xacro" />
+  <xacro:include filename="$(find iiwa_description)/urdf/pulsating_surface.urdf.xacro" />
   <!-- some constants -->
   <xacro:property name="safety_controller_k_pos" value="100" />
   <xacro:property name="safety_controller_k_vel" value="2" />
-  <xacro:property name="joint_damping" value="0.5" />
+  <xacro:property name="joint_damping" value="0.1" />
+  <xacro:property name="joint_friction" value="0.1"/>
   <xacro:property name="max_effort" value="300"/>
   <xacro:property name="max_velocity" value="10"/>
@@ -60,5 +65,5 @@
                          k_position="${safety_controller_k_pos}"
                          k_velocity="${safety_controller_k_vel}"/>
-      <dynamics damping="${joint_damping}"/>
+      <dynamics damping="${joint_damping}" friction="${joint_friction}"/>
     </joint>
     <link name="${robot_name}_link_1">
@@ -95,5 +100,5 @@
                          k_position="${safety_controller_k_pos}"
                          k_velocity="${safety_controller_k_vel}"/>
-      <dynamics damping="${joint_damping}"/>
+      <dynamics damping="${joint_damping}" friction="${joint_friction}"/>
     </joint>
     <link name="${robot_name}_link_2">
@@ -130,5 +135,5 @@
                          k_position="${safety_controller_k_pos}"
                          k_velocity="${safety_controller_k_vel}"/>
-      <dynamics damping="${joint_damping}"/>
+      <dynamics damping="${joint_damping}" friction="${joint_friction}"/>
     </joint>
     <link name="${robot_name}_link_3">
@@ -165,5 +170,5 @@
                          k_position="${safety_controller_k_pos}"
                          k_velocity="${safety_controller_k_vel}"/>
-      <dynamics damping="${joint_damping}"/>
+      <dynamics damping="${joint_damping}" friction="${joint_friction}"/>
     </joint>
     <link name="${robot_name}_link_4">
@@ -200,5 +205,5 @@
                          k_position="${safety_controller_k_pos}"
                          k_velocity="${safety_controller_k_vel}"/>
-      <dynamics damping="${joint_damping}"/>
+      <dynamics damping="${joint_damping}" friction="${joint_friction}"/>
     </joint>
     <link name="${robot_name}_link_5">
@@ -235,5 +240,5 @@
                          k_position="${safety_controller_k_pos}"
                          k_velocity="${safety_controller_k_vel}"/>
-      <dynamics damping="${joint_damping}"/>
+      <dynamics damping="${joint_damping}" friction="${joint_friction}"/>
     </joint>
     <link name="${robot_name}_link_6">
@@ -270,5 +275,5 @@
                          k_position="${safety_controller_k_pos}"
                          k_velocity="${safety_controller_k_vel}"/>
-      <dynamics damping="${joint_damping}"/>
+      <dynamics damping="${joint_damping}" friction="${joint_friction}"/>
     </joint>
     <link name="${robot_name}_link_7">
@@ -293,4 +298,5 @@
       </collision>
     </link>
+    <!-- Commented force sensor EOAT
     <joint name="${robot_name}_joint_ee" type="fixed">
       <parent link="${robot_name}_link_7"/>
@@ -298,6 +304,6 @@
       <origin xyz="0 0 0.0525" rpy="1.57 0 0"/>
     </joint>
-    <!--link name="${robot_name}_link_ee">
-    </link-->
+    <link name="${robot_name}_link_ee">
+    </link>
   <link
     name="${robot_name}_link_ee">
@@ -340,6 +346,10 @@
     </collision>
   </link>
+-->
     <!--Extensions -->
-    <xacro:iiwa_gazebo robot_name="${robot_name}" />
+    <!--<xacro:juans_eoat robot_name="${robot_name}"/>--> <!--Comented out EOAT-->
+    <xacro:gripper_eoat robot_name="${robot_name}"/>
+    <xacro:pulsating_surface />
+    <xacro:iiwa_gazebo robot_name="${robot_name}"/>
     <xacro:iiwa_transmission hardware_interface="${hardware_interface}"/>
   </xacro:macro>

Commit message: Trying to stablize model

File: iiwa_description/urdf/iiwa.gazebo.xacro (robot description, xacro)
@@ -27,5 +27,5 @@
 -->
     <gazebo>
-      <static>1</static>
+      <static>0</static>
     </gazebo>
     <!--Frame-->
@@ -34,5 +34,5 @@
       <mu1>0.2</mu1>
       <mu2>0.2</mu2>
-      <selfCollide>1</selfCollide>
+      <selfCollide>0</selfCollide>
     </gazebo>
     <!-- Link0 -->
@@ -41,5 +41,5 @@
       <mu1>0.2</mu1>
       <mu2>0.2</mu2>
-      <selfCollide>1</selfCollide>
+      <selfCollide>0</selfCollide>
     </gazebo>
     <!-- Link1 -->
@@ -48,5 +48,5 @@
       <mu1>0.2</mu1>
       <mu2>0.2</mu2>
-      <selfCollide>1</selfCollide>
+      <selfCollide>0</selfCollide>
     </gazebo>
     <!-- Link2 -->
@@ -55,5 +55,5 @@
       <mu1>0.2</mu1>
       <mu2>0.2</mu2>
-      <selfCollide>1</selfCollide>
+      <selfCollide>0</selfCollide>
     </gazebo>
     <!-- Link3 -->
@@ -62,5 +62,5 @@
       <mu1>0.2</mu1>
       <mu2>0.2</mu2>
-      <selfCollide>1</selfCollide>
+      <selfCollide>0</selfCollide>
     </gazebo>
     <!-- Link4 -->
@@ -69,5 +69,5 @@
       <mu1>0.2</mu1>
       <mu2>0.2</mu2>
-      <selfCollide>1</selfCollide>
+      <selfCollide>0</selfCollide>
     </gazebo>
     <!-- Link5 -->
@@ -76,5 +76,5 @@
       <mu1>0.2</mu1>
       <mu2>0.2</mu2>
-      <selfCollide>1</selfCollide>
+      <selfCollide>0</selfCollide>
     </gazebo>
     <!-- Link6 -->
@@ -83,5 +83,5 @@
       <mu1>0.2</mu1>
       <mu2>0.2</mu2>
-      <selfCollide>1</selfCollide>
+      <selfCollide>0</selfCollide>
     </gazebo>
     <!-- Link7 -->
@@ -90,5 +90,35 @@
       <mu1>0.2</mu1>
       <mu2>0.2</mu2>
-      <selfCollide>1</selfCollide>
+      <selfCollide>0</selfCollide>
+    </gazebo>
+    <gazebo reference="base_link">
+      <material>Gazebo/White</material>
+      <mu1>0.2</mu1>
+      <mu2>0.2</mu2>
+      <selfCollide>0</selfCollide>
+    </gazebo>
+    <gazebo reference="Link1">
+      <material>Gazebo/White</material>
+      <mu1>0.2</mu1>
+      <mu2>0.2</mu2>
+      <selfCollide>0</selfCollide>
+    </gazebo>
+    <gazebo reference="Link2">
+      <material>Gazebo/White</material>
+      <mu1>0.2</mu1>
+      <mu2>0.2</mu2>
+      <selfCollide>0</selfCollide>
+    </gazebo>
+    <gazebo reference="Link3">
+      <material>Gazebo/White</material>
+      <mu1>0.2</mu1>
+      <mu2>0.2</mu2>
+      <selfCollide>0</selfCollide>
+    </gazebo>
+    <gazebo reference="Link4">
+      <material>Gazebo/White</material>
+      <mu1>0.2</mu1>
+      <mu2>0.2</mu2>
+      <selfCollide>0</selfCollide>
     </gazebo>
     <gazebo reference="${robot_name}_joint_7">
