Commit message: changed the model to melodic

File: iiwa_description/urdf/iiwa.gazebo.xacro (robot description, xacro)
@@ -93,19 +93,4 @@
       <provideFeedback>true</provideFeedback>
     </gazebo>
-    <!--EOAT-->
-<!--
-    <gazebo reference="rotating_base_link">
-      <material>Gazebo/Grey</material>
-      <mu1>0.2</mu1>
-      <mu2>0.2</mu2>
-      <selfCollide>1</selfCollide>
-    </gazebo>
-    <gazebo reference="rotating_arm_link">
-      <material>Gazebo/Orange</material>
-      <mu1>0.2</mu1>
-      <mu2>0.2</mu2>
-      <selfCollide>1</selfCollide>
-    </gazebo>
--->
     <gazebo reference="gripper_base_link">
       <material>Gazebo/White</material>

File: iiwa_description/urdf/iiwa.transmission.xacro (robot description, xacro)
@@ -6,8 +6,7 @@
       <type>transmission_interface/SimpleTransmission</type>
       <joint name="${robot_name}_joint_1">
-	<hardwareInterface>${hardware_interface}</hardwareInterface>
+	<hardwareInterface>hardware_interface/${hardware_interface}</hardwareInterface>
       </joint>
       <actuator name="${robot_name}_motor_1">
-	<hardwareInterface>${hardware_interface}</hardwareInterface>
 	<mechanicalReduction>1</mechanicalReduction>
       </actuator>
@@ -17,8 +16,7 @@
       <type>transmission_interface/SimpleTransmission</type>
       <joint name="${robot_name}_joint_2">
-	<hardwareInterface>${hardware_interface}</hardwareInterface>
+	<hardwareInterface>hardware_interface/${hardware_interface}</hardwareInterface>
       </joint>
       <actuator name="${robot_name}_motor_2">
-	<hardwareInterface>${hardware_interface}</hardwareInterface>
 	<mechanicalReduction>1</mechanicalReduction>
       </actuator>
@@ -28,8 +26,7 @@
       <type>transmission_interface/SimpleTransmission</type>
       <joint name="${robot_name}_joint_3">
-	<hardwareInterface>${hardware_interface}</hardwareInterface>
+	<hardwareInterface>hardware_interface/${hardware_interface}</hardwareInterface>
       </joint>
       <actuator name="${robot_name}_motor_3">
-	<hardwareInterface>${hardware_interface}</hardwareInterface>
 	<mechanicalReduction>1</mechanicalReduction>
       </actuator>
@@ -39,8 +36,7 @@
       <type>transmission_interface/SimpleTransmission</type>
       <joint name="${robot_name}_joint_4">
-	<hardwareInterface>${hardware_interface}</hardwareInterface>
+	<hardwareInterface>hardware_interface/${hardware_interface}</hardwareInterface>
       </joint>
       <actuator name="${robot_name}_motor_4">
-	<hardwareInterface>${hardware_interface}</hardwareInterface>
 	<mechanicalReduction>1</mechanicalReduction>
       </actuator>
@@ -50,8 +46,7 @@
       <type>transmission_interface/SimpleTransmission</type>
       <joint name="${robot_name}_joint_5">
-	<hardwareInterface>${hardware_interface}</hardwareInterface>
+	<hardwareInterface>hardware_interface/${hardware_interface}</hardwareInterface>
       </joint>
       <actuator name="${robot_name}_motor_5">
-	<hardwareInterface>${hardware_interface}</hardwareInterface>
 	<mechanicalReduction>1</mechanicalReduction>
       </actuator>
@@ -61,8 +56,7 @@
       <type>transmission_interface/SimpleTransmission</type>
       <joint name="${robot_name}_joint_6">
-	<hardwareInterface>${hardware_interface}</hardwareInterface>
+	<hardwareInterface>hardware_interface/${hardware_interface}</hardwareInterface>
       </joint>
       <actuator name="${robot_name}_motor_6">
-	<hardwareInterface>${hardware_interface}</hardwareInterface>
 	<mechanicalReduction>1</mechanicalReduction>
       </actuator>
@@ -72,8 +66,7 @@
       <type>transmission_interface/SimpleTransmission</type>
       <joint name="${robot_name}_joint_7">
-	<hardwareInterface>${hardware_interface}</hardwareInterface>
+	<hardwareInterface>hardware_interface/${hardware_interface}</hardwareInterface>
       </joint>
       <actuator name="${robot_name}_motor_7">
-	<hardwareInterface>${hardware_interface}</hardwareInterface>
 	<mechanicalReduction>1</mechanicalReduction>
       </actuator>
@@ -108,8 +101,7 @@
       <type>transmission_interface/SimpleTransmission</type>
       <joint name="claw_1_joint">
-  <hardwareInterface>${hardware_interface}</hardwareInterface>
+  <hardwareInterface>hardware_interface/${hardware_interface}</hardwareInterface>
       </joint>
       <actuator name="claw_1_motor">
-  <hardwareInterface>${hardware_interface}</hardwareInterface>
   <mechanicalReduction>1</mechanicalReduction>
       </actuator>
@@ -119,8 +111,7 @@
       <type>transmission_interface/SimpleTransmission</type>
       <joint name="claw_2_joint">
-  <hardwareInterface>${hardware_interface}</hardwareInterface>
+  <hardwareInterface>hardware_interface/${hardware_interface}</hardwareInterface>
       </joint>
       <actuator name="claw_2_motor">
-  <hardwareInterface>${hardware_interface}</hardwareInterface>
   <mechanicalReduction>1</mechanicalReduction>
       </actuator>
@@ -130,8 +121,7 @@
       <type>transmission_interface/SimpleTransmission</type>
       <joint name="claw_3_joint">
-  <hardwareInterface>${hardware_interface}</hardwareInterface>
+  <hardwareInterface>hardware_interface/${hardware_interface}</hardwareInterface>
       </joint>
       <actuator name="claw_3_motor">
-  <hardwareInterface>${hardware_interface}</hardwareInterface>
   <mechanicalReduction>1</mechanicalReduction>
       </actuator>
@@ -141,8 +131,7 @@
       <type>transmission_interface/SimpleTransmission</type>
       <joint name="claw_4_joint">
-  <hardwareInterface>${hardware_interface}</hardwareInterface>
+  <hardwareInterface>hardware_interface/${hardware_interface}</hardwareInterface>
       </joint>
       <actuator name="claw_4_motor">
-  <hardwareInterface>${hardware_interface}</hardwareInterface>
   <mechanicalReduction>1</mechanicalReduction>
       </actuator>
@@ -152,8 +141,7 @@
       <type>transmission_interface/SimpleTransmission</type>
       <joint name="prismatic_joint">
-  <hardwareInterface>${hardware_interface}</hardwareInterface>
+  <hardwareInterface>hardware_interface/${hardware_interface}</hardwareInterface>
       </joint>
       <actuator name="pulsating_surface_motor_1">
-  <hardwareInterface>${hardware_interface}</hardwareInterface>
   <mechanicalReduction>1</mechanicalReduction>
       </actuator>

File: iiwa_description/urdf/iiwa14.urdf.xacro (robot description, xacro)
@@ -1,4 +1,4 @@
 <?xml version="1.0"?>
-<robot name="iiwa14" xmlns:xacro="http://www.ros.org/wiki/xacro">
+<robot name="kuka" xmlns:xacro="http://www.ros.org/wiki/xacro">
   <!-- Import Rviz colors -->
   <xacro:include filename="$(find iiwa_description)/urdf/materials.xacro" />
