Commit message: Working controllers for 1 arm

File: iiwa_description/urdf/Dual_Arm.xacro (robot description, xacro)
@@ -59,6 +59,6 @@
       xyz="0 0 1" />
     <limit
-      lower="0"
-      upper="0"
+      lower="-3.14"
+      upper="3.14"
       effort="2000"
       velocity="13" />
@@ -116,8 +116,8 @@
       link="Link1" />
     <axis
-      xyz="0 0 -1" />
-    <limit
-      lower="0"
-      upper="0"
+      xyz="0 0 1" />
+    <limit
+      lower="-0.5"
+      upper="0.5"
       effort="2000"
       velocity="13" />
@@ -174,8 +174,8 @@
       link="Link2" />
     <axis
-      xyz="-0.494322793221048 -0.869278422659933 0" />
-    <limit
-      lower="0"
-      upper="0"
+      xyz="0 0 1" />
+    <limit
+      lower="-0.5"
+      upper="0.5"
       effort="2000"
       velocity="13" />
@@ -232,8 +232,8 @@
       link="Link3" />
     <axis
-      xyz="-0.869278422659933 0 0.494322793221049" />
-    <limit
-      lower="0"
-      upper="0"
+      xyz="0 0 1" />
+    <limit
+      lower="-0.5"
+      upper="0.5"
       effort="2000"
       velocity="13" />
@@ -246,12 +246,12 @@
         rpy="0 0 0" />
       <mass
-        value="0.0456606488806743" />
-      <inertia
-        ixx="4.32770392148837E-05"
-        ixy="-6.50658263909868E-07"
-        ixz="-9.78467852722041E-09"
-        iyy="1.95693570544345E-08"
-        iyz="-6.5065826390888E-07"
-        izz="4.32770392148837E-05" />
+        value="0.117746913814738" />
+      <inertia
+        ixx="9.95073774261661E-05"
+        ixy="-2.667473422779E-07"
+        ixz="-3.12070252262036E-06"
+        iyy="0.000106288781760734"
+        iyz="-2.88857039626312E-06"
+        izz="6.98820523527226E-06" />
     </inertial>
     <visual>
@@ -290,8 +290,8 @@
       link="Link4" />
     <axis
-      xyz="0.362830675905036 -0.335721498447973 -0.869278422659934" />
-    <limit
-      lower="0"
-      upper="0"
+      xyz="0 0 1" />
+    <limit
+      lower="-0.5"
+      upper="0.5"
       effort="2000"
       velocity="13" />

File: iiwa_description/urdf/iiwa.gazebo.xacro (robot description, xacro)
@@ -8,5 +8,5 @@
       </plugin>
     </gazebo>
-<!--
+<!--Force sensors
     <gazebo>
       <plugin name='gazebo_ros_ft_sensor' filename='libgazebo_ros_ft_sensor.so'>

File: iiwa_description/urdf/iiwa.transmission.xacro (robot description, xacro)
@@ -104,50 +104,59 @@
   </transmission>
 -->
-<!--
-<transmission name="claw_1_tran">
+<transmission name="manipulator_tran_1">
       <robotNamespace>/${robot_name}</robotNamespace>
       <type>transmission_interface/SimpleTransmission</type>
-      <joint name="claw_1_joint">
+      <joint name="dual_arm_base_joint">
   <hardwareInterface>${hardware_interface}</hardwareInterface>
       </joint>
-      <actuator name="claw_1_motor">
+      <actuator name="dual_arm_base_motor">
   <hardwareInterface>${hardware_interface}</hardwareInterface>
   <mechanicalReduction>1</mechanicalReduction>
       </actuator>
     </transmission>
-    <transmission name="claw_2_tran">
+    <transmission name="J_1_tran">
       <robotNamespace>/${robot_name}</robotNamespace>
       <type>transmission_interface/SimpleTransmission</type>
-      <joint name="claw_2_joint">
+      <joint name="J_1">
   <hardwareInterface>${hardware_interface}</hardwareInterface>
       </joint>
-      <actuator name="claw_2_motor">
+      <actuator name="J_1_motor">
   <hardwareInterface>${hardware_interface}</hardwareInterface>
   <mechanicalReduction>1</mechanicalReduction>
       </actuator>
     </transmission>
-    <transmission name="claw_3_tran">
+    <transmission name="J_2_tran">
       <robotNamespace>/${robot_name}</robotNamespace>
       <type>transmission_interface/SimpleTransmission</type>
-      <joint name="claw_3_joint">
+      <joint name="J_2">
   <hardwareInterface>${hardware_interface}</hardwareInterface>
       </joint>
-      <actuator name="claw_3_motor">
+      <actuator name="J_2_motor">
   <hardwareInterface>${hardware_interface}</hardwareInterface>
   <mechanicalReduction>1</mechanicalReduction>
       </actuator>
     </transmission>
-<transmission name="claw_4_tran">
+<transmission name="J_3_tran">
       <robotNamespace>/${robot_name}</robotNamespace>
       <type>transmission_interface/SimpleTransmission</type>
-      <joint name="claw_4_joint">
+      <joint name="J_3">
   <hardwareInterface>${hardware_interface}</hardwareInterface>
       </joint>
-      <actuator name="claw_4_motor">
+      <actuator name="J_3_motor">
   <hardwareInterface>${hardware_interface}</hardwareInterface>
   <mechanicalReduction>1</mechanicalReduction>
       </actuator>
     </transmission>
-  -->
+    <transmission name="J_4_tran">
+      <robotNamespace>/${robot_name}</robotNamespace>
+      <type>transmission_interface/SimpleTransmission</type>
+      <joint name="J_4">
+  <hardwareInterface>${hardware_interface}</hardwareInterface>
+      </joint>
+      <actuator name="J_4_motor">
+  <hardwareInterface>${hardware_interface}</hardwareInterface>
+  <mechanicalReduction>1</mechanicalReduction>
+      </actuator>
+    </transmission>
 <transmission name="pulsating_surface_tran_1">
       <robotNamespace>/${robot_name}</robotNamespace>
