Commit message: Loaded controllers for all joints, added grippers

File: iiwa_description/urdf/Dual_Arm.xacro (robot description, xacro)
@@ -2,6 +2,6 @@
 <robot xmlns:xacro="http://www.ros.org/wiki/xacro">
   <xacro:macro name="dual_arm_manipulator" params="robot_name">
-  <xacro:property name="joint_friction" value="0.0001" />
-  <xacro:property name="joint_damping" value="0.0001" />
+  <xacro:property name="joint_friction" value="0.01" />
+  <xacro:property name="joint_damping" value="0.01" />
   <xacro:property name="PIhalf" value="1.570796" />
   <xacro:property name="PI" value="3.141592" />
@@ -122,4 +122,5 @@
       effort="2000"
       velocity="13" />
+    <dynamics damping="${joint_damping}" friction = "${joint_friction}"/>
   </joint>
   <link
@@ -167,6 +168,6 @@
     type="revolute">
     <origin
-      xyz="0.000622197162453347 -0.00110714528903752 -0.0543559999999998"
-      rpy="1.57079632679489 -0.517055614178857 0.511996865187095" />
+      xyz="0 0 -0.0635"
+      rpy="1.57079632679489 -0.380374098489847 0.317429885556193" />
     <parent
       link="Link1" />
@@ -180,4 +181,5 @@
       effort="2000"
       velocity="13" />
+    <dynamics damping="${joint_damping}" friction = "${joint_friction}"/>
   </joint>
   <link
@@ -226,5 +228,5 @@
     <origin
       xyz="-0.178688999999999 -0.00012700000000021 0"
-      rpy="-1.57079632679489 -1.0547118733939E-15 1.5707963267949" />
+      rpy="-1.57079632679489 -0.00547118733939 1.5707963267949" />
     <parent
       link="Link2" />
@@ -238,4 +240,5 @@
       effort="2000"
       velocity="13" />
+    <dynamics damping="${joint_damping}" friction = "${joint_friction}"/>
   </joint>
   <link
@@ -296,4 +299,241 @@
       effort="2000"
       velocity="13" />
+    <dynamics damping="${joint_damping}" friction = "${joint_friction}"/>
+  </joint>
+  <link
+    name="L2_1">
+    <inertial>
+      <origin
+        xyz="0.00302464836897415 0.00148467584367146 -0.0196712040191069"
+        rpy="0 0 0" />
+      <mass
+        value="0.323170961054133" />
+      <inertia
+        ixx="9.86315700006277E-05"
+        ixy="-1.83712585125958E-06"
+        ixz="1.50310533353745E-05"
+        iyy="0.000101226511355012"
+        iyz="6.90483440689725E-06"
+        izz="4.61898687854836E-06" />
+    </inertial>
+    <visual>
+      <origin
+        xyz="0 0 0"
+        rpy="0 0 0" />
+      <geometry>
+        <mesh
+          filename="package://iiwa_description/meshes/iiwa14/collision/Dual_Arm/Link1.STL" />
+      </geometry>
+      <material
+        name="">
+        <color
+          rgba="1 1 1 1" />
+      </material>
+    </visual>
+    <collision>
+      <origin
+        xyz="0 0 0"
+        rpy="0 0 0" />
+      <geometry>
+        <mesh
+          filename="package://iiwa_description/meshes/iiwa14/collision/Dual_Arm/Link1.STL" />
+      </geometry>
+    </collision>
+  </link>
+  <joint
+    name="J_21"
+    type="revolute">
+    <origin
+      xyz="-0.0744445637977397 -0.152871273073736 -0.110435575211296"
+      rpy="1.43251148060093 -0.775712981728982 -2.94539473140516" />
+    <parent
+      link="base_link" />
+    <child
+      link="L2_1" />
+    <axis
+      xyz="0 0 1" />
+    <limit
+      lower="-0.5"
+      upper="0.5"
+      effort="2000"
+      velocity="13" />
+    <dynamics damping="${joint_damping}" friction = "${joint_friction}"/>
+ </joint>
+  <link
+    name="L2_2">
+    <inertial>
+      <origin
+        xyz="-0.0841816926424142 -9.94783774485586E-05 0.00119770428720625"
+        rpy="0 0 0" />
+      <mass
+        value="0.161073886022953" />
+      <inertia
+        ixx="1.38598083295319E-06"
+        ixy="-3.76180464461997E-07"
+        ixz="5.01830776658136E-09"
+        iyy="0.000417336089370728"
+        iyz="3.07943156555252E-09"
+        izz="0.000417240402620394" />
+    </inertial>
+    <visual>
+      <origin
+        xyz="0 0 0"
+        rpy="0 0 0" />
+      <geometry>
+        <mesh
+          filename="package://iiwa_description/meshes/iiwa14/collision/Dual_Arm/Link2.STL" />
+      </geometry>
+      <material
+        name="">
+        <color
+          rgba="0.898039215686275 0.898039215686275 0.898039215686275 1" />
+      </material>
+    </visual>
+    <collision>
+      <origin
+        xyz="0 0 0"
+        rpy="0 0 0" />
+      <geometry>
+        <mesh
+          filename="package://iiwa_description/meshes/iiwa14/collision/Dual_Arm/Link2.STL" />
+      </geometry>
+    </collision>
+  </link>
+  <joint
+    name="J_22"
+    type="revolute">
+    <origin
+      xyz="0 0 -0.0635"
+      rpy="1.57079632679489 -0.380374098489847 0.317429885556193" />
+    <parent
+      link="L2_1" />
+    <child
+      link="L2_2" />
+    <axis
+      xyz="0 0 1" />
+    <limit
+      lower="-0.5"
+      upper="0.5"
+      effort="2000"
+      velocity="13" />
+    <dynamics damping="${joint_damping}" friction = "${joint_friction}"/>
+  </joint>
+  <link
+    name="L2_3">
+    <inertial>
+      <origin
+        xyz="0.00289722994622221 0.00112305403125196 0.0290055866352336"
+        rpy="0 0 0" />
+      <mass
+        value="0.117746913814738" />
+      <inertia
+        ixx="9.95073774261661E-05"
+        ixy="-2.667473422779E-07"
+        ixz="-3.12070252262036E-06"
+        iyy="0.000106288781760734"
+        iyz="-2.88857039626312E-06"
+        izz="6.98820523527226E-06" />
+    </inertial>
+    <visual>
+      <origin
+        xyz="0 0 0"
+        rpy="0 0 0" />
+      <geometry>
+        <mesh
+          filename="package://iiwa_description/meshes/iiwa14/collision/Dual_Arm/Link3.STL" />
+      </geometry>
+      <material
+        name="">
+        <color
+          rgba="1 1 1 1" />
+      </material>
+    </visual>
+    <collision>
+      <origin
+        xyz="0 0 0"
+        rpy="0 0 0" />
+      <geometry>
+        <mesh
+          filename="package://iiwa_description/meshes/iiwa14/collision/Dual_Arm/Link3.STL" />
+      </geometry>
+    </collision>
+  </link>
+  <joint
+    name="J_23"
+    type="revolute">
+    <origin
+      xyz="-0.178688999999999 -0.00012700000000021 0"
+      rpy="-1.57079632679489 -1.0547118733939E-15 1.5707963267949" />
+    <parent
+      link="L2_2" />
+    <child
+      link="L2_3" />
+    <axis
+      xyz="0 0 1" />
+    <limit
+      lower="-0.5"
+      upper="0.5"
+      effort="2000"
+      velocity="13" />
+    <dynamics damping="${joint_damping}" friction = "${joint_friction}"/>
+  </joint>
+  <link
+    name="L2_4">
+      <inertial>
+      <origin
+        xyz="-0.00106966507570738 -0.0713978397746767 -0.00106966507570611"
+        rpy="0 0 0" />
+      <mass
+        value="0.117746913814738" />
+      <inertia
+        ixx="9.95073774261661E-05"
+        ixy="-2.667473422779E-07"
+        ixz="-3.12070252262036E-06"
+        iyy="0.000106288781760734"
+        iyz="-2.88857039626312E-06"
+        izz="6.98820523527226E-06" />
+    </inertial>
+    <visual>
+      <origin
+        xyz="0 0 0"
+        rpy="0 0 0" />
+      <geometry>
+        <mesh
+          filename="package://iiwa_description/meshes/iiwa14/collision/Dual_Arm/Link4.STL" />
+      </geometry>
+      <material
+        name="">
+        <color
+          rgba="1 1 1 1" />
+      </material>
+    </visual>
+    <collision>
+      <origin
+        xyz="0 0 0"
+        rpy="0 0 0" />
+      <geometry>
+        <mesh
+          filename="package://iiwa_description/meshes/iiwa14/collision/Dual_Arm/Link4.STL" />
+      </geometry>
+    </collision>
+  </link>
+  <joint
+    name="J_24"
+    type="revolute">
+    <origin
+      xyz="0.0266700000000004 0.0019050000000066 0.0609600000000012"
+      rpy="-1.5707963267949 -0.824186362211141 -1.57079632679489" />
+    <parent
+      link="L2_3" />
+    <child
+      link="L2_4" />
+    <axis
+      xyz="0 0 1" />
+    <limit
+      lower="-0.5"
+      upper="0.5"
+      effort="2000"
+      velocity="13" />
+    <dynamics damping="${joint_damping}" friction = "${joint_friction}"/>
   </joint>
   </xacro:macro>

File: iiwa_description/urdf/gripper_eoat.xacro (robot description, xacro)
@@ -50,8 +50,8 @@
     type="revolute">
     <origin
-      xyz="0 0 0.045"
-      rpy="0 0 0" />
-    <parent
-      link="${robot_name}_link_7" />
+      xyz="0 -0.16 0"
+      rpy="${PIhalf} 0 0" />
+    <parent
+      link="Link4" />
     <child
       link="gripper_base_link" />
@@ -189,6 +189,65 @@
     <dynamics damping="${joint_damping}" friction = "${joint_friction}"/>
   </joint>
-   <link
-    name="claw_3_link">
+  <link
+    name="2_gripper_base_link">
+    <inertial>
+      <origin
+        xyz="0 0 0.00892"
+        rpy="0 0 0" />
+      <mass
+        value="1" />
+      <inertia
+        ixx="0.00003391"
+        ixy="0"
+        ixz="0"
+        iyy="0.00003391"
+        iyz="0"
+        izz="0.00003391" />
+    </inertial>
+    <visual>
+      <origin
+        xyz="0 0 0"
+        rpy="0 0 0" />
+      <geometry>
+        <mesh
+          filename="package://iiwa_description/meshes/iiwa14/collision/gripper_base.STL" />
+      </geometry>
+      <material
+        name="">
+        <color
+          rgba="0.79216 0.81961 0.93333 1" />
+      </material>
+    </visual>
+    <collision>
+      <origin
+        xyz="0 0 0"
+        rpy="0 0 0" />
+      <geometry>
+        <mesh
+          filename="package://iiwa_description/meshes/iiwa14/collision/gripper_base.STL" />
+      </geometry>
+    </collision>
+  </link>
+  <joint
+    name="2_gripper_base_joint"
+    type="revolute">
+    <origin
+      xyz="0 -0.16 0"
+      rpy="${PIhalf} 0 0" />
+    <parent
+      link="L2_4" />
+    <child
+      link="2_gripper_base_link" />
+    <axis
+      xyz="0 0 1" />
+    <limit
+      lower="0"
+      upper="0"
+      effort="2000"
+      velocity="13" />
+    <dynamics damping="${joint_damping}" friction = "${joint_friction}"/>
+  </joint>
+  <link
+    name="2_claw_1_link">
     <inertial>
       <origin
@@ -233,13 +292,13 @@
   </link>
   <joint
-    name="claw_3_joint"
-    type="revolute">
-    <origin
-      xyz="0.01979 0 0.0175"
-      rpy="0 0.1 ${PI}" />
-    <parent
-      link="gripper_base_link" />
-    <child
-      link="claw_3_link" />
+    name="2_claw_1_joint"
+    type="revolute">
+    <origin
+      xyz="0 -0.01979 0.0175"
+      rpy="0 0.1 ${PIhalf}" />
+    <parent
+      link="2_gripper_base_link" />
+    <child
+      link="2_claw_1_link" />
     <axis
       xyz="0 1 0" />
@@ -251,6 +310,6 @@
     <dynamics damping="${joint_damping}" friction = "${joint_friction}"/>
   </joint>
-     <link
-    name="claw_4_link">
+   <link
+    name="2_claw_2_link">
     <inertial>
       <origin
@@ -295,4 +354,129 @@
   </link>
   <joint
+    name="2_claw_2_joint"
+    type="revolute">
+    <origin
+      xyz="0 0.01979 0.0175"
+      rpy="0 0.1 -${PIhalf}" />
+    <parent
+      link="2_gripper_base_link" />
+    <child
+      link="2_claw_2_link" />
+    <axis
+      xyz="0 1 0" />
+    <limit
+      lower="-1.57"
+      upper="1.57"
+      effort="2000"
+      velocity="13" />
+    <dynamics damping="${joint_damping}" friction = "${joint_friction}"/>
+  </joint>
+  <!--
+   <link
+    name="claw_3_link">
+    <inertial>
+      <origin
+        xyz="-0.02212 0 0.0052"
+        rpy="0 0 0" />
+      <mass
+        value="0.00848" />
+      <inertia
+        ixx="3.2E-7"
+        ixy="0"
+        ixz="0"
+        iyx="0"
+        iyy="1.89E-6"
+        iyz="0"
+        izx="-6.7E-7"
+        izy="0"
+        izz="1.6E-6" />
+    </inertial>
+    <visual>
+      <origin
+        xyz="0 0 0"
+        rpy="0 0 0" />
+      <geometry>
+        <mesh
+          filename="package://iiwa_description/meshes/iiwa14/collision/gripper_claw.STL" />
+      </geometry>
+      <material
+        name="">
+        <color
+          rgba="0.79216 0.81961 0.93333 1" />
+      </material>
+    </visual>
+    <collision>
+      <origin
+        xyz="0 0 0"
+        rpy="0 0 0" />
+      <geometry>
+        <mesh
+          filename="package://iiwa_description/meshes/iiwa14/collision/gripper_claw.STL" />
+      </geometry>
+    </collision>
+  </link>
+  <joint
+    name="claw_3_joint"
+    type="revolute">
+    <origin
+      xyz="0.01979 0 0.0175"
+      rpy="0 0.1 ${PI}" />
+    <parent
+      link="gripper_base_link" />
+    <child
+      link="claw_3_link" />
+    <axis
+      xyz="0 1 0" />
+    <limit
+      lower="-1.57"
+      upper="1.57"
+      effort="2000"
+      velocity="13" />
+    <dynamics damping="${joint_damping}" friction = "${joint_friction}"/>
+  </joint>
+     <link
+    name="claw_4_link">
+    <inertial>
+      <origin
+        xyz="-0.02212 0 0.0052"
+        rpy="0 0 0" />
+      <mass
+        value="0.00848" />
+      <inertia
+        ixx="3.2E-7"
+        ixy="0"
+        ixz="0"
+        iyx="0"
+        iyy="1.89E-6"
+        iyz="0"
+        izx="-6.7E-7"
+        izy="0"
+        izz="1.6E-6" />
+    </inertial>
+    <visual>
+      <origin
+        xyz="0 0 0"
+        rpy="0 0 0" />
+      <geometry>
+        <mesh
+          filename="package://iiwa_description/meshes/iiwa14/collision/gripper_claw.STL" />
+      </geometry>
+      <material
+        name="">
+        <color
+          rgba="0.79216 0.81961 0.93333 1" />
+      </material>
+    </visual>
+    <collision>
+      <origin
+        xyz="0 0 0"
+        rpy="0 0 0" />
+      <geometry>
+        <mesh
+          filename="package://iiwa_description/meshes/iiwa14/collision/gripper_claw.STL" />
+      </geometry>
+    </collision>
+  </link>
+  <joint
     name="claw_4_joint"
     type="revolute">
@@ -313,4 +497,5 @@
     <dynamics damping="${joint_damping}" friction = "${joint_friction}"/>
   </joint>
+-->
   </xacro:macro>
 </robot>

File: iiwa_description/urdf/iiwa.gazebo.xacro (robot description, xacro)
@@ -3,5 +3,5 @@
   <xacro:macro name="iiwa_gazebo" params="robot_name">
     <!-- Load Gazebo lib and set the robot namespace -->
-    <gazebo>
+   <gazebo>
       <plugin name="gazebo_ros_control" filename="libgazebo_ros_control.so">
         <robotNamespace>/${robot_name}</robotNamespace>
@@ -31,5 +31,5 @@
     <!--Frame-->
     <gazebo reference="frame">
-      <material>Gazebo/White</material>
+      <material>Gazebo/Orange</material>
       <mu1>0.2</mu1>
       <mu2>0.2</mu2>
@@ -93,5 +93,5 @@
     </gazebo>
     <gazebo reference="base_link">
-      <material>Gazebo/White</material>
+      <material>Gazebo/Grey</material>
       <mu1>0.2</mu1>
       <mu2>0.2</mu2>
@@ -105,5 +105,5 @@
     </gazebo>
     <gazebo reference="Link2">
-      <material>Gazebo/White</material>
+      <material>Gazebo/Red</material>
       <mu1>0.2</mu1>
       <mu2>0.2</mu2>
@@ -117,8 +117,68 @@
     </gazebo>
     <gazebo reference="Link4">
-      <material>Gazebo/White</material>
-      <mu1>0.2</mu1>
-      <mu2>0.2</mu2>
-      <selfCollide>0</selfCollide>
+      <material>Gazebo/Red</material>
+      <mu1>0.2</mu1>
+      <mu2>0.2</mu2>
+      <selfCollide>0</selfCollide>
+    </gazebo>
+    <gazebo reference="L2_1">
+      <material>Gazebo/White</material>
+      <mu1>0.2</mu1>
+      <mu2>0.2</mu2>
+      <selfCollide>0</selfCollide>
+    </gazebo>
+    <gazebo reference="L2_2">
+      <material>Gazebo/Red</material>
+      <mu1>0.2</mu1>
+      <mu2>0.2</mu2>
+      <selfCollide>0</selfCollide>
+    </gazebo>
+    <gazebo reference="L2_3">
+      <material>Gazebo/White</material>
+      <mu1>0.2</mu1>
+      <mu2>0.2</mu2>
+      <selfCollide>0</selfCollide>
+    </gazebo>
+    <gazebo reference="L2_4">
+      <material>Gazebo/Red</material>
+      <mu1>0.2</mu1>
+      <mu2>0.2</mu2>
+      <selfCollide>0</selfCollide>
+    </gazebo>
+    <gazebo reference="gripper_base_link">
+      <material>Gazebo/White</material>
+      <mu1>0.2</mu1>
+      <mu2>0.2</mu2>
+      <selfCollide>0</selfCollide>
+    </gazebo>
+    <gazebo reference="claw_1_link">
+      <material>Gazebo/Red</material>
+      <mu1>0.2</mu1>
+      <mu2>0.2</mu2>
+      <selfCollide>1</selfCollide>
+    </gazebo>
+    <gazebo reference="claw_2_link">
+      <material>Gazebo/Red</material>
+      <mu1>0.2</mu1>
+      <mu2>0.2</mu2>
+      <selfCollide>1</selfCollide>
+    </gazebo>
+    <gazebo reference="2_gripper_base_link">
+      <material>Gazebo/White</material>
+      <mu1>0.2</mu1>
+      <mu2>0.2</mu2>
+      <selfCollide>0</selfCollide>
+    </gazebo>
+    <gazebo reference="2_claw_1_link">
+      <material>Gazebo/Red</material>
+      <mu1>0.2</mu1>
+      <mu2>0.2</mu2>
+      <selfCollide>1</selfCollide>
+    </gazebo>
+    <gazebo reference="2_claw_2_link">
+      <material>Gazebo/Red</material>
+      <mu1>0.2</mu1>
+      <mu2>0.2</mu2>
+      <selfCollide>1</selfCollide>
     </gazebo>
     <gazebo reference="${robot_name}_joint_7">
@@ -182,4 +242,5 @@
       <mu1>0.2</mu1>
       <mu2>0.2</mu2>
+      <selfCollide>0</selfCollide>
     </gazebo>
     <gazebo reference="surface">
@@ -189,5 +250,5 @@
       <kd>2500</kd>
       <kp>10000</kp>
-      <selfCollide>1</selfCollide>
+      <selfCollide>0</selfCollide>
     </gazebo>
   </xacro:macro>

File: iiwa_description/urdf/iiwa.transmission.xacro (robot description, xacro)
@@ -159,5 +159,115 @@
       </actuator>
     </transmission>
-<transmission name="pulsating_surface_tran_1">
+  <transmission name="J_21_tran">
+      <robotNamespace>/${robot_name}</robotNamespace>
+      <type>transmission_interface/SimpleTransmission</type>
+      <joint name="J_21">
+  <hardwareInterface>${hardware_interface}</hardwareInterface>
+      </joint>
+      <actuator name="J_21_motor">
+  <hardwareInterface>${hardware_interface}</hardwareInterface>
+  <mechanicalReduction>1</mechanicalReduction>
+      </actuator>
+    </transmission>
+  <transmission name="J_22_tran">
+      <robotNamespace>/${robot_name}</robotNamespace>
+      <type>transmission_interface/SimpleTransmission</type>
+      <joint name="J_22">
+  <hardwareInterface>${hardware_interface}</hardwareInterface>
+      </joint>
+      <actuator name="J_22_motor">
+  <hardwareInterface>${hardware_interface}</hardwareInterface>
+  <mechanicalReduction>1</mechanicalReduction>
+      </actuator>
+    </transmission>
+  <transmission name="J_23_tran">
+      <robotNamespace>/${robot_name}</robotNamespace>
+      <type>transmission_interface/SimpleTransmission</type>
+      <joint name="J_23">
+  <hardwareInterface>${hardware_interface}</hardwareInterface>
+      </joint>
+      <actuator name="J_23_motor">
+  <hardwareInterface>${hardware_interface}</hardwareInterface>
+  <mechanicalReduction>1</mechanicalReduction>
+      </actuator>
+    </transmission>
+  <transmission name="J_24_tran">
+      <robotNamespace>/${robot_name}</robotNamespace>
+      <type>transmission_interface/SimpleTransmission</type>
+      <joint name="J_24">
+  <hardwareInterface>${hardware_interface}</hardwareInterface>
+      </joint>
+      <actuator name="J_24_motor">
+  <hardwareInterface>${hardware_interface}</hardwareInterface>
+  <mechanicalReduction>1</mechanicalReduction>
+      </actuator>
+    </transmission>
+  <transmission name="gripper_base_joint_tran">
+      <robotNamespace>/${robot_name}</robotNamespace>
+      <type>transmission_interface/SimpleTransmission</type>
+      <joint name="gripper_base_joint">
+  <hardwareInterface>${hardware_interface}</hardwareInterface>
+      </joint>
+      <actuator name="gripper_base_joint_motor">
+  <hardwareInterface>${hardware_interface}</hardwareInterface>
+  <mechanicalReduction>1</mechanicalReduction>
+      </actuator>
+    </transmission>
+  <transmission name="claw_1_joint_tran">
+      <robotNamespace>/${robot_name}</robotNamespace>
+      <type>transmission_interface/SimpleTransmission</type>
+      <joint name="claw_1_joint">
+  <hardwareInterface>${hardware_interface}</hardwareInterface>
+      </joint>
+      <actuator name="claw_1_motor">
+  <hardwareInterface>${hardware_interface}</hardwareInterface>
+  <mechanicalReduction>1</mechanicalReduction>
+      </actuator>
+    </transmission>
+  <transmission name="claw_2_joint_tran">
+      <robotNamespace>/${robot_name}</robotNamespace>
+      <type>transmission_interface/SimpleTransmission</type>
+      <joint name="claw_2_joint">
+  <hardwareInterface>${hardware_interface}</hardwareInterface>
+      </joint>
+      <actuator name="claw_2_motor">
+  <hardwareInterface>${hardware_interface}</hardwareInterface>
+  <mechanicalReduction>1</mechanicalReduction>
+      </actuator>
+    </transmission>
+  <transmission name="2_gripper_base_joint_tran">
+      <robotNamespace>/${robot_name}</robotNamespace>
+      <type>transmission_interface/SimpleTransmission</type>
+      <joint name="2_gripper_base_joint">
+  <hardwareInterface>${hardware_interface}</hardwareInterface>
+      </joint>
+      <actuator name="2_gripper_base_joint_motor">
+  <hardwareInterface>${hardware_interface}</hardwareInterface>
+  <mechanicalReduction>1</mechanicalReduction>
+      </actuator>
+    </transmission>
+  <transmission name="2_claw_1_joint_tran">
+      <robotNamespace>/${robot_name}</robotNamespace>
+      <type>transmission_interface/SimpleTransmission</type>
+      <joint name="2_claw_1_joint">
+  <hardwareInterface>${hardware_interface}</hardwareInterface>
+      </joint>
+      <actuator name="2_claw_1_motor">
+  <hardwareInterface>${hardware_interface}</hardwareInterface>
+  <mechanicalReduction>1</mechanicalReduction>
+      </actuator>
+    </transmission>
+  <transmission name="2_claw_2_joint_tran">
+      <robotNamespace>/${robot_name}</robotNamespace>
+      <type>transmission_interface/SimpleTransmission</type>
+      <joint name="2_claw_2_joint">
+  <hardwareInterface>${hardware_interface}</hardwareInterface>
+      </joint>
+      <actuator name="2_claw_2_motor">
+  <hardwareInterface>${hardware_interface}</hardwareInterface>
+  <mechanicalReduction>1</mechanicalReduction>
+      </actuator>
+    </transmission>
+  <transmission name="pulsating_surface_tran_1">
       <robotNamespace>/${robot_name}</robotNamespace>
       <type>transmission_interface/SimpleTransmission</type>

File: iiwa_description/urdf/iiwa14.xacro (robot description, xacro)
@@ -10,9 +10,10 @@
   <xacro:include filename="$(find iiwa_description)/urdf/Dual_Arm.xacro" />
   <xacro:include filename="$(find iiwa_description)/urdf/pulsating_surface.urdf.xacro" />
+  <xacro:include filename="$(find iiwa_description)/urdf/gripper_eoat.xacro" />
   <!-- some constants -->
   <xacro:property name="safety_controller_k_pos" value="100" />
   <xacro:property name="safety_controller_k_vel" value="2" />
-  <xacro:property name="joint_damping" value="0.1" />
-  <xacro:property name="joint_friction" value="0.1"/>
+  <xacro:property name="joint_damping" value="0.4" />
+  <xacro:property name="joint_friction" value="0.4"/>
   <xacro:property name="max_effort" value="300"/>
   <xacro:property name="max_velocity" value="10"/>
@@ -349,4 +350,5 @@
     <!--<xacro:juans_eoat robot_name="${robot_name}"/>--> <!--Comented out EOAT-->
     <xacro:dual_arm_manipulator robot_name="${robot_name}"/>
+    <xacro:gripper_eoat robot_name="${robot_name}"/>
     <xacro:pulsating_surface />
     <xacro:iiwa_gazebo robot_name="${robot_name}"/>
