Commit message: Loaded controllers for all joints, added grippers

File: iiwa_description/urdf/pulsating_surface.urdf.xacro (robot description, xacro)
@@ -21,5 +21,5 @@
         <origin xyz="0 0 0" rpy="0 0 0"/>
         <geometry>
-          <mesh filename="package://iiwa_description/meshes/iiwa14/collision/Pulsating Surface/Base.STL"/>
+         <!-- <mesh filename="package://iiwa_description/meshes/iiwa14/collision/Pulsating Surface/Base.STL"/>-->
         </geometry>
         <material name="Grey"/>
@@ -37,7 +37,7 @@
       <parent link="post"/>
       <child link="surface"/>
-      <origin xyz="0 0 0.3" rpy="0 0 1.5707"/>
+      <origin xyz="0 0 -0.3" rpy="0 0 1.5707"/>
       <axis xyz="0 0 1"/>
-      <limit lower="-0.1" upper="0.3"
+      <limit lower="-0.8" upper="0.3"
              effort="10000" velocity="10000" />
       <dynamics damping="1" friction = "1"/>

Commit message: Updated some effort limits, using JointEffortControl for J2

File: iiwa_description/urdf/Dual_Arm.xacro (robot description, xacro)
@@ -61,5 +61,5 @@
       lower="-3.14"
       upper="3.14"
-      effort="2000"
+      effort="20000"
       velocity="13" />
     <dynamics damping="${joint_damping}" friction = "${joint_friction}"/>
@@ -120,5 +120,5 @@
       lower="-0.5"
       upper="0.5"
-      effort="2000"
+      effort="20000"
       velocity="13" />
     <dynamics damping="${joint_damping}" friction = "${joint_friction}"/>
@@ -179,5 +179,5 @@
       lower="-0.5"
       upper="0.5"
-      effort="2000"
+      effort="20000"
       velocity="13" />
     <dynamics damping="${joint_damping}" friction = "${joint_friction}"/>
@@ -238,5 +238,5 @@
       lower="-0.5"
       upper="0.5"
-      effort="2000"
+      effort="20000"
       velocity="13" />
     <dynamics damping="${joint_damping}" friction = "${joint_friction}"/>
@@ -297,5 +297,5 @@
       lower="-0.5"
       upper="0.5"
-      effort="2000"
+      effort="20000"
       velocity="13" />
     <dynamics damping="${joint_damping}" friction = "${joint_friction}"/>
@@ -356,5 +356,5 @@
       lower="-0.5"
       upper="0.5"
-      effort="2000"
+      effort="20000"
       velocity="13" />
     <dynamics damping="${joint_damping}" friction = "${joint_friction}"/>
@@ -415,5 +415,5 @@
       lower="-0.5"
       upper="0.5"
-      effort="2000"
+      effort="20000"
       velocity="13" />
     <dynamics damping="${joint_damping}" friction = "${joint_friction}"/>
@@ -474,5 +474,5 @@
       lower="-0.5"
       upper="0.5"
-      effort="2000"
+      effort="20000"
       velocity="13" />
     <dynamics damping="${joint_damping}" friction = "${joint_friction}"/>
@@ -533,5 +533,5 @@
       lower="-0.5"
       upper="0.5"
-      effort="2000"
+      effort="20000"
       velocity="13" />
     <dynamics damping="${joint_damping}" friction = "${joint_friction}"/>

File: iiwa_description/urdf/gripper_eoat.xacro (robot description, xacro)
@@ -59,7 +59,7 @@
       xyz="0 0 1" />
     <limit
-      lower="0"
-      upper="0"
-      effort="2000"
+      lower="-1.57"
+      upper="1.57"
+      effort="20000"
       velocity="13" />
     <dynamics damping="${joint_damping}" friction = "${joint_friction}"/>
@@ -123,5 +123,5 @@
       lower="-1.57"
       upper="1.57"
-      effort="2000"
+      effort="20000"
       velocity="13" />
     <dynamics damping="${joint_damping}" friction = "${joint_friction}"/>
@@ -185,5 +185,5 @@
       lower="-1.57"
       upper="1.57"
-      effort="2000"
+      effort="20000"
       velocity="13" />
     <dynamics damping="${joint_damping}" friction = "${joint_friction}"/>
@@ -242,7 +242,7 @@
       xyz="0 0 1" />
     <limit
-      lower="0"
-      upper="0"
-      effort="2000"
+      lower="-1.57"
+      upper="1.57"
+      effort="20000"
       velocity="13" />
     <dynamics damping="${joint_damping}" friction = "${joint_friction}"/>
@@ -306,5 +306,5 @@
       lower="-1.57"
       upper="1.57"
-      effort="2000"
+      effort="20000"
       velocity="13" />
     <dynamics damping="${joint_damping}" friction = "${joint_friction}"/>
@@ -368,5 +368,5 @@
       lower="-1.57"
       upper="1.57"
-      effort="2000"
+      effort="20000"
       velocity="13" />
     <dynamics damping="${joint_damping}" friction = "${joint_friction}"/>

File: iiwa_description/urdf/iiwa.gazebo.xacro (robot description, xacro)
@@ -156,5 +156,5 @@
       <mu1>0.2</mu1>
       <mu2>0.2</mu2>
-      <selfCollide>1</selfCollide>
+      <selfCollide>0</selfCollide>
     </gazebo>
     <gazebo reference="claw_2_link">
@@ -162,5 +162,5 @@
       <mu1>0.2</mu1>
       <mu2>0.2</mu2>
-      <selfCollide>1</selfCollide>
+      <selfCollide>0</selfCollide>
     </gazebo>
     <gazebo reference="2_gripper_base_link">
@@ -174,5 +174,5 @@
       <mu1>0.2</mu1>
       <mu2>0.2</mu2>
-      <selfCollide>1</selfCollide>
+      <selfCollide>0</selfCollide>
     </gazebo>
     <gazebo reference="2_claw_2_link">
@@ -180,5 +180,5 @@
       <mu1>0.2</mu1>
       <mu2>0.2</mu2>
-      <selfCollide>1</selfCollide>
+      <selfCollide>0</selfCollide>
     </gazebo>
     <gazebo reference="${robot_name}_joint_7">

File: iiwa_description/urdf/iiwa14.xacro (robot description, xacro)
@@ -16,5 +16,5 @@
   <xacro:property name="joint_damping" value="0.4" />
   <xacro:property name="joint_friction" value="0.4"/>
-  <xacro:property name="max_effort" value="300"/>
+  <xacro:property name="max_effort" value="5000"/>
   <xacro:property name="max_velocity" value="10"/>
   <xacro:macro name="iiwa14" params="parent hardware_interface robot_name *origin">

Commit message: Stable robot, tuning gains. Kuka has PositionJointInterface controllers while the manipulator has EffortJointInterface controllers

File: iiwa_description/urdf/Dual_Arm.xacro (robot description, xacro)
@@ -2,6 +2,6 @@
 <robot xmlns:xacro="http://www.ros.org/wiki/xacro">
   <xacro:macro name="dual_arm_manipulator" params="robot_name">
-  <xacro:property name="joint_friction" value="0.01" />
-  <xacro:property name="joint_damping" value="0.01" />
+  <xacro:property name="joint_friction" value="0.005" />
+  <xacro:property name="joint_damping" value="0.005" />
   <xacro:property name="PIhalf" value="1.570796" />
   <xacro:property name="PI" value="3.141592" />
@@ -118,6 +118,6 @@
       xyz="0 0 1" />
     <limit
-      lower="-0.5"
-      upper="0.5"
+      lower="-1"
+      upper="1"
       effort="20000"
       velocity="13" />
@@ -177,6 +177,6 @@
       xyz="0 0 1" />
     <limit
-      lower="-0.5"
-      upper="0.5"
+      lower="-1"
+      upper="1"
       effort="20000"
       velocity="13" />
@@ -236,6 +236,6 @@
       xyz="0 0 1" />
     <limit
-      lower="-0.5"
-      upper="0.5"
+      lower="-1"
+      upper="1"
       effort="20000"
       velocity="13" />
@@ -295,6 +295,6 @@
       xyz="0 0 1" />
     <limit
-      lower="-0.5"
-      upper="0.5"
+      lower="-1"
+      upper="1"
       effort="20000"
       velocity="13" />
@@ -354,6 +354,6 @@
       xyz="0 0 1" />
     <limit
-      lower="-0.5"
-      upper="0.5"
+      lower="-1"
+      upper="1"
       effort="20000"
       velocity="13" />
@@ -413,6 +413,6 @@
       xyz="0 0 1" />
     <limit
-      lower="-0.5"
-      upper="0.5"
+      lower="-1"
+      upper="1"
       effort="20000"
       velocity="13" />
@@ -472,6 +472,6 @@
       xyz="0 0 1" />
     <limit
-      lower="-0.5"
-      upper="0.5"
+      lower="-1"
+      upper="1"
       effort="20000"
       velocity="13" />
@@ -531,6 +531,6 @@
       xyz="0 0 1" />
     <limit
-      lower="-0.5"
-      upper="0.5"
+      lower="-1"
+      upper="1"
       effort="20000"
       velocity="13" />

File: iiwa_description/urdf/iiwa.transmission.xacro (robot description, xacro)
@@ -6,8 +6,8 @@
       <type>transmission_interface/SimpleTransmission</type>
       <joint name="${robot_name}_joint_1">
-	<hardwareInterface>${hardware_interface}</hardwareInterface>
+	<hardwareInterface>PositionJointInterface</hardwareInterface>
       </joint>
       <actuator name="${robot_name}_motor_1">
-	<hardwareInterface>${hardware_interface}</hardwareInterface>
+	<hardwareInterface>PositionJointInterface</hardwareInterface>
 	<mechanicalReduction>1</mechanicalReduction>
       </actuator>
@@ -17,8 +17,8 @@
       <type>transmission_interface/SimpleTransmission</type>
       <joint name="${robot_name}_joint_2">
-	<hardwareInterface>${hardware_interface}</hardwareInterface>
+	<hardwareInterface>PositionJointInterface</hardwareInterface>
       </joint>
       <actuator name="${robot_name}_motor_2">
-	<hardwareInterface>${hardware_interface}</hardwareInterface>
+	<hardwareInterface>PositionJointInterface</hardwareInterface>
 	<mechanicalReduction>1</mechanicalReduction>
       </actuator>
@@ -28,8 +28,8 @@
       <type>transmission_interface/SimpleTransmission</type>
       <joint name="${robot_name}_joint_3">
-	<hardwareInterface>${hardware_interface}</hardwareInterface>
+	<hardwareInterface>PositionJointInterface</hardwareInterface>
       </joint>
       <actuator name="${robot_name}_motor_3">
-	<hardwareInterface>${hardware_interface}</hardwareInterface>
+	<hardwareInterface>PositionJointInterface</hardwareInterface>
 	<mechanicalReduction>1</mechanicalReduction>
       </actuator>
@@ -39,8 +39,8 @@
       <type>transmission_interface/SimpleTransmission</type>
       <joint name="${robot_name}_joint_4">
-	<hardwareInterface>${hardware_interface}</hardwareInterface>
+	<hardwareInterface>PositionJointInterface</hardwareInterface>
       </joint>
       <actuator name="${robot_name}_motor_4">
-	<hardwareInterface>${hardware_interface}</hardwareInterface>
+	<hardwareInterface>PositionJointInterface</hardwareInterface>
 	<mechanicalReduction>1</mechanicalReduction>
       </actuator>
@@ -50,8 +50,8 @@
       <type>transmission_interface/SimpleTransmission</type>
       <joint name="${robot_name}_joint_5">
-	<hardwareInterface>${hardware_interface}</hardwareInterface>
+	<hardwareInterface>PositionJointInterface</hardwareInterface>
       </joint>
       <actuator name="${robot_name}_motor_5">
-	<hardwareInterface>${hardware_interface}</hardwareInterface>
+	<hardwareInterface>PositionJointInterface</hardwareInterface>
 	<mechanicalReduction>1</mechanicalReduction>
       </actuator>
@@ -61,8 +61,8 @@
       <type>transmission_interface/SimpleTransmission</type>
       <joint name="${robot_name}_joint_6">
-	<hardwareInterface>${hardware_interface}</hardwareInterface>
+	<hardwareInterface>PositionJointInterface</hardwareInterface>
       </joint>
       <actuator name="${robot_name}_motor_6">
-	<hardwareInterface>${hardware_interface}</hardwareInterface>
+	<hardwareInterface>PositionJointInterface</hardwareInterface>
 	<mechanicalReduction>1</mechanicalReduction>
       </actuator>
@@ -72,8 +72,8 @@
       <type>transmission_interface/SimpleTransmission</type>
       <joint name="${robot_name}_joint_7">
-	<hardwareInterface>${hardware_interface}</hardwareInterface>
+	<hardwareInterface>PositionJointInterface</hardwareInterface>
       </joint>
       <actuator name="${robot_name}_motor_7">
-	<hardwareInterface>${hardware_interface}</hardwareInterface>
+	<hardwareInterface>PositionJointInterface</hardwareInterface>
 	<mechanicalReduction>1</mechanicalReduction>
       </actuator>

File: iiwa_description/urdf/pulsating_surface.urdf.xacro (robot description, xacro)
@@ -2,4 +2,5 @@
 <robot xmlns:xacro="http://www.ros.org/wiki/xacro">
 <xacro:macro name = "pulsating_surface">
+<!--
   <joint
     name="fixed_1"
@@ -21,5 +22,4 @@
         <origin xyz="0 0 0" rpy="0 0 0"/>
         <geometry>
-         <!-- <mesh filename="package://iiwa_description/meshes/iiwa14/collision/Pulsating Surface/Base.STL"/>-->
         </geometry>
         <material name="Grey"/>
@@ -32,10 +32,10 @@
         <material name="Grey"/>
       </collision>
-    </link>
+    </link>-->
     <!-- joint between post and surface -->
     <joint name="prismatic_joint" type="prismatic">
-      <parent link="post"/>
+      <parent link="world"/>
       <child link="surface"/>
-      <origin xyz="0 0 -0.3" rpy="0 0 1.5707"/>
+      <origin xyz="1.5 0.25 0" rpy="0 0 1.5707"/>
       <axis xyz="0 0 1"/>
       <limit lower="-0.8" upper="0.3"
