Commit message: reorganized, updated the model for melodic

File: iiwa_description/urdf/Dual_Arm.xacro (robot description, xacro)
@@ -1,4 +1,6 @@
 <?xml version="1.0"?>
 <robot xmlns:xacro="http://www.ros.org/wiki/xacro">
+  <xacro:include filename="$(find iiwa_description)/urdf/dual_arm_right.xacro" />
+  <xacro:include filename="$(find iiwa_description)/urdf/dual_arm_left.xacro" />
   <xacro:macro name="dual_arm_manipulator" params="robot_name">
   <xacro:property name="joint_friction" value="0.005" />
@@ -13,5 +15,5 @@
         rpy="0 0 0" />
       <mass
-        value="81.613834759363" />
+        value="1.613834759363" />
       <inertia
         ixx="0"
@@ -65,476 +67,6 @@
     <dynamics damping="${joint_damping}" friction = "${joint_friction}"/>
   </joint>
-  <link
-    name="Link1">
-    <inertial>
-      <origin
-        xyz="0.00302464836897415 0.00148467584367146 -0.0196712040191069"
-        rpy="0 0 0" />
-      <mass
-        value="0.323170961054133" />
-      <inertia
-        ixx="9.86315700006277E-05"
-        ixy="-1.83712585125958E-06"
-        ixz="1.50310533353745E-05"
-        iyy="0.000101226511355012"
-        iyz="6.90483440689725E-06"
-        izz="4.61898687854836E-06" />
-    </inertial>
-    <visual>
-      <origin
-        xyz="0 0 0"
-        rpy="0 0 0" />
-      <geometry>
-        <mesh
-          filename="package://iiwa_description/meshes/iiwa14/collision/Dual_Arm/Link1.STL" />
-      </geometry>
-      <material
-        name="">
-        <color
-          rgba="1 1 1 1" />
-      </material>
-    </visual>
-    <collision>
-      <origin
-        xyz="0 0 0"
-        rpy="0 0 0" />
-      <geometry>
-        <mesh
-          filename="package://iiwa_description/meshes/iiwa14/collision/Dual_Arm/Link1.STL" />
-      </geometry>
-    </collision>
-  </link>
-  <joint
-    name="J_1"
-    type="revolute">
-    <origin
-      xyz="-0.0744445637977397 0.152871273073736 -0.110435575211296"
-      rpy="-1.43251148060093 -0.775712981728982 2.94539473140516" />
-    <parent
-      link="base_link" />
-    <child
-      link="Link1" />
-    <axis
-      xyz="0 0 1" />
-    <limit
-      lower="-3.14"
-      upper="3.14"
-      effort="20000"
-      velocity="13" />
-    <dynamics damping="${joint_damping}" friction = "${joint_friction}"/>
-  </joint>
-  <link
-    name="Link2">
-    <inertial>
-      <origin
-        xyz="-0.0841816926424142 -9.94783774485586E-05 0.00119770428720625"
-        rpy="0 0 0" />
-      <mass
-        value="0.161073886022953" />
-      <inertia
-        ixx="1.38598083295319E-06"
-        ixy="-3.76180464461997E-07"
-        ixz="5.01830776658136E-09"
-        iyy="0.000417336089370728"
-        iyz="3.07943156555252E-09"
-        izz="0.000417240402620394" />
-    </inertial>
-    <visual>
-      <origin
-        xyz="0 0 0"
-        rpy="0 0 0" />
-      <geometry>
-        <mesh
-          filename="package://iiwa_description/meshes/iiwa14/collision/Dual_Arm/Link2.STL" />
-      </geometry>
-      <material
-        name="">
-        <color
-          rgba="1 1 1 1" />
-      </material>
-    </visual>
-    <collision>
-      <origin
-        xyz="0 0 0"
-        rpy="0 0 0" />
-      <geometry>
-        <mesh
-          filename="package://iiwa_description/meshes/iiwa14/collision/Dual_Arm/Link2.STL" />
-      </geometry>
-    </collision>
-  </link>
-  <joint
-    name="J_2"
-    type="revolute">
-    <origin
-      xyz="0 0 -0.0635"
-      rpy="1.57079632679489 -0.380374098489847 0.317429885556193" />
-    <parent
-      link="Link1" />
-    <child
-      link="Link2" />
-    <axis
-      xyz="0 0 1" />
-    <limit
-      lower="-1.57"
-      upper="1.57"
-      effort="20000"
-      velocity="13" />
-    <dynamics damping="${joint_damping}" friction = "${joint_friction}"/>
-  </joint>
-  <link
-    name="Link3">
-    <inertial>
-      <origin
-        xyz="0.00289722994622221 0.00112305403125196 0.0290055866352336"
-        rpy="0 0 0" />
-      <mass
-        value="0.117746913814738" />
-      <inertia
-        ixx="9.95073774261661E-05"
-        ixy="-2.667473422779E-07"
-        ixz="-3.12070252262036E-06"
-        iyy="0.000106288781760734"
-        iyz="-2.88857039626312E-06"
-        izz="6.98820523527226E-06" />
-    </inertial>
-    <visual>
-      <origin
-        xyz="0 0 0"
-        rpy="0 0 0" />
-      <geometry>
-        <mesh
-          filename="package://iiwa_description/meshes/iiwa14/collision/Dual_Arm/Link3.STL" />
-      </geometry>
-      <material
-        name="">
-        <color
-          rgba="1 1 1 1" />
-      </material>
-    </visual>
-    <collision>
-      <origin
-        xyz="0 0 0"
-        rpy="0 0 0" />
-      <geometry>
-        <mesh
-          filename="package://iiwa_description/meshes/iiwa14/collision/Dual_Arm/Link3.STL" />
-      </geometry>
-    </collision>
-  </link>
-  <joint
-    name="J_3"
-    type="revolute">
-    <origin
-      xyz="-0.178688999999999 -0.00012700000000021 0"
-      rpy="-1.57079632679489 -0.00547118733939 1.5707963267949" />
-    <parent
-      link="Link2" />
-    <child
-      link="Link3" />
-    <axis
-      xyz="0 0 1" />
-    <limit
-      lower="-3.14"
-      upper="3.14"
-      effort="20000"
-      velocity="13" />
-    <dynamics damping="${joint_damping}" friction = "${joint_friction}"/>
-  </joint>
-  <link
-    name="Link4">
-    <inertial>
-      <origin
-        xyz="-0.00106966507570738 -0.0713978397746767 -0.00106966507570611"
-        rpy="0 0 0" />
-      <mass
-        value="0.117746913814738" />
-      <inertia
-        ixx="9.95073774261661E-05"
-        ixy="-2.667473422779E-07"
-        ixz="-3.12070252262036E-06"
-        iyy="0.000106288781760734"
-        iyz="-2.88857039626312E-06"
-        izz="6.98820523527226E-06" />
-    </inertial>
-    <visual>
-      <origin
-        xyz="0 0 0"
-        rpy="0 0 0" />
-      <geometry>
-        <mesh
-          filename="package://iiwa_description/meshes/iiwa14/collision/Dual_Arm/Link4.STL" />
-      </geometry>
-      <material
-        name="">
-        <color
-          rgba="1 1 1 1" />
-      </material>
-    </visual>
-    <collision>
-      <origin
-        xyz="0 0 0"
-        rpy="0 0 0" />
-      <geometry>
-        <mesh
-          filename="package://iiwa_description/meshes/iiwa14/collision/Dual_Arm/Link4.STL" />
-      </geometry>
-    </collision>
-  </link>
-  <joint
-    name="J_4"
-    type="revolute">
-    <origin
-      xyz="0.0266700000000004 0.0019050000000066 0.0609600000000012"
-      rpy="-1.5707963267949 -0.824186362211141 -1.57079632679489" />
-    <parent
-      link="Link3" />
-    <child
-      link="Link4" />
-    <axis
-      xyz="0 0 1" />
-    <limit
-      lower="-1.57"
-      upper="1.57"
-      effort="20000"
-      velocity="13" />
-    <dynamics damping="${joint_damping}" friction = "${joint_friction}"/>
-  </joint>
-  <link
-    name="L2_1">
-    <inertial>
-      <origin
-        xyz="0.00302464836897415 0.00148467584367146 -0.0196712040191069"
-        rpy="0 0 0" />
-      <mass
-        value="0.323170961054133" />
-      <inertia
-        ixx="9.86315700006277E-05"
-        ixy="-1.83712585125958E-06"
-        ixz="1.50310533353745E-05"
-        iyy="0.000101226511355012"
-        iyz="6.90483440689725E-06"
-        izz="4.61898687854836E-06" />
-    </inertial>
-    <visual>
-      <origin
-        xyz="0 0 0"
-        rpy="0 0 0" />
-      <geometry>
-        <mesh
-          filename="package://iiwa_description/meshes/iiwa14/collision/Dual_Arm/Link1.STL" />
-      </geometry>
-      <material
-        name="">
-        <color
-          rgba="1 1 1 1" />
-      </material>
-    </visual>
-    <collision>
-      <origin
-        xyz="0 0 0"
-        rpy="0 0 0" />
-      <geometry>
-        <mesh
-          filename="package://iiwa_description/meshes/iiwa14/collision/Dual_Arm/Link1.STL" />
-      </geometry>
-    </collision>
-  </link>
-  <joint
-    name="J_21"
-    type="revolute">
-    <origin
-      xyz="-0.0744445637977397 -0.152871273073736 -0.110435575211296"
-      rpy="1.43251148060093 -0.775712981728982 -2.94539473140516" />
-    <parent
-      link="base_link" />
-    <child
-      link="L2_1" />
-    <axis
-      xyz="0 0 1" />
-    <limit
-      lower="-3.14"
-      upper="3.14"
-      effort="20000"
-      velocity="13" />
-    <dynamics damping="${joint_damping}" friction = "${joint_friction}"/>
- </joint>
-  <link
-    name="L2_2">
-    <inertial>
-      <origin
-        xyz="-0.0841816926424142 -9.94783774485586E-05 0.00119770428720625"
-        rpy="0 0 0" />
-      <mass
-        value="0.161073886022953" />
-      <inertia
-        ixx="1.38598083295319E-06"
-        ixy="-3.76180464461997E-07"
-        ixz="5.01830776658136E-09"
-        iyy="0.000417336089370728"
-        iyz="3.07943156555252E-09"
-        izz="0.000417240402620394" />
-    </inertial>
-    <visual>
-      <origin
-        xyz="0 0 0"
-        rpy="0 0 0" />
-      <geometry>
-        <mesh
-          filename="package://iiwa_description/meshes/iiwa14/collision/Dual_Arm/Link2.STL" />
-      </geometry>
-      <material
-        name="">
-        <color
-          rgba="0.898039215686275 0.898039215686275 0.898039215686275 1" />
-      </material>
-    </visual>
-    <collision>
-      <origin
-        xyz="0 0 0"
-        rpy="0 0 0" />
-      <geometry>
-        <mesh
-          filename="package://iiwa_description/meshes/iiwa14/collision/Dual_Arm/Link2.STL" />
-      </geometry>
-    </collision>
-  </link>
-  <joint
-    name="J_22"
-    type="revolute">
-    <origin
-      xyz="0 0 -0.0635"
-      rpy="1.57079632679489 -0.380374098489847 0.317429885556193" />
-    <parent
-      link="L2_1" />
-    <child
-      link="L2_2" />
-    <axis
-      xyz="0 0 1" />
-    <limit
-      lower="-1.57"
-      upper="1.57"
-      effort="20000"
-      velocity="13" />
-    <dynamics damping="${joint_damping}" friction = "${joint_friction}"/>
-  </joint>
-  <link
-    name="L2_3">
-    <inertial>
-      <origin
-        xyz="0.00289722994622221 0.00112305403125196 0.0290055866352336"
-        rpy="0 0 0" />
-      <mass
-        value="0.117746913814738" />
-      <inertia
-        ixx="9.95073774261661E-05"
-        ixy="-2.667473422779E-07"
-        ixz="-3.12070252262036E-06"
-        iyy="0.000106288781760734"
-        iyz="-2.88857039626312E-06"
-        izz="6.98820523527226E-06" />
-    </inertial>
-    <visual>
-      <origin
-        xyz="0 0 0"
-        rpy="0 0 0" />
-      <geometry>
-        <mesh
-          filename="package://iiwa_description/meshes/iiwa14/collision/Dual_Arm/Link3.STL" />
-      </geometry>
-      <material
-        name="">
-        <color
-          rgba="1 1 1 1" />
-      </material>
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
File: iiwa_description/urdf/gripper_eoat.xacro (robot description, xacro)
@@ -53,5 +53,5 @@
       rpy="${PIhalf} 0 0" />
     <parent
-      link="Link4" />
+      link="Link_L4" />
     <child
       link="gripper_base_link" />
@@ -236,5 +236,5 @@
       rpy="${PIhalf} 0 0" />
     <parent
-      link="L2_4" />
+      link="Link_R4" />
     <child
       link="2_gripper_base_link" />
@@ -372,130 +372,4 @@
     <dynamics damping="${joint_damping}" friction = "${joint_friction}"/>
   </joint>
-  <!--
-   <link
-    name="claw_3_link">
-    <inertial>
-      <origin
-        xyz="-0.02212 0 0.0052"
-        rpy="0 0 0" />
-      <mass
-        value="0.00848" />
-      <inertia
-        ixx="3.2E-7"
-        ixy="0"
-        ixz="0"
-        iyx="0"
-        iyy="1.89E-6"
-        iyz="0"
-        izx="-6.7E-7"
-        izy="0"
-        izz="1.6E-6" />
-    </inertial>
-    <visual>
-      <origin
-        xyz="0 0 0"
-        rpy="0 0 0" />
-      <geometry>
-        <mesh
-          filename="package://iiwa_description/meshes/iiwa14/collision/gripper_claw.STL" />
-      </geometry>
-      <material
-        name="">
-        <color
-          rgba="0.79216 0.81961 0.93333 1" />
-      </material>
-    </visual>
-    <collision>
-      <origin
-        xyz="0 0 0"
-        rpy="0 0 0" />
-      <geometry>
-        <mesh
-          filename="package://iiwa_description/meshes/iiwa14/collision/gripper_claw.STL" />
-      </geometry>
-    </collision>
-  </link>
-  <joint
-    name="claw_3_joint"
-    type="revolute">
-    <origin
-      xyz="0.01979 0 0.0175"
-      rpy="0 0.1 ${PI}" />
-    <parent
-      link="gripper_base_link" />
-    <child
-      link="claw_3_link" />
-    <axis
-      xyz="0 1 0" />
-    <limit
-      lower="-1.57"
-      upper="1.57"
-      effort="2000"
-      velocity="13" />
-    <dynamics damping="${joint_damping}" friction = "${joint_friction}"/>
-  </joint>
-     <link
-    name="claw_4_link">
-    <inertial>
-      <origin
-        xyz="-0.02212 0 0.0052"
-        rpy="0 0 0" />
-      <mass
-        value="0.00848" />
-      <inertia
-        ixx="3.2E-7"
-        ixy="0"
-        ixz="0"
-        iyx="0"
-        iyy="1.89E-6"
-        iyz="0"
-        izx="-6.7E-7"
-        izy="0"
-        izz="1.6E-6" />
-    </inertial>
-    <visual>
-      <origin
-        xyz="0 0 0"
-        rpy="0 0 0" />
-      <geometry>
-        <mesh
-          filename="package://iiwa_description/meshes/iiwa14/collision/gripper_claw.STL" />
-      </geometry>
-      <material
-        name="">
-        <color
-          rgba="0.79216 0.81961 0.93333 1" />
-      </material>
-    </visual>
-    <collision>
-      <origin
-        xyz="0 0 0"
-        rpy="0 0 0" />
-      <geometry>
-        <mesh
-          filename="package://iiwa_description/meshes/iiwa14/collision/gripper_claw.STL" />
-      </geometry>
-    </collision>
-  </link>
-  <joint
-    name="claw_4_joint"
-    type="revolute">
-    <origin
-      xyz="-0.01979 0 0.0175"
-      rpy="0 0.1 0" />
-    <parent
-      link="gripper_base_link" />
-    <child
-      link="claw_4_link" />
-    <axis
-      xyz="0 1 0" />
-    <limit
-      lower="-1.57"
-      upper="1.57"
-      effort="2000"
-      velocity="13" />
-    <dynamics damping="${joint_damping}" friction = "${joint_friction}"/>
-  </joint>
--->
   </xacro:macro>
 </robot>
