Commit message: reorganized, updated the model for melodic

File: iiwa_description/urdf/iiwa.transmission.xacro (robot description, xacro)
@@ -1,13 +1,12 @@
 <?xml version="1.0"?>
 <robot xmlns:xacro="http://www.ros.org/wiki/xacro">
-  <xacro:macro name="iiwa_transmission" params="hardware_interface">
+  <xacro:macro name="iiwa_transmission" params="hardware_interface robot_name">
     <transmission name="${robot_name}_tran_1">
       <robotNamespace>/${robot_name}</robotNamespace>
       <type>transmission_interface/SimpleTransmission</type>
       <joint name="${robot_name}_joint_1">
-	<hardwareInterface>PositionJointInterface</hardwareInterface>
+	<hardwareInterface>hardware_interface/PositionJointInterface</hardwareInterface>
       </joint>
       <actuator name="${robot_name}_motor_1">
-	<hardwareInterface>PositionJointInterface</hardwareInterface>
 	<mechanicalReduction>1</mechanicalReduction>
       </actuator>
@@ -17,8 +16,7 @@
       <type>transmission_interface/SimpleTransmission</type>
       <joint name="${robot_name}_joint_2">
-	<hardwareInterface>PositionJointInterface</hardwareInterface>
+	    <hardwareInterface>hardware_interface/PositionJointInterface</hardwareInterface>
       </joint>
       <actuator name="${robot_name}_motor_2">
-	<hardwareInterface>PositionJointInterface</hardwareInterface>
 	<mechanicalReduction>1</mechanicalReduction>
       </actuator>
@@ -28,8 +26,8 @@
       <type>transmission_interface/SimpleTransmission</type>
       <joint name="${robot_name}_joint_3">
-	<hardwareInterface>PositionJointInterface</hardwareInterface>
+	    <hardwareInterface>hardware_interface/PositionJointInterface</hardwareInterface>
       </joint>
       <actuator name="${robot_name}_motor_3">
-	<hardwareInterface>PositionJointInterface</hardwareInterface>
+        <hardwareInterface>hardware_interface/PositionJointInterface</hardwareInterface>
 	<mechanicalReduction>1</mechanicalReduction>
       </actuator>
@@ -39,8 +37,7 @@
       <type>transmission_interface/SimpleTransmission</type>
       <joint name="${robot_name}_joint_4">
-	<hardwareInterface>PositionJointInterface</hardwareInterface>
+	    <hardwareInterface>hardware_interface/PositionJointInterface</hardwareInterface>
       </joint>
       <actuator name="${robot_name}_motor_4">
-	<hardwareInterface>PositionJointInterface</hardwareInterface>
 	<mechanicalReduction>1</mechanicalReduction>
       </actuator>
@@ -50,8 +47,7 @@
       <type>transmission_interface/SimpleTransmission</type>
       <joint name="${robot_name}_joint_5">
-	<hardwareInterface>PositionJointInterface</hardwareInterface>
+	    <hardwareInterface>hardware_interface/PositionJointInterface</hardwareInterface>
       </joint>
       <actuator name="${robot_name}_motor_5">
-	<hardwareInterface>PositionJointInterface</hardwareInterface>
 	<mechanicalReduction>1</mechanicalReduction>
       </actuator>
@@ -61,8 +57,7 @@
       <type>transmission_interface/SimpleTransmission</type>
       <joint name="${robot_name}_joint_6">
-	<hardwareInterface>PositionJointInterface</hardwareInterface>
+	    <hardwareInterface>hardware_interface/PositionJointInterface</hardwareInterface>
       </joint>
       <actuator name="${robot_name}_motor_6">
-	<hardwareInterface>PositionJointInterface</hardwareInterface>
 	<mechanicalReduction>1</mechanicalReduction>
       </actuator>
@@ -72,44 +67,17 @@
       <type>transmission_interface/SimpleTransmission</type>
       <joint name="${robot_name}_joint_7">
-	<hardwareInterface>PositionJointInterface</hardwareInterface>
+	    <hardwareInterface>hardware_interface/PositionJointInterface</hardwareInterface>
       </joint>
       <actuator name="${robot_name}_motor_7">
-	<hardwareInterface>PositionJointInterface</hardwareInterface>
-	<mechanicalReduction>1</mechanicalReduction>
-      </actuator>
-    </transmission>
-    <!--Added for EOAT-->
-<!--
-  <transmission name="eoat_tran1">
-    <robotNamespace>/${robot_name}</robotNamespace>
-    <type>transmission_interface/SimpleTransmission</type>
-    <joint name="rotating_base_joint">
-      <hardwareInterface>${hardware_interface}</hardwareInterface>
-    </joint>
-    <actuator name="motor1">
-      <hardwareInterface>${hardware_interface}</hardwareInterface>
-      <mechanicalReduction>1</mechanicalReduction>
-    </actuator>
-  </transmission>
-  <transmission name="eoat_tran2">
-    <robotNamespace>/${robot_name}</robotNamespace>
-    <type>transmission_interface/SimpleTransmission</type>
-    <joint name="rotating_arm_joint">
-      <hardwareInterface>${hardware_interface}</hardwareInterface>
-    </joint>
-    <actuator name="motor2">
-      <hardwareInterface>${hardware_interface}</hardwareInterface>
-      <mechanicalReduction>1</mechanicalReduction>
-    </actuator>
-  </transmission>
--->
+	<mechanicalReduction>1</mechanicalReduction>
+      </actuator>
+    </transmission>
 <transmission name="manipulator_tran_1">
       <robotNamespace>/${robot_name}</robotNamespace>
       <type>transmission_interface/SimpleTransmission</type>
       <joint name="dual_arm_base_joint">
-  <hardwareInterface>${hardware_interface}</hardwareInterface>
+      <hardwareInterface>hardware_interface/${hardware_interface}</hardwareInterface>
       </joint>
       <actuator name="dual_arm_base_motor">
-  <hardwareInterface>${hardware_interface}</hardwareInterface>
   <mechanicalReduction>1</mechanicalReduction>
       </actuator>
@@ -118,9 +86,8 @@
       <robotNamespace>/${robot_name}</robotNamespace>
       <type>transmission_interface/SimpleTransmission</type>
-      <joint name="J_1">
-  <hardwareInterface>${hardware_interface}</hardwareInterface>
+      <joint name="J_L1">
+      <hardwareInterface>hardware_interface/${hardware_interface}</hardwareInterface>
       </joint>
       <actuator name="J_1_motor">
-  <hardwareInterface>${hardware_interface}</hardwareInterface>
   <mechanicalReduction>1</mechanicalReduction>
       </actuator>
@@ -129,9 +96,8 @@
       <robotNamespace>/${robot_name}</robotNamespace>
       <type>transmission_interface/SimpleTransmission</type>
-      <joint name="J_2">
-  <hardwareInterface>${hardware_interface}</hardwareInterface>
+      <joint name="J_L2">
+  <hardwareInterface>hardware_interface/${hardware_interface}</hardwareInterface>
       </joint>
       <actuator name="J_2_motor">
-  <hardwareInterface>${hardware_interface}</hardwareInterface>
   <mechanicalReduction>1</mechanicalReduction>
       </actuator>
@@ -140,9 +106,8 @@
       <robotNamespace>/${robot_name}</robotNamespace>
       <type>transmission_interface/SimpleTransmission</type>
-      <joint name="J_3">
-  <hardwareInterface>${hardware_interface}</hardwareInterface>
+      <joint name="J_L3">
+  <hardwareInterface>hardware_interface/${hardware_interface}</hardwareInterface>
       </joint>
       <actuator name="J_3_motor">
-  <hardwareInterface>${hardware_interface}</hardwareInterface>
   <mechanicalReduction>1</mechanicalReduction>
       </actuator>
@@ -151,9 +116,8 @@
       <robotNamespace>/${robot_name}</robotNamespace>
       <type>transmission_interface/SimpleTransmission</type>
-      <joint name="J_4">
-  <hardwareInterface>${hardware_interface}</hardwareInterface>
+      <joint name="J_L4">
+  <hardwareInterface>hardware_interface/${hardware_interface}</hardwareInterface>
       </joint>
       <actuator name="J_4_motor">
-  <hardwareInterface>${hardware_interface}</hardwareInterface>
   <mechanicalReduction>1</mechanicalReduction>
       </actuator>
@@ -162,9 +126,8 @@
       <robotNamespace>/${robot_name}</robotNamespace>
       <type>transmission_interface/SimpleTransmission</type>
-      <joint name="J_21">
-  <hardwareInterface>${hardware_interface}</hardwareInterface>
-      </joint>
-      <actuator name="J_21_motor">
-  <hardwareInterface>${hardware_interface}</hardwareInterface>
+      <joint name="J_R1">
+  <hardwareInterface>hardware_interface/${hardware_interface}</hardwareInterface>
+      </joint>
+      <actuator name="J_R1_motor">
   <mechanicalReduction>1</mechanicalReduction>
       </actuator>
@@ -173,9 +136,8 @@
       <robotNamespace>/${robot_name}</robotNamespace>
       <type>transmission_interface/SimpleTransmission</type>
-      <joint name="J_22">
-  <hardwareInterface>${hardware_interface}</hardwareInterface>
-      </joint>
-      <actuator name="J_22_motor">
-  <hardwareInterface>${hardware_interface}</hardwareInterface>
+      <joint name="J_R2">
+  <hardwareInterface>hardware_interface/${hardware_interface}</hardwareInterface>
+      </joint>
+      <actuator name="J_R2_motor">
   <mechanicalReduction>1</mechanicalReduction>
       </actuator>
@@ -184,9 +146,8 @@
       <robotNamespace>/${robot_name}</robotNamespace>
       <type>transmission_interface/SimpleTransmission</type>
-      <joint name="J_23">
-  <hardwareInterface>${hardware_interface}</hardwareInterface>
-      </joint>
-      <actuator name="J_23_motor">
-  <hardwareInterface>${hardware_interface}</hardwareInterface>
+      <joint name="J_R3">
+  <hardwareInterface>hardware_interface/${hardware_interface}</hardwareInterface>
+      </joint>
+      <actuator name="J_R3_motor">
   <mechanicalReduction>1</mechanicalReduction>
       </actuator>
@@ -195,9 +156,8 @@
       <robotNamespace>/${robot_name}</robotNamespace>
       <type>transmission_interface/SimpleTransmission</type>
-      <joint name="J_24">
-  <hardwareInterface>${hardware_interface}</hardwareInterface>
-      </joint>
-      <actuator name="J_24_motor">
-  <hardwareInterface>${hardware_interface}</hardwareInterface>
+      <joint name="J_R4">
+  <hardwareInterface>hardware_interface/${hardware_interface}</hardwareInterface>
+      </joint>
+      <actuator name="J_R4_motor">
   <mechanicalReduction>1</mechanicalReduction>
       </actuator>
@@ -207,8 +167,7 @@
       <type>transmission_interface/SimpleTransmission</type>
       <joint name="gripper_base_joint">
-  <hardwareInterface>${hardware_interface}</hardwareInterface>
+  <hardwareInterface>hardware_interface/${hardware_interface}</hardwareInterface>
       </joint>
       <actuator name="gripper_base_joint_motor">
-  <hardwareInterface>${hardware_interface}</hardwareInterface>
   <mechanicalReduction>1</mechanicalReduction>
       </actuator>
@@ -218,8 +177,7 @@
       <type>transmission_interface/SimpleTransmission</type>
       <joint name="claw_1_joint">
-  <hardwareInterface>${hardware_interface}</hardwareInterface>
+  <hardwareInterface>hardware_interface/${hardware_interface}</hardwareInterface>
       </joint>
       <actuator name="claw_1_motor">
-  <hardwareInterface>${hardware_interface}</hardwareInterface>
   <mechanicalReduction>1</mechanicalReduction>
       </actuator>
@@ -229,8 +187,7 @@
       <type>transmission_interface/SimpleTransmission</type>
       <joint name="claw_2_joint">
-  <hardwareInterface>${hardware_interface}</hardwareInterface>
+  <hardwareInterface>hardware_interface/${hardware_interface}</hardwareInterface>
       </joint>
       <actuator name="claw_2_motor">
-  <hardwareInterface>${hardware_interface}</hardwareInterface>
   <mechanicalReduction>1</mechanicalReduction>
       </actuator>
@@ -240,8 +197,7 @@
       <type>transmission_interface/SimpleTransmission</type>
       <joint name="2_gripper_base_joint">
-  <hardwareInterface>${hardware_interface}</hardwareInterface>
+  <hardwareInterface>hardware_interface/${hardware_interface}</hardwareInterface>
       </joint>
       <actuator name="2_gripper_base_joint_motor">
-  <hardwareInterface>${hardware_interface}</hardwareInterface>
   <mechanicalReduction>1</mechanicalReduction>
       </actuator>
@@ -251,8 +207,7 @@
       <type>transmission_interface/SimpleTransmission</type>
       <joint name="2_claw_1_joint">
-  <hardwareInterface>${hardware_interface}</hardwareInterface>
+  <hardwareInterface>hardware_interface/${hardware_interface}</hardwareInterface>
       </joint>
       <actuator name="2_claw_1_motor">
-  <hardwareInterface>${hardware_interface}</hardwareInterface>
   <mechanicalReduction>1</mechanicalReduction>
       </actuator>
@@ -262,8 +217,7 @@
       <type>transmission_interface/SimpleTransmission</type>
       <joint name="2_claw_2_joint">
-  <hardwareInterface>${hardware_interface}</hardwareInterface>
+  <hardwareInterface>hardware_interface/${hardware_interface}</hardwareInterface>
       </joint>
       <actuator name="2_claw_2_motor">
-  <hardwareInterface>${hardware_interface}</hardwareInterface>
   <mechanicalReduction>1</mechanicalReduction>
       </actuator>
@@ -273,8 +227,7 @@
       <type>transmission_interface/SimpleTransmission</type>
       <joint name="prismatic_joint">
-  <hardwareInterface>${hardware_interface}</hardwareInterface>
+  <hardwareInterface>hardware_interface/${hardware_interface}</hardwareInterface>
       </joint>
       <actuator name="pulsating_surface_motor_1">
-  <hardwareInterface>${hardware_interface}</hardwareInterface>
   <mechanicalReduction>1</mechanicalReduction>
       </actuator>

File: iiwa_description/urdf/iiwa14.xacro (robot description, xacro)
@@ -1,14 +1,4 @@
 <?xml version="1.0"?>
 <robot xmlns:xacro="http://www.ros.org/wiki/xacro">
-  <!-- Import all Gazebo-customization elements, including Gazebo colors -->
-  <xacro:include filename="$(find iiwa_description)/urdf/iiwa.gazebo.xacro" />
-  <!-- Import Transmissions -->
-  <xacro:include filename="$(find iiwa_description)/urdf/iiwa.transmission.xacro" />
-  <!-- Include Utilities -->
-  <xacro:include filename="$(find iiwa_description)/urdf/utilities.xacro" />
-  <!-- Include EOAT -->
-  <xacro:include filename="$(find iiwa_description)/urdf/Dual_Arm.xacro" />
-  <xacro:include filename="$(find iiwa_description)/urdf/pulsating_surface.urdf.xacro" />
-  <xacro:include filename="$(find iiwa_description)/urdf/gripper_eoat.xacro" />
   <!-- some constants -->
   <xacro:property name="safety_controller_k_pos" value="100" />
@@ -18,4 +8,8 @@
   <xacro:property name="max_effort" value="5000"/>
   <xacro:property name="max_velocity" value="100"/>
+  <xacro:property name="joint_friction" value="0.005" />
+  <xacro:property name="joint_damping" value="0.005" />
+  <xacro:property name="PIhalf" value="1.570796" />
+  <xacro:property name="PI" value="3.141592" />
   <xacro:macro name="iiwa14" params="parent hardware_interface robot_name *origin">
     <!--joint between {parent} and link_0-->
@@ -270,60 +264,4 @@
       </collision>
     </link>
-    <!-- Commented force sensor EOAT
-    <joint name="${robot_name}_joint_ee" type="fixed">
-      <parent link="${robot_name}_link_7"/>
-      <child link="${robot_name}_link_ee"/>
-      <origin xyz="0 0 0.0525" rpy="1.57 0 0"/>
-    </joint>
-    <link name="${robot_name}_link_ee">
-    </link>
-  <link
-    name="${robot_name}_link_ee">
-    <inertial>
-      <origin
-        xyz="9.5698E-05 0.0082673 2.27179999999949E-06"
-        rpy="0 0 0" />
-      <mass
-        value="0.042407" />
-      <inertia
-        ixx="2.09361562697698E-05"
-        ixy="-1.03008820969214E-10"
-        ixz="7.85583672233988E-16"
-        iyy="1.20677052581546E-05"
-        iyz="1.27817724850131E-09"
-        izz="2.2947402405232E-05" />
-    </inertial>
-    <visual>
-      <origin
-        xyz="0 0 0"
-        rpy="1.5707963267949 0 0" />
-      <geometry>
-        <mesh
-          filename="package://iiwa_description/meshes/iiwa14/collision/flange.STL" />
-      </geometry>
-      <material
-        name="">
-        <color
-          rgba="0.79216 0.81961 0.93333 1" />
-      </material>
-    </visual>
-    <collision>
-      <origin
-        xyz="0 0 0"
-        rpy="1.5707963267949 0 0" />
-      <geometry>
-        <mesh
-          filename="package://iiwa_description/meshes/iiwa14/collision/flange.STL" />
-      </geometry>
-    </collision>
-  </link>
--->
-    <!--Extensions -->
-    <!--<xacro:juans_eoat robot_name="${robot_name}"/>--> <!--Comented out EOAT-->
-    <xacro:dual_arm_manipulator robot_name="${robot_name}"/>
-    <xacro:gripper_eoat robot_name="${robot_name}"/>
-    <xacro:pulsating_surface />
-    <xacro:iiwa_gazebo robot_name="${robot_name}"/>
-    <xacro:iiwa_transmission hardware_interface="${hardware_interface}"/>
   </xacro:macro>
 </robot>

File: iiwa_description/urdf/kuka_base_frame.xacro (robot description, xacro)
@@ -1,14 +1,9 @@
 <?xml version="1.0"?>
-<robot name="iiwa14" xmlns:xacro="http://www.ros.org/wiki/xacro">
-  <xacro:arg name="hardware_interface" default="PositionJointInterface"/>
-  <xacro:arg name="robot_name" default="iiwa"/>
-  <xacro:arg name="origin_xyz" default="0 0 0"/>
-  <xacro:arg name="origin_rpy" default="0 0 0"/>
-  <!-- Import Rviz colors -->
-  <xacro:include filename="$(find iiwa_description)/urdf/iiwa.gazebo.xacro" />
-  <xacro:include filename="$(find iiwa_description)/urdf/materials.xacro" />
-  <!--Import the lbr iiwa macro -->
-  <xacro:include filename="$(find iiwa_description)/urdf/iiwa14.xacro"/>
-  <!-- Fix to world just for testing -->
+<robot xmlns:xacro="http://www.ros.org/wiki/xacro">
+  <xacro:property name="joint_friction" value="0.005" />
+  <xacro:property name="joint_damping" value="0.005" />
+  <xacro:property name="PIhalf" value="1.570796" />
+  <xacro:property name="PI" value="3.141592" />
+  <xacro:macro name="kuka_base_frame" params="robot_name">
   <link name="world" />
   <joint
@@ -61,8 +56,4 @@
     </collision>
   </link>
-  <!--iiwa-->
-  <xacro:iiwa14 hardware_interface="$(arg hardware_interface)" robot_name="$(arg robot_name)" parent="world">
-    <origin xyz="$(arg origin_xyz)" rpy="$(arg origin_rpy)" />
-  </xacro:iiwa14>
-  <xacro:iiwa_gazebo robot_name="$(arg robot_name)"/>
+  </xacro:macro>
 </robot>

File: iiwa_description/urdf/pulsating_surface.xacro (robot description, xacro)
@@ -1,36 +1,5 @@
 <?xml version="1.0"?>
 <robot xmlns:xacro="http://www.ros.org/wiki/xacro">
-<xacro:macro name = "pulsating_surface">
-<!--
-  <joint
-    name="fixed_1"
-    type="fixed">
-    <parent
-      link="world" />
-    <child
-      link="post" />
-     <origin xyz="1.5 0.25 0" rpy="0 0 0"/>
-    <axis xyz="0 0 1"/>
-  </joint>
-  <link name="post">
-      <inertial>
-        <origin xyz="0 0 0" rpy="0 0 0"/>
-        <mass value="5"/>
-        <inertia ixx="1"  ixy="0"  ixz="0" iyy="1" iyz="0" izz="1" />
-      </inertial>
-      <visual>
-        <origin xyz="0 0 0" rpy="0 0 0"/>
-        <geometry>
-        </geometry>
-        <material name="Grey"/>
-      </visual>
-      <collision>
-        <origin xyz="0 0 0" rpy="0 0 0"/>
-        <geometry>
-          <mesh filename="package://iiwa_description/meshes/iiwa14/collision/Pulsating Surface/Base.STL"/>
-        </geometry>
-        <material name="Grey"/>
-      </collision>
-    </link>-->
+<xacro:macro name = "pulsating_surface" >
     <!-- joint between post and surface -->
     <joint name="prismatic_joint" type="prismatic">
