Commit message: completed model works in melodic, changed the structure of the tree

File: iiwa_description/urdf/Dual_Arm.xacro (robot description, xacro)
@@ -3,4 +3,6 @@
   <xacro:include filename="$(find iiwa_description)/urdf/dual_arm_right.xacro" />
   <xacro:include filename="$(find iiwa_description)/urdf/dual_arm_left.xacro" />
+  <xacro:include filename="$(find iiwa_description)/urdf/gripper_L.xacro" />
+  <xacro:include filename="$(find iiwa_description)/urdf/gripper_R.xacro" />
   <xacro:macro name="dual_arm_manipulator" params="robot_name">
   <xacro:property name="joint_friction" value="0.005" />
@@ -8,24 +10,32 @@
   <xacro:property name="PIhalf" value="1.570796" />
   <xacro:property name="PI" value="3.141592" />
+  <joint
+  name="dual_arm_base_joint"
+  type="fixed">
+  <origin
+    xyz="0 0 0.045"
+    rpy="${PI} 0 0" />
+  <parent
+    link="${robot_name}_link_7" />
+  <child
+    link="base_link" />
+  <axis
+    xyz="0 0 1" />
+  <limit
+    lower="-3.14"
+    upper="3.14"
+    effort="20000"
+    velocity="13" />
+  <dynamics damping="${joint_damping}" friction = "${joint_friction}"/>
+ </joint>
   <link
     name="base_link">
     <inertial>
-      <origin
-        xyz="-0.0746188127206768 -5.55111512312578E-17 -0.0854799809858157"
-        rpy="0 0 0" />
-      <mass
-        value="1.613834759363" />
-      <inertia
-        ixx="0"
-        ixy="0"
-        ixz="0"
-        iyy="0"
-        iyz="0"
-        izz="0" />
+      <origin xyz="-0.0746188127206768 -5.55111512312578E-17 -0.0854799809858157" rpy="0 0 0" />
+      <mass value="1.613834759363" />
+      <inertia ixx="0" ixy="0" ixz="0" iyy="0" iyz="0" izz="0" />
     </inertial>
     <visual>
-      <origin
-        xyz="0 0 0"
-        rpy="0 0 0" />
+      <origin xyz="0 0 0" rpy="0 0 0" />
       <geometry>
         <mesh
@@ -48,25 +58,8 @@
     </collision>
   </link>
-  <joint
-    name="dual_arm_base_joint"
-    type="revolute">
-    <origin
-      xyz="0 0 0.045"
-      rpy="${PI} 0 0" />
-    <parent
-      link="${robot_name}_link_7" />
-    <child
-      link="base_link" />
-    <axis
-      xyz="0 0 1" />
-    <limit
-      lower="-3.14"
-      upper="3.14"
-      effort="20000"
-      velocity="13" />
-    <dynamics damping="${joint_damping}" friction = "${joint_friction}"/>
-  </joint>
   <xacro:dual_arm_right robot_name="${robot_name}"/>
   <xacro:dual_arm_left robot_name="${robot_name}"/>
+  <xacro:gripper_R robot_name="$(arg robot_name)"/>
+  <xacro:gripper_L robot_name="$(arg robot_name)"/>
   </xacro:macro>
 </robot>

File: iiwa_description/urdf/complete_chain.urdf.xacro (robot description, xacro)
@@ -2,28 +2,14 @@
 <robot name="complete_chain" xmlns:xacro="http://www.ros.org/wiki/xacro">
 	<!-- Import all Gazebo-customization elements, including Gazebo colors -->
+	<xacro:include filename="$(find iiwa_description)/urdf/complete_chain.xacro" />
+	<xacro:include filename="$(find iiwa_description)/urdf/pulsating_surface.xacro" />
 	<xacro:include filename="$(find iiwa_description)/urdf/iiwa.gazebo.xacro" />
-	<!-- Import Transmissions -->
+	<xacro:include filename="$(find iiwa_description)/urdf/pulsating_surface.transmission.xacro" />
 	<xacro:include filename="$(find iiwa_description)/urdf/iiwa.transmission.xacro" />
-	<!-- Include Utilities -->
-	<xacro:include filename="$(find iiwa_description)/urdf/utilities.xacro" />
-	<!-- Include EOAT -->
-	<xacro:include filename="$(find iiwa_description)/urdf/iiwa14.xacro"/>
-	<xacro:include filename="$(find iiwa_description)/urdf/kuka_base_frame.xacro" />
-	<xacro:include filename="$(find iiwa_description)/urdf/Dual_Arm.xacro" />
-	<xacro:include filename="$(find iiwa_description)/urdf/pulsating_surface.xacro" />
-	<xacro:include filename="$(find iiwa_description)/urdf/gripper_eoat.xacro" />
-	<xacro:arg name="hardware_interface" default="EffortJointInterface"/>
-	<xacro:arg name="robot_name" default="iiwa"/>
-	<xacro:arg name="origin_xyz" default="0 0 0"/>
-	<xacro:arg name="origin_rpy" default="0 0 0"/>
-	<xacro:kuka_base_frame robot_name="$(arg robot_name)"/>
-	<xacro:iiwa14 hardware_interface="$(arg hardware_interface)" robot_name="$(arg robot_name)" parent="world">
-    	<origin xyz="$(arg origin_xyz)" rpy="$(arg origin_rpy)" />
-  	</xacro:iiwa14>
-  	<xacro:iiwa_gazebo robot_name="$(arg robot_name)"/>
-	<xacro:dual_arm_manipulator robot_name="$(arg robot_name)"/>
-	<xacro:gripper_eoat robot_name="$(arg robot_name)"/>
-	<xacro:pulsating_surface />
+	<xacro:pulsating_surface robot_name="$(arg robot_name)"/>
+	<xacro:complete_chain robot_name="$(arg robot_name)"/>
+	<!-- <xacro:pulsating_surface_gazebo robot_name="$(arg robot_name)"/> -->
 	<xacro:iiwa_gazebo robot_name="$(arg robot_name)"/>
 	<xacro:iiwa_transmission hardware_interface="$(arg hardware_interface)" robot_name="$(arg robot_name)"/>
+	<xacro:pulsating_surface_transmission hardware_interface="$(arg hardware_interface)" robot_name="$(arg robot_name)"/>
 </robot>

File: iiwa_description/urdf/dual_arm_left.xacro (robot description, xacro)
@@ -2,8 +2,27 @@
 <robot xmlns:xacro="http://www.ros.org/wiki/xacro">
   <xacro:property name="joint_friction" value="0.005" />
-  <xacro:property name="joint_damping" value="0.005" />
+  <xacro:property name="joint_damping" value="0.8" />
   <xacro:property name="PIhalf" value="1.570796" />
   <xacro:property name="PI" value="3.141592" />
   <xacro:macro name="dual_arm_left" params="robot_name">
+  <joint
+    name="J_L1"
+    type="revolute">
+    <origin
+      xyz="-0.0744445637977397 0.152871273073736 -0.110435575211296"
+      rpy="-1.43251148060093 -0.775712981728982 2.94539473140516" />
+    <parent
+      link="base_link" />
+    <child
+      link="Link_L1" />
+    <axis
+      xyz="0 0 1" />
+    <limit
+      lower="-3.14"
+      upper="3.14"
+      effort="20000"
+      velocity="13" />
+    <dynamics damping="${joint_damping}" friction = "${joint_friction}"/>
+  </joint>
   <link
     name="Link_L1">
@@ -13,5 +32,5 @@
         rpy="0 0 0" />
       <mass
-        value="0.323170961054133" />
+        value="0.523170961054133" />
       <inertia
         ixx="9.86315700006277E-05"
@@ -47,18 +66,18 @@
   </link>
   <joint
-    name="J_L1"
-    type="revolute">
-    <origin
-      xyz="-0.0744445637977397 0.152871273073736 -0.110435575211296"
-      rpy="-1.43251148060093 -0.775712981728982 2.94539473140516" />
-    <parent
-      link="base_link" />
-    <child
+    name="J_L2"
+    type="revolute">
+    <origin
+      xyz="0 0 -0.0635"
+      rpy="1.57079632679489 -0.380374098489847 0.317429885556193" />
+    <parent
       link="Link_L1" />
-    <axis
-      xyz="0 0 1" />
-    <limit
-      lower="-3.14"
-      upper="3.14"
+    <child
+      link="Link_L2" />
+    <axis
+      xyz="0 0 1" />
+    <limit
+      lower="-1.57"
+      upper="1.57"
       effort="20000"
       velocity="13" />
@@ -72,5 +91,5 @@
         rpy="0 0 0" />
       <mass
-        value="0.161073886022953" />
+        value="0.361073886022953" />
       <inertia
         ixx="1.38598083295319E-06"
@@ -106,30 +125,26 @@
   </link>
   <joint
-    name="J_L2"
-    type="revolute">
-    <origin
-      xyz="0 0 -0.0635"
-      rpy="1.57079632679489 -0.380374098489847 0.317429885556193" />
-    <parent
-      link="Link_L1" />
-    <child
+    name="J_L3"
+    type="revolute">
+    <origin
+      xyz="-0.178688999999999 -0.00012700000000021 0"
+      rpy="-1.57079632679489 -1.0547118733939E-15 1.5707963267949" />
+    <parent
       link="Link_L2" />
-    <axis
-      xyz="0 0 1" />
-    <limit
-      lower="-1.57"
-      upper="1.57"
-      effort="20000"
-      velocity="13" />
-    <dynamics damping="${joint_damping}" friction = "${joint_friction}"/>
-  </joint>
-  <link
-    name="Link_L3">
+    <child
+      link="Link_L3" />
+    <axis
+      xyz="0 0 1" />
+    <limit
+      lower="-3.14"
+      upper="3.14"
+      effort="20000"
+      velocity="13" />
+    <dynamics damping="${joint_damping}" friction = "${joint_friction}"/>
+  </joint>
+  <link name="Link_L3">
     <inertial>
-      <origin
-        xyz="0.00289722994622221 0.00112305403125196 0.0290055866352336"
-        rpy="0 0 0" />
-      <mass
-        value="0.117746913814738" />
+      <origin xyz="0.00289722994622221 0.00112305403125196 0.0290055866352336" rpy="0 0 0" />
+      <mass value="0.217746913814738" />
       <inertia
         ixx="9.95073774261661E-05"
@@ -141,4 +156,15 @@
     </inertial>
     <visual>
+      <origin xyz="0 0 0" rpy="0 0 0" />
+      <geometry>
+        <mesh filename="package://iiwa_description/meshes/iiwa14/collision/Dual_Arm/Link3.STL" />
+      </geometry>
+      <material
+        name="">
+        <color
+          rgba="1 1 1 1" />
+      </material>
+    </visual>
+    <collision>
       <origin
         xyz="0 0 0"
@@ -148,47 +174,33 @@
           filename="package://iiwa_description/meshes/iiwa14/collision/Dual_Arm/Link3.STL" />
       </geometry>
-      <material
-        name="">
-        <color
-          rgba="1 1 1 1" />
-      </material>
-    </visual>
-    <collision>
-      <origin
-        xyz="0 0 0"
-        rpy="0 0 0" />
-      <geometry>
-        <mesh
-          filename="package://iiwa_description/meshes/iiwa14/collision/Dual_Arm/Link3.STL" />
-      </geometry>
-    </collision>
-  </link>
-  <joint
-    name="J_L3"
-    type="revolute">
-    <origin
-      xyz="-0.178688999999999 -0.00012700000000021 0"
-      rpy="-1.57079632679489 -0.00547118733939 1.5707963267949" />
-    <parent
-      link="Link_L2" />
-    <child
+    </collision>
+  </link>
+  <joint
+    name="J_L4"
+    type="revolute">
+    <origin
+      xyz="0.0266700000000004 0.0019050000000066 0.0609600000000012"
+      rpy="-1.5707963267949 -0.824186362211141 -1.57079632679489" />
+    <parent
       link="Link_L3" />
-    <axis
-      xyz="0 0 1" />
-    <limit
-      lower="-3.14"
-      upper="3.14"
-      effort="20000"
-      velocity="13" />
-    <dynamics damping="${joint_damping}" friction = "${joint_friction}"/>
-  </joint>
-  <link
+    <child
+      link="Link_L4" />
+    <axis
+      xyz="0 0 1" />
+    <limit
+      lower="-1.57"
+      upper="1.57"
+      effort="20000"
+      velocity="13" />
+    <dynamics damping="${joint_damping}" friction = "${joint_friction}"/>
+  </joint>
+ <link
     name="Link_L4">
-    <inertial>
+      <inertial>
       <origin
         xyz="-0.00106966507570738 -0.0713978397746767 -0.00106966507570611"
         rpy="0 0 0" />
       <mass
-        value="0.117746913814738" />
+        value="0.217746913814738" />
       <inertia
         ixx="9.95073774261661E-05"
@@ -223,23 +235,4 @@
     </collision>
   </link>
-  <joint
-    name="J_L4"
-    type="revolute">
-    <origin
-      xyz="0.0266700000000004 0.0019050000000066 0.0609600000000012"
-      rpy="-1.5707963267949 -0.824186362211141 -1.57079632679489" />
-    <parent
-      link="Link_L3" />
-    <child
-      link="Link_L4" />
-    <axis
-      xyz="0 0 1" />
-    <limit
-      lower="-1.57"
-      upper="1.57"
-      effort="20000"
-      velocity="13" />
-    <dynamics damping="${joint_damping}" friction = "${joint_friction}"/>
-  </joint>
   </xacro:macro>
 </robot>

File: iiwa_description/urdf/dual_arm_right.xacro (robot description, xacro)
@@ -2,8 +2,27 @@
 <robot xmlns:xacro="http://www.ros.org/wiki/xacro">
   <xacro:property name="joint_friction" value="0.005" />
-  <xacro:property name="joint_damping" value="0.005" />
+  <xacro:property name="joint_damping" value="0.8" />
   <xacro:property name="PIhalf" value="1.570796" />
   <xacro:property name="PI" value="3.141592" />
   <xacro:macro name="dual_arm_right" params="robot_name">
+  <joint
+    name="J_R1"
+    type="revolute">
+    <origin
+      xyz="-0.0744445637977397 -0.152871273073736 -0.110435575211296"
+      rpy="1.43251148060093 -0.775712981728982 -2.94539473140516" />
+    <parent
+      link="base_link" />
+    <child
+      link="Link_R1" />
+    <axis
+      xyz="0 0 1" />
+    <limit
+      lower="-3.14"
+      upper="3.14"
+      effort="20000"
+      velocity="13" />
+    <dynamics damping="${joint_damping}" friction = "${joint_friction}"/>
+ </joint>
   <link
     name="Link_R1">
@@ -13,5 +32,5 @@
         rpy="0 0 0" />
       <mass
-        value="0.323170961054133" />
+        value="0.523170961054133" />
       <inertia
         ixx="9.86315700006277E-05"
@@ -47,23 +66,23 @@
   </link>
   <joint
-    name="J_R1"
-    type="revolute">
-    <origin
-      xyz="-0.0744445637977397 -0.152871273073736 -0.110435575211296"
-      rpy="1.43251148060093 -0.775712981728982 -2.94539473140516" />
-    <parent
-      link="base_link" />
-    <child
+    name="J_R2"
+    type="revolute">
+    <origin
+      xyz="0 0 -0.0635"
+      rpy="1.57079632679489 -0.380374098489847 0.317429885556193" />
+    <parent
       link="Link_R1" />
-    <axis
-      xyz="0 0 1" />
-    <limit
-      lower="-3.14"
-      upper="3.14"
-      effort="20000"
-      velocity="13" />
-    <dynamics damping="${joint_damping}" friction = "${joint_friction}"/>
- </joint>
-  <link
+    <child
+      link="Link_R2" />
+    <axis
+      xyz="0 0 1" />
+    <limit
+      lower="-1.57"
+      upper="1.57"
+      effort="20000"
+      velocity="13" />
+    <dynamics damping="${joint_damping}" friction = "${joint_friction}"/>
+  </joint>
+<link
     name="Link_R2">
     <inertial>
@@ -72,5 +91,5 @@
         rpy="0 0 0" />
       <mass
-        value="0.161073886022953" />
+        value="0.361073886022953" />
       <inertia
         ixx="1.38598083295319E-06"
@@ -106,18 +125,18 @@
   </link>
   <joint
-    name="J_R2"
-    type="revolute">
-    <origin
-      xyz="0 0 -0.0635"
-      rpy="1.57079632679489 -0.380374098489847 0.317429885556193" />
-    <parent
-      link="Link_R1" />
-    <child
+    name="J_R3"
+    type="revolute">
+    <origin
+      xyz="-0.178688999999999 -0.00012700000000021 0"
+      rpy="-1.57079632679489 -1.0547118733939E-15 1.5707963267949" />
+    <parent
       link="Link_R2" />
-    <axis
-      xyz="0 0 1" />
-    <limit
-      lower="-1.57"
-      upper="1.57"
+    <child
+      link="Link_R3" />
+    <axis
+      xyz="0 0 1" />
+    <limit
+      lower="-3.14"
+      upper="3.14"
       effort="20000"
       velocity="13" />
@@ -131,5 +150,5 @@
         rpy="0 0 0" />
       <mass
-        value="0.117746913814738" />
+        value="0.217746913814738" />
       <inertia
         ixx="9.95073774261661E-05"
@@ -165,23 +184,23 @@
   </link>
   <joint
-    name="J_R3"
-    type="revolute">
-    <origin
-      xyz="-0.178688999999999 -0.00012700000000021 0"
-      rpy="-1.57079632679489 -1.0547118733939E-15 1.5707963267949" />
-    <parent
-      link="Link_R2" />
-    <child
+    name="J_R4"
+    type="revolute">
+    <origin
+      xyz="0.0266700000000004 0.0019050000000066 0.0609600000000012"
+      rpy="-1.5707963267949 -0.824186362211141 -1.57079632679489" />
+    <parent
       link="Link_R3" />
-    <axis
-      xyz="0 0 1" />
-    <limit
-      lower="-3.14"
-      upper="3.14"
+    <child
+      link="Link_R4" />
+    <axis
+      xyz="0 0 1" />
+    <limit
+      lower="-1.57"
+      upper="1.57"
       effort="20000"
       velocity="13" />
     <dynamics damping="${joint_damping}" friction = "${joint_friction}"/>
   </joint>
-  <link
+ <link
     name="Link_R4">
       <inertial>
@@ -190,5 +209,5 @@
         rpy="0 0 0" />
       <mass
-        value="0.117746913814738" />
+        value="0.217746913814738" />
       <inertia
         ixx="9.95073774261661E-05"
@@ -223,23 +242,4 @@
     </collision>
   </link>
-  <joint
-    name="J_R4"
-    type="revolute">
-    <origin
-      xyz="0.0266700000000004 0.0019050000000066 0.0609600000000012"
-      rpy="-1.5707963267949 -0.824186362211141 -1.57079632679489" />
-    <parent
-      link="Link_R3" />
-    <child
-      link="Link_R4" />
-    <axis
-      xyz="0 0 1" />
-    <limit
-      lower="-1.57"
-      upper="1.57"
-      effort="20000"
-      velocity="13" />
-    <dynamics damping="${joint_damping}" friction = "${joint_friction}"/>
-  </joint>
   </xacro:macro>
 </robot>

File: iiwa_description/urdf/iiwa.gazebo.xacro (robot description, xacro)
@@ -31,5 +31,5 @@
     <!--Frame-->
     <gazebo reference="frame">
-      <material>Gazebo/Orange</material>
+      <material>Gazebo/Grey</material>
       <mu1>0.2</mu1>
       <mu2>0.2</mu2>
@@ -98,47 +98,47 @@
       <selfCollide>0</selfCollide>
     </gazebo>
-    <gazebo reference="Link1">
-      <material>Gazebo/White</material>
-      <mu1>0.2</mu1>
-      <mu2>0.2</mu2>
-      <selfCollide>0</selfCollide>
-    </gazebo>
-    <gazebo reference="Link2">
-      <material>Gazebo/Red</material>
-      <mu1>0.2</mu1>
-      <mu2>0.2</mu2>
-      <selfCollide>0</selfCollide>
-    </gazebo>
-    <gazebo reference="Link3">
-      <material>Gazebo/White</material>
-      <mu1>0.2</mu1>
-      <mu2>0.2</mu2>
-      <selfCollide>0</selfCollide>
-    </gazebo>
-    <gazebo reference="Link4">
-      <material>Gazebo/Red</material>
-      <mu1>0.2</mu1>
-      <mu2>0.2</mu2>
-      <selfCollide>0</selfCollide>
-    </gazebo>
-    <gazebo reference="L2_1">
-      <material>Gazebo/White</material>
-      <mu1>0.2</mu1>
-      <mu2>0.2</mu2>
-      <selfCollide>0</selfCollide>
-    </gazebo>
-    <gazebo reference="L2_2">
-      <material>Gazebo/Red</material>
-      <mu1>0.2</mu1>
-      <mu2>0.2</mu2>
-      <selfCollide>0</selfCollide>
-    </gazebo>
-    <gazebo reference="L2_3">
-      <material>Gazebo/White</material>
-      <mu1>0.2</mu1>
-      <mu2>0.2</mu2>
-      <selfCollide>0</selfCollide>
-    </gazebo>
-    <gazebo reference="L2_4">
+    <gazebo reference="Link_L1">
+      <material>Gazebo/White</material>
+      <mu1>0.2</mu1>
+      <mu2>0.2</mu2>
+      <selfCollide>0</selfCollide>
+    </gazebo>
+    <gazebo reference="Link_L2">
+      <material>Gazebo/Red</material>
+      <mu1>0.2</mu1>
+      <mu2>0.2</mu2>
+      <selfCollide>0</selfCollide>
+    </gazebo>
+    <gazebo reference="Link_L3">
+      <material>Gazebo/White</material>
+      <mu1>0.2</mu1>
+      <mu2>0.2</mu2>
+      <selfCollide>0</selfCollide>
+    </gazebo>
+    <gazebo reference="Link_L4">
+      <material>Gazebo/Red</material>
+      <mu1>0.2</mu1>
+      <mu2>0.2</mu2>
+      <selfCollide>0</selfCollide>
+    </gazebo>
+    <gazebo reference="Link_R1">
+      <material>Gazebo/White</material>
+      <mu1>0.2</mu1>
+      <mu2>0.2</mu2>
+      <selfCollide>0</selfCollide>
+    </gazebo>
+    <gazebo reference="Link_R2">
+      <material>Gazebo/Red</material>
+      <mu1>0.2</mu1>
+      <mu2>0.2</mu2>
+      <selfCollide>0</selfCollide>
+    </gazebo>
+    <gazebo reference="Link_R3">
+      <material>Gazebo/White</material>
+      <mu1>0.2</mu1>
+      <mu2>0.2</mu2>
+      <selfCollide>0</selfCollide>
+    </gazebo>
+    <gazebo reference="Link_R4">
       <material>Gazebo/Red</material>
       <mu1>0.2</mu1>
@@ -164,17 +164,17 @@
       <selfCollide>0</selfCollide>
     </gazebo>
-    <gazebo reference="2_gripper_base_link">
-      <material>Gazebo/White</material>
-      <mu1>0.2</mu1>
-      <mu2>0.2</mu2>
-      <selfCollide>0</selfCollide>
-    </gazebo>
-    <gazebo reference="2_claw_1_link">
-      <material>Gazebo/Red</material>
-      <mu1>0.2</mu1>
-      <mu2>0.2</mu2>
-      <selfCollide>0</selfCollide>
-    </gazebo>
-    <gazebo reference="2_claw_2_link">
+    <gazebo reference="gripper_base_link_2">
+      <material>Gazebo/White</material>
+      <mu1>0.2</mu1>
+      <mu2>0.2</mu2>
+      <selfCollide>0</selfCollide>
+    </gazebo>
+    <gazebo reference="claw_1_link_2">
+      <material>Gazebo/Red</material>
+      <mu1>0.2</mu1>
+      <mu2>0.2</mu2>
+      <selfCollide>0</selfCollide>
+    </gazebo>
+    <gazebo reference="claw_2_link_2">
       <material>Gazebo/Red</material>
       <mu1>0.2</mu1>
@@ -244,11 +244,11 @@
       <selfCollide>0</selfCollide>
     </gazebo>
-    <gazebo reference="surface">
-      <material>Gazebo/Orange</material>
+    <gazebo reference="table_surface">
+      <material>Gazebo/WhiteEmissive</material>
       <mu1>0.2</mu1>
       <mu2>0.2</mu2>
       <kd>2500</kd>
       <kp>10000</kp>
-      <selfCollide>0</selfCollide>
+      <selfCollide>1</selfCollide>
     </gazebo>
   </xacro:macro>
