Commit message: completed model works in melodic, changed the structure of the tree

File: iiwa_description/urdf/iiwa.transmission.xacro (robot description, xacro)
@@ -6,5 +6,5 @@
       <type>transmission_interface/SimpleTransmission</type>
       <joint name="${robot_name}_joint_1">
-	<hardwareInterface>hardware_interface/PositionJointInterface</hardwareInterface>
+	<hardwareInterface>hardware_interface/${hardware_interface}</hardwareInterface>
       </joint>
       <actuator name="${robot_name}_motor_1">
@@ -16,5 +16,5 @@
       <type>transmission_interface/SimpleTransmission</type>
       <joint name="${robot_name}_joint_2">
-	    <hardwareInterface>hardware_interface/PositionJointInterface</hardwareInterface>
+	    <hardwareInterface>hardware_interface/${hardware_interface}</hardwareInterface>
       </joint>
       <actuator name="${robot_name}_motor_2">
@@ -26,8 +26,7 @@
       <type>transmission_interface/SimpleTransmission</type>
       <joint name="${robot_name}_joint_3">
-	    <hardwareInterface>hardware_interface/PositionJointInterface</hardwareInterface>
+	    <hardwareInterface>hardware_interface/${hardware_interface}</hardwareInterface>
       </joint>
       <actuator name="${robot_name}_motor_3">
-        <hardwareInterface>hardware_interface/PositionJointInterface</hardwareInterface>
 	<mechanicalReduction>1</mechanicalReduction>
       </actuator>
@@ -37,5 +36,5 @@
       <type>transmission_interface/SimpleTransmission</type>
       <joint name="${robot_name}_joint_4">
-	    <hardwareInterface>hardware_interface/PositionJointInterface</hardwareInterface>
+	    <hardwareInterface>hardware_interface/${hardware_interface}</hardwareInterface>
       </joint>
       <actuator name="${robot_name}_motor_4">
@@ -47,5 +46,5 @@
       <type>transmission_interface/SimpleTransmission</type>
       <joint name="${robot_name}_joint_5">
-	    <hardwareInterface>hardware_interface/PositionJointInterface</hardwareInterface>
+	    <hardwareInterface>hardware_interface/${hardware_interface}</hardwareInterface>
       </joint>
       <actuator name="${robot_name}_motor_5">
@@ -57,5 +56,5 @@
       <type>transmission_interface/SimpleTransmission</type>
       <joint name="${robot_name}_joint_6">
-	    <hardwareInterface>hardware_interface/PositionJointInterface</hardwareInterface>
+	    <hardwareInterface>hardware_interface/${hardware_interface}</hardwareInterface>
       </joint>
       <actuator name="${robot_name}_motor_6">
@@ -67,5 +66,5 @@
       <type>transmission_interface/SimpleTransmission</type>
       <joint name="${robot_name}_joint_7">
-	    <hardwareInterface>hardware_interface/PositionJointInterface</hardwareInterface>
+	    <hardwareInterface>hardware_interface/${hardware_interface}</hardwareInterface>
       </joint>
       <actuator name="${robot_name}_motor_7">
@@ -73,15 +72,5 @@
       </actuator>
     </transmission>
-<transmission name="manipulator_tran_1">
-      <robotNamespace>/${robot_name}</robotNamespace>
-      <type>transmission_interface/SimpleTransmission</type>
-      <joint name="dual_arm_base_joint">
-      <hardwareInterface>hardware_interface/${hardware_interface}</hardwareInterface>
-      </joint>
-      <actuator name="dual_arm_base_motor">
-  <mechanicalReduction>1</mechanicalReduction>
-      </actuator>
-    </transmission>
-    <transmission name="J_1_tran">
+    <transmission name="J_L1_trans">
       <robotNamespace>/${robot_name}</robotNamespace>
       <type>transmission_interface/SimpleTransmission</type>
@@ -89,9 +78,9 @@
       <hardwareInterface>hardware_interface/${hardware_interface}</hardwareInterface>
       </joint>
-      <actuator name="J_1_motor">
-  <mechanicalReduction>1</mechanicalReduction>
-      </actuator>
-    </transmission>
-    <transmission name="J_2_tran">
+      <actuator name="J_L1_motor">
+  <mechanicalReduction>1</mechanicalReduction>
+      </actuator>
+    </transmission>
+    <transmission name="J_L2_tran">
       <robotNamespace>/${robot_name}</robotNamespace>
       <type>transmission_interface/SimpleTransmission</type>
@@ -99,9 +88,9 @@
   <hardwareInterface>hardware_interface/${hardware_interface}</hardwareInterface>
       </joint>
-      <actuator name="J_2_motor">
-  <mechanicalReduction>1</mechanicalReduction>
-      </actuator>
-    </transmission>
-<transmission name="J_3_tran">
+      <actuator name="J_L2_motor">
+  <mechanicalReduction>1</mechanicalReduction>
+      </actuator>
+    </transmission>
+<transmission name="J_L3_tran">
       <robotNamespace>/${robot_name}</robotNamespace>
       <type>transmission_interface/SimpleTransmission</type>
@@ -109,9 +98,9 @@
   <hardwareInterface>hardware_interface/${hardware_interface}</hardwareInterface>
       </joint>
-      <actuator name="J_3_motor">
-  <mechanicalReduction>1</mechanicalReduction>
-      </actuator>
-    </transmission>
-    <transmission name="J_4_tran">
+      <actuator name="J_L3_motor">
+  <mechanicalReduction>1</mechanicalReduction>
+      </actuator>
+    </transmission>
+    <transmission name="J_L4_tran">
       <robotNamespace>/${robot_name}</robotNamespace>
       <type>transmission_interface/SimpleTransmission</type>
@@ -119,9 +108,9 @@
   <hardwareInterface>hardware_interface/${hardware_interface}</hardwareInterface>
       </joint>
-      <actuator name="J_4_motor">
-  <mechanicalReduction>1</mechanicalReduction>
-      </actuator>
-    </transmission>
-  <transmission name="J_21_tran">
+      <actuator name="J_L4_motor">
+  <mechanicalReduction>1</mechanicalReduction>
+      </actuator>
+    </transmission>
+  <transmission name="J_R1_tran">
       <robotNamespace>/${robot_name}</robotNamespace>
       <type>transmission_interface/SimpleTransmission</type>
@@ -133,5 +122,5 @@
       </actuator>
     </transmission>
-  <transmission name="J_22_tran">
+  <transmission name="J_R2_tran">
       <robotNamespace>/${robot_name}</robotNamespace>
       <type>transmission_interface/SimpleTransmission</type>
@@ -143,5 +132,5 @@
       </actuator>
     </transmission>
-  <transmission name="J_23_tran">
+  <transmission name="J_R3_tran">
       <robotNamespace>/${robot_name}</robotNamespace>
       <type>transmission_interface/SimpleTransmission</type>
@@ -153,5 +142,5 @@
       </actuator>
     </transmission>
-  <transmission name="J_24_tran">
+  <transmission name="J_R4_tran">
       <robotNamespace>/${robot_name}</robotNamespace>
       <type>transmission_interface/SimpleTransmission</type>
@@ -172,5 +161,5 @@
   <mechanicalReduction>1</mechanicalReduction>
       </actuator>
-    </transmission>
+  </transmission>
   <transmission name="claw_1_joint_tran">
       <robotNamespace>/${robot_name}</robotNamespace>
@@ -193,38 +182,39 @@
       </actuator>
     </transmission>
-  <transmission name="2_gripper_base_joint_tran">
-      <robotNamespace>/${robot_name}</robotNamespace>
-      <type>transmission_interface/SimpleTransmission</type>
-      <joint name="2_gripper_base_joint">
-  <hardwareInterface>hardware_interface/${hardware_interface}</hardwareInterface>
-      </joint>
-      <actuator name="2_gripper_base_joint_motor">
-  <mechanicalReduction>1</mechanicalReduction>
-      </actuator>
-    </transmission>
-  <transmission name="2_claw_1_joint_tran">
-      <robotNamespace>/${robot_name}</robotNamespace>
-      <type>transmission_interface/SimpleTransmission</type>
-      <joint name="2_claw_1_joint">
-  <hardwareInterface>hardware_interface/${hardware_interface}</hardwareInterface>
-      </joint>
-      <actuator name="2_claw_1_motor">
-  <mechanicalReduction>1</mechanicalReduction>
-      </actuator>
-    </transmission>
-  <transmission name="2_claw_2_joint_tran">
-      <robotNamespace>/${robot_name}</robotNamespace>
-      <type>transmission_interface/SimpleTransmission</type>
-      <joint name="2_claw_2_joint">
-  <hardwareInterface>hardware_interface/${hardware_interface}</hardwareInterface>
-      </joint>
-      <actuator name="2_claw_2_motor">
-  <mechanicalReduction>1</mechanicalReduction>
-      </actuator>
-    </transmission>
+  <transmission name="gripper_base_joint_tran_2">
+      <robotNamespace>/${robot_name}</robotNamespace>
+      <type>transmission_interface/SimpleTransmission</type>
+      <joint name="gripper_base_joint_2">
+  <hardwareInterface>hardware_interface/${hardware_interface}</hardwareInterface>
+      </joint>
+      <actuator name="gripper_base_joint_motor_2">
+  <mechanicalReduction>1</mechanicalReduction>
+      </actuator>
+    </transmission>
+  <transmission name="claw_1_joint_tran_2">
+      <robotNamespace>/${robot_name}</robotNamespace>
+      <type>transmission_interface/SimpleTransmission</type>
+      <joint name="claw_1_joint_2">
+  <hardwareInterface>hardware_interface/${hardware_interface}</hardwareInterface>
+      </joint>
+      <actuator name="claw_1_motor_2">
+  <mechanicalReduction>1</mechanicalReduction>
+      </actuator>
+    </transmission>
+  <transmission name="claw_2_joint_tran_2">
+      <robotNamespace>/${robot_name}</robotNamespace>
+      <type>transmission_interface/SimpleTransmission</type>
+      <joint name="claw_2_joint_2">
+  <hardwareInterface>hardware_interface/${hardware_interface}</hardwareInterface>
+      </joint>
+      <actuator name="claw_2_motor_2">
+  <mechanicalReduction>1</mechanicalReduction>
+      </actuator>
+    </transmission>
+<!--
   <transmission name="pulsating_surface_tran_1">
       <robotNamespace>/${robot_name}</robotNamespace>
       <type>transmission_interface/SimpleTransmission</type>
-      <joint name="prismatic_joint">
+      <joint name="table_joint">
   <hardwareInterface>hardware_interface/${hardware_interface}</hardwareInterface>
       </joint>
@@ -232,5 +222,5 @@
   <mechanicalReduction>1</mechanicalReduction>
       </actuator>
-    </transmission>
+    </transmission> -->
   </xacro:macro>
 </robot>

File: iiwa_description/urdf/iiwa14.xacro (robot description, xacro)
@@ -9,5 +9,5 @@
   <xacro:property name="max_velocity" value="100"/>
   <xacro:property name="joint_friction" value="0.005" />
-  <xacro:property name="joint_damping" value="0.005" />
+  <xacro:property name="joint_damping" value="0.5" />
   <xacro:property name="PIhalf" value="1.570796" />
   <xacro:property name="PI" value="3.141592" />

File: iiwa_description/urdf/kuka_base_frame.xacro (robot description, xacro)
@@ -7,53 +7,63 @@
   <xacro:macro name="kuka_base_frame" params="robot_name">
   <link name="world" />
-  <joint
-    name="fixed"
-    type="fixed">
-    <parent
-      link="world" />
-    <child
-      link="frame" />
+  <joint name="fixed_frame_joint" type="fixed">
+    <parent link="world" />
+    <child link="frame_kuka" />
     <axis xyz="0 0 1"/>
   </joint>
-  <link
-    name="frame">
+  <link name="frame_kuka">
     <inertial>
-      <origin
-        xyz="1.5 0.25 1.25"
-        rpy="0 0 0" />
-      <mass
-        value="2697" />
-      <inertia
-        ixx="0"
-        ixy="0"
-        ixz="0"
-        iyy="0"
-        iyz="0"
-        izz="0" />
+      <origin xyz="1.5 0.25 1.25" rpy="0 0 0" />
+      <mass value="2697" />
+      <inertia ixx="0" ixy="0" ixz="0" iyy="0" iyz="0" izz="0" />
     </inertial>
     <visual>
-      <origin
-        xyz="0 0 0"
-        rpy="0 0 0" />
+      <origin xyz="0 0 0" rpy="0 0 0" />
       <geometry>
-        <mesh
-          filename="package://iiwa_description/meshes/iiwa14/visual/base_link.STL"/>
+        <mesh filename="package://iiwa_description/meshes/iiwa14/visual/base_link.STL"/>
       </geometry>
       <material
         name="">
-        <color
-          rgba="0.64706 0.61961 0.58824 1" />
+        <color rgba="0.64706 0.61961 0.58824 1" />
       </material>
     </visual>
     <collision>
-      <origin
-        xyz="0 0 0"
-        rpy="0 0 0" />
+      <origin xyz="0 0 0" rpy="0 0 0" />
       <geometry>
-        <mesh
-          filename="package://iiwa_description/meshes/iiwa14/collision/base_link.STL" />
+        <mesh filename="package://iiwa_description/meshes/iiwa14/collision/base_link.STL" />
       </geometry>
     </collision>
   </link>
+    <!-- joint between post and surface -->
+  <!-- joint name="table_joint" type="prismatic">
+    <parent link="world"/>
+    <child link="surface_table"/>
+    <origin xyz="1.5 15 0.10" rpy="0 0 1.5707"/>
+    <axis xyz="0 0 1"/>
+    <limit lower="-0.8" upper="0.3"
+           effort="10000" velocity="10000" />
+    <dynamics damping="0.5" friction = "0.1"/>
+  </joint>
+  <link name="surface_table">
+    <inertial>
+      <origin xyz="0 0 0.0015" rpy="0 0 0"/>
+      <mass value="3.645"/>
+      <inertia ixx="0.0276"  ixy="0"  ixz="0" iyy="0.00711" iyz="0" izz="0.03417" />
+    </inertial>
+    <visual>
+      <origin xyz="0 0 0" rpy="0 0 0"/>
+      <geometry>
+        <mesh filename="package://iiwa_description/meshes/iiwa14/collision/Pulsating Surface/Surface.STL"/>
+      </geometry>
+      <material name="Grey"/>
+    </visual>
+    <collision>
+      <origin xyz="0 0 0" rpy="0 0 0"/>
+      <geometry>
+        <mesh filename="package://iiwa_description/meshes/iiwa14/collision/Pulsating Surface/Surface.STL"/>
+      </geometry>
+      <material name="Grey"/>
+    </collision>
+  </link> -->
   </xacro:macro>
 </robot>

File: iiwa_description/urdf/pulsating_surface.gazebo.xacro (robot description, xacro)
@@ -1,10 +1,10 @@
 <?xml version="1.0"?>
 <robot xmlns:xacro="http://www.ros.org/wiki/xacro">
-  <xacro:macro name="pulsating_surface_gazebo">
-  	<gazebo>
+  <xacro:macro name="pulsating_surface_gazebo" params="robot_name">
+<!--   	<gazebo>
       <plugin name="gazebo_ros_control" filename="libgazebo_ros_control.so">
         <robotNamespace>/${robot_name}</robotNamespace>
       </plugin>
-    </gazebo>
+    </gazebo> -->
     <gazebo reference="post">
       <material>Gazebo/White</material>
@@ -13,5 +13,5 @@
     </gazebo>
     <gazebo reference="surface">
-      <material>Gazebo/Orange</material>
+      <material>Gazebo/Black</material>
       <mu1>0.2</mu1>
       <mu2>0.2</mu2>

File: iiwa_description/urdf/pulsating_surface.transmission.xacro (robot description, xacro)
@@ -1,16 +1,15 @@
 <?xml version="1.0"?>
 <robot xmlns:xacro="http://www.ros.org/wiki/xacro">
-	<xacro:macro name="pulsating_surface_transmission" params = "hardware_interface">
-<transmission name="pulsating_surface_tran_1">
+	<xacro:macro name="pulsating_surface_transmission" params = "hardware_interface robot_name">
+  <transmission name="pulsating_surface_tran_1">
       <robotNamespace>/pulsating_surface</robotNamespace>
       <type>transmission_interface/SimpleTransmission</type>
-      <joint name="prismatic_joint">
-	<hardwareInterface>${hardware_interface}</hardwareInterface>
-      </joint>
-      <actuator name="pulsating_surface_motor_1">
-	<hardwareInterface>${hardware_interface}</hardwareInterface>
-	<mechanicalReduction>1</mechanicalReduction>
-      </actuator>
-    </transmission>
-</xacro:macro>
+  <joint name="table_joint">
+	 <hardwareInterface>hardware_interface/${hardware_interface}</hardwareInterface>
+  </joint>
+  <actuator name="pulsating_surface_motor_1">
+	 <mechanicalReduction>1</mechanicalReduction>
+  </actuator>
+  </transmission>
+  </xacro:macro>
 </robot>

File: iiwa_description/urdf/pulsating_surface.xacro (robot description, xacro)
@@ -1,20 +1,20 @@
 <?xml version="1.0"?>
 <robot xmlns:xacro="http://www.ros.org/wiki/xacro">
-<xacro:macro name = "pulsating_surface" >
+  <xacro:macro name = "pulsating_surface" params="robot_name">
     <!-- joint between post and surface -->
-    <joint name="prismatic_joint" type="prismatic">
+    <joint name="table_joint" type="revolute">
       <parent link="world"/>
-      <child link="surface"/>
-      <origin xyz="1.5 0.25 0" rpy="0 0 1.5707"/>
+      <child link="table_surface"/>
+      <origin xyz="1.5 0.25 0.15" rpy="0 0 1.5707"/>
       <axis xyz="0 0 1"/>
       <limit lower="-0.8" upper="0.3"
              effort="10000" velocity="10000" />
-      <dynamics damping="1" friction = "1"/>
+      <dynamics damping="0.5" friction = "0.1"/>
     </joint>
-    <link name="surface">
+    <link name="table_surface">
       <inertial>
-        <origin xyz="0 0 0.0015" rpy="0 0 0"/>
-        <mass value="3.645"/>
-        <inertia ixx="0.0276"  ixy="0"  ixz="0" iyy="0.00711" iyz="0" izz="0.03417" />
+        <origin xyz="0 0 0" rpy="0 0 0"/>
+        <mass value="0.645"/>
+        <inertia ixx="0.0276" ixy="0" ixz="0" iyy="0.00711" iyz="0" izz="0.03417" />
       </inertial>
       <visual>
@@ -23,5 +23,8 @@
           <mesh filename="package://iiwa_description/meshes/iiwa14/collision/Pulsating Surface/Surface.STL"/>
         </geometry>
-        <material name="Grey"/>
+        <material
+          name="">
+          <color rgba="0.64706 0.61961 0.58824 1" />
+        </material>
       </visual>
       <collision>
@@ -33,4 +36,4 @@
       </collision>
     </link>
-</xacro:macro>
+  </xacro:macro>
 </robot>
