Commit message: renamed sim scripts folder

File: iiwa_description/urdf/force_control_platform/iiwa.gazebo.xacro (robot description, xacro)
@@ -245,5 +245,5 @@
     </gazebo>
 -->
-    <gazebo reference="post">
+  <!--   <gazebo reference="post">
       <material>Gazebo/White</material>
       <mu1>0.2</mu1>
@@ -259,4 +259,5 @@
       <selfCollide>1</selfCollide>
     </gazebo>
+ -->
   </xacro:macro>
 </robot>

File: iiwa_description/urdf/force_control_platform/kuka_pulsating_surface.urdf.xacro (robot description, xacro)
@@ -4,4 +4,5 @@
 	<xacro:include filename="$(find iiwa_description)/urdf/force_control_platform/pulsating_surface.xacro" />
 	<xacro:include filename="$(find iiwa_description)/urdf/force_control_platform/iiwa.gazebo.xacro" />
+	<xacro:include filename="$(find iiwa_description)/urdf/force_control_platform/pulsating_surface.gazebo.xacro" />
 	<!-- Import Transmissions -->
 	<xacro:include filename="$(find iiwa_description)/urdf/force_control_platform/pulsating_surface.transmission.xacro" />
@@ -14,3 +15,4 @@
 	<xacro:pulsating_surface_transmission hardware_interface="$(arg hardware_interface)" robot_name="$(arg robot_name)"/>
 	<xacro:pulsating_surface robot_name="$(arg robot_name)"/>
+	<xacro:pulsating_surface_gazebo robot_name="$(arg robot_name)"/>
 </robot>

File: iiwa_description/urdf/force_control_platform/kuka_pulsating_surface.xacro (robot description, xacro)
@@ -4,5 +4,4 @@
 	<!-- Import all Gazebo-customization elements, including Gazebo colors -->
 	<xacro:include filename="$(find iiwa_description)/urdf/iiwa.gazebo.xacro" />
-	<xacro:include filename="$(find iiwa_description)/urdf/force_control_platform/pulsating_surface.gazebo.xacro" />
 	<!-- Import Transmissions -->
 	<xacro:include filename="$(find iiwa_description)/urdf/iiwa.transmission.xacro" />

File: iiwa_description/urdf/force_control_platform/pulsating_surface.gazebo.xacro (robot description, xacro)
@@ -12,8 +12,12 @@
       <mu2>0.2</mu2>
     </gazebo>
-    <gazebo reference="surface">
-      <material>Gazebo/Black</material>
-      <mu1>0.2</mu1>
-      <mu2>0.2</mu2>
+    <gazebo reference="table_surface">
+      <material>Gazebo/WoodPallet</material>
+      <turnGravityOff>true</turnGravityOff>
+      <mu1>0.5</mu1>
+      <mu2>0.5</mu2>
+      <kd>20</kd>
+      <kp>0.1</kp>
+      <selfCollide>1</selfCollide>
     </gazebo>
   </xacro:macro>

File: iiwa_description/urdf/force_control_platform/pulsating_surface.transmission.xacro (robot description, xacro)
@@ -3,6 +3,6 @@
 	<xacro:macro name="pulsating_surface_transmission" params = "hardware_interface robot_name">
   <transmission name="pulsating_surface_tran_1">
-      <robotNamespace>/pulsating_surface</robotNamespace>
-      <type>transmission_interface/SimpleTransmission</type>
+      <robotNamespace>/${robot_name}</robotNamespace>
+  <type>transmission_interface/SimpleTransmission</type>
   <joint name="table_joint">
 	 <hardwareInterface>hardware_interface/${hardware_interface}</hardwareInterface>
@@ -12,4 +12,14 @@
   </actuator>
   </transmission>
+  <transmission name="pulsating_surface_tran_2">
+      <robotNamespace>/${robot_name}</robotNamespace>
+      <type>transmission_interface/SimpleTransmission</type>
+  <joint name="table_joint_tilt">
+   <hardwareInterface>hardware_interface/${hardware_interface}</hardwareInterface>
+  </joint>
+  <actuator name="pulsating_surface_motor_2">
+   <mechanicalReduction>1</mechanicalReduction>
+  </actuator>
+  </transmission>
   </xacro:macro>
 </robot>

File: iiwa_description/urdf/force_control_platform/pulsating_surface.xacro (robot description, xacro)
@@ -3,7 +3,7 @@
   <xacro:macro name = "pulsating_surface" params="robot_name">
     <!-- joint between post and surface -->
-    <joint name="table_joint" type="revolute">
+    <joint name="table_joint" type="prismatic">
       <parent link="world"/>
-      <child link="table_surface"/>
+      <child link="table_surface_interface"/>
       <origin xyz="1.5 0.25 0.15" rpy="0 0 1.5707"/>
       <axis xyz="0 0 1"/>
@@ -35,5 +35,64 @@
         <material name="Grey"/>
       </collision>
+      <surface>
+        <friction>
+          <ode>
+            <mu>0.5</mu>
+            <mu2>0.5</mu2>
+          </ode>
+        </friction>
+        <bounce>
+          <restitution_coefficient>0.01</restitution_coefficient>
+          <threshold>0.01</threshold>
+        </bounce>
+        <contact>
+          <ode>
+            <max_vel>0.1</max_vel>
+            <soft_cfm>0.8</soft_cfm>
+            <soft_erp>0.8</soft_erp>
+            <kd>2500</kd>
+            <kp>10</kp>
+            <min_depth>0.001</min_depth>
+          </ode>
+        </contact>
+      </surface>
     </link>
+    <joint name="table_joint_tilt" type="revolute">
+      <parent link="table_surface_interface"/>
+      <child link="table_surface"/>
+      <origin xyz="0 0 0" rpy="0 0 1.5707"/>
+      <axis xyz="0 1 0"/>
+      <limit lower="-0.8" upper="0.3"
+             effort="10000" velocity="10000" />
+      <dynamics damping="0.5" friction = "0.1"/>
+    </joint>
+    <link name="table_surface_interface">
+        <visual><geometry><sphere radius=".00001"/></geometry></visual>
+        <collision><geometry><sphere radius=".00001"/></geometry></collision>
+        <inertial>
+            <origin xyz="0 0 0" rpy="0 0 0"/>
+            <mass value="0.0001"/>
+            <inertia ixx="0.1" ixy="0.0" ixz="0.0" iyy="0.1"  iyz="0.0" izz="0.1"/>
+        </inertial>
+    </link>
+<!--     <joint name="table_joint_tilt2" type="revolute">
+      <parent link="table_surface_interface"/>
+      <child link="table_surface"/>
+      <origin xyz="0 0 0" rpy="0 0 1.5707"/>
+      <axis xyz="0 1 0"/>
+      <limit lower="-0.8" upper="0.3"
+             effort="10000" velocity="10000" />
+      <dynamics damping="0.5" friction = "0.1"/>
+    </joint>
+    <link name="table_surface_interface">
+        <visual><geometry><sphere radius=".00001"/></geometry></visual>
+        <collision><geometry><sphere radius=".00001"/></geometry></collision>
+        <inertial>
+            <origin xyz="0 0 0" rpy="0 0 0"/>
+            <mass value="0.0001"/>
+            <inertia ixx="0.1" ixy="0.0" ixz="0.0" iyy="0.1"  iyz="0.0" izz="0.1"/>
+        </inertial>
+    </link>
+ -->
   </xacro:macro>
 </robot>

File: iiwa_description/urdf/iiwa.gazebo.xacro (robot description, xacro)
@@ -8,14 +8,14 @@
       </plugin>
     </gazebo>
-<!--Force sensors
+<!-- Force sensors -->
     <gazebo>
       <plugin name='gazebo_ros_ft_sensor' filename='libgazebo_ros_ft_sensor.so'>
           <robotNamespace>/${robot_name}</robotNamespace>
-          <topicName>ft_sensor_data</topicName>
+          <topicName>ft_sensor_ee</topicName>
           <jointName>${robot_name}_joint_7</jointName>
           <updateRate>10</updateRate>
       </plugin>
   </gazebo>
-  <gazebo>
+<!--   <gazebo>
       <plugin name='gazebo_ros_ft_sensor_claw' filename='libgazebo_ros_ft_sensor.so'>
           <robotNamespace>/${robot_name}</robotNamespace>
@@ -24,6 +24,5 @@
           <updateRate>10</updateRate>
       </plugin>
-  </gazebo>
--->
+  </gazebo> -->
     <gazebo>
       <static>0</static>

File: iiwa_description/urdf/iiwa14.xacro (robot description, xacro)
@@ -242,4 +242,7 @@
              effort="${max_effort}" velocity="${max_velocity}" />
       <dynamics damping="${joint_damping}" friction="${joint_friction}"/>
+      <sensor name="force_torque" type="force_torque">
+          <update_rate>100</update_rate>
+      </sensor>
     </joint>
     <link name="${robot_name}_link_7">
