Commit message: sim works for python ik solver

File: iiwa_description/urdf/force_control_platform/force_control.transmission.xacro (robot description, xacro)
@@ -72,4 +72,14 @@
       </actuator>
     </transmission>
+<!--   <transmission name="${robot_name}_tran_8">
+      <robotNamespace>/${robot_name}</robotNamespace>
+      <type>transmission_interface/SimpleTransmission</type>
+      <joint name="kuka_fitting_ee">
+      <hardwareInterface>hardware_interface/${hardware_interface}</hardwareInterface>
+      </joint>
+      <actuator name="${robot_name}_motor_8">
+  <mechanicalReduction>1</mechanicalReduction>
+      </actuator>
+    </transmission> -->
 <!--
   <transmission name="pulsating_surface_tran_1">

File: iiwa_description/urdf/kuka_fittings/kuka_fitting_base.xacro (robot description, xacro)
@@ -48,4 +48,24 @@
     </collision>
   </link>
+<!--
+  <joint name="kuka_fitting_ee" type="revolute">
+    <parent link="kuka_fitting_link"/>
+    <child link="kuka_fitting_ee_"/>
+    <origin xyz="0 0 0.1" rpy="0 3.14 0"/>
+    <limit lower="0" upper="0"
+           effort="0" velocity="0" />
+  </joint>
+  <link name="kuka_fitting_ee_">
+    <visual><geometry><sphere radius=".00001"/></geometry></visual>
+    <collision><geometry><sphere radius=".00001"/></geometry></collision>
+    <inertial>
+      <origin xyz="0 0 0" rpy="0 0 0" />
+      <mass value="0.001" />
+      <inertia
+        ixx="0.0001" ixy="0.0" ixz="0.0"
+        iyy="0.0001" iyz="0.0"
+        izz="0.0001" />
+    </inertial>
+  </link> -->
   </xacro:macro>
 </robot>

Commit message: sim works for python ik solver

File: iiwa_description/urdf/force_control_platform/force_control.transmission.xacro (robot description, xacro)
@@ -72,5 +72,5 @@
       </actuator>
     </transmission>
-<!--   <transmission name="${robot_name}_tran_8">
+  <transmission name="${robot_name}_tran_8">
       <robotNamespace>/${robot_name}</robotNamespace>
       <type>transmission_interface/SimpleTransmission</type>
@@ -81,5 +81,5 @@
   <mechanicalReduction>1</mechanicalReduction>
       </actuator>
-    </transmission> -->
+    </transmission>
 <!--
   <transmission name="pulsating_surface_tran_1">

File: iiwa_description/urdf/kuka_fittings/kuka_fitting_base.xacro (robot description, xacro)
@@ -48,5 +48,4 @@
     </collision>
   </link>
-<!--
   <joint name="kuka_fitting_ee" type="revolute">
     <parent link="kuka_fitting_link"/>
@@ -67,5 +66,5 @@
         izz="0.0001" />
     </inertial>
-  </link> -->
+  </link>
   </xacro:macro>
 </robot>
