Commit message: modified the pulsating surface model

File: iiwa_description/urdf/force_control_platform/pulsating_surface.transmission.xacro (robot description, xacro)
@@ -12,5 +12,5 @@
   </actuator>
   </transmission>
-  <transmission name="pulsating_surface_tran_2">
+<!--   <transmission name="pulsating_surface_tran_2">
       <robotNamespace>/${robot_name}</robotNamespace>
       <type>transmission_interface/SimpleTransmission</type>
@@ -21,5 +21,45 @@
    <mechanicalReduction>1</mechanicalReduction>
   </actuator>
+  </transmission> -->
+  <transmission name="pulsating_surface_tran_3">
+      <robotNamespace>/${robot_name}</robotNamespace>
+      <type>transmission_interface/SimpleTransmission</type>
+  <joint name="table_joint_x">
+   <hardwareInterface>hardware_interface/${hardware_interface}</hardwareInterface>
+  </joint>
+  <actuator name="pulsating_surface_motor_3">
+   <mechanicalReduction>1</mechanicalReduction>
+  </actuator>
   </transmission>
+  <transmission name="pulsating_surface_tran_4">
+      <robotNamespace>/${robot_name}</robotNamespace>
+      <type>transmission_interface/SimpleTransmission</type>
+  <joint name="table_joint_y">
+   <hardwareInterface>hardware_interface/${hardware_interface}</hardwareInterface>
+  </joint>
+  <actuator name="pulsating_surface_motor_4">
+   <mechanicalReduction>1</mechanicalReduction>
+  </actuator>
+  </transmission>
+  <transmission name="pulsating_surface_tran_5">
+      <robotNamespace>/${robot_name}</robotNamespace>
+      <type>transmission_interface/SimpleTransmission</type>
+  <joint name="table_joint_tilt_x">
+   <hardwareInterface>hardware_interface/${hardware_interface}</hardwareInterface>
+  </joint>
+  <actuator name="pulsating_surface_motor_5">
+   <mechanicalReduction>1</mechanicalReduction>
+  </actuator>
+  </transmission>
+<!--   <transmission name="pulsating_surface_tran_6">
+      <robotNamespace>/${robot_name}</robotNamespace>
+      <type>transmission_interface/SimpleTransmission</type>
+  <joint name="table_joint_tilt_y">
+   <hardwareInterface>hardware_interface/${hardware_interface}</hardwareInterface>
+  </joint>
+  <actuator name="pulsating_surface_motor_6">
+   <mechanicalReduction>1</mechanicalReduction>
+  </actuator>
+  </transmission> -->
   </xacro:macro>
 </robot>

File: iiwa_description/urdf/force_control_platform/pulsating_surface.xacro (robot description, xacro)
@@ -8,5 +8,5 @@
       <origin xyz="1.5 0.25 0.15" rpy="0 0 1.5707"/>
       <axis xyz="0 0 1"/>
-      <limit lower="-0.8" upper="0.3"
+      <limit lower="-0.8" upper="1.0"
              effort="10000" velocity="10000" />
       <dynamics damping="0.5" friction = "0.1"/>
@@ -58,13 +58,4 @@
       </surface>
     </link>
-    <joint name="table_joint_tilt" type="revolute">
-      <parent link="table_surface_interface"/>
-      <child link="table_surface"/>
-      <origin xyz="0 0 0" rpy="0 0 1.5707"/>
-      <axis xyz="0 1 0"/>
-      <limit lower="-0.8" upper="0.3"
-             effort="10000" velocity="10000" />
-      <dynamics damping="0.5" friction = "0.1"/>
-    </joint>
     <link name="table_surface_interface">
         <visual><geometry><sphere radius=".00001"/></geometry></visual>
@@ -76,4 +67,68 @@
         </inertial>
     </link>
+    <joint name="table_joint_y" type="prismatic">
+        <parent link="table_surface_interface"/>
+        <child link="table_surface_interface_y"/>
+        <origin xyz="0.0 0.0 0.15" rpy="0 0 0"/>
+        <axis xyz="1 0 0"/>
+        <limit lower="-0.8" upper="1.0"
+               effort="10000" velocity="10000" />
+        <dynamics damping="0.5" friction = "0.1"/>
+    </joint>
+    <link name="table_surface_interface_y">
+        <visual><geometry><sphere radius=".00001"/></geometry></visual>
+        <collision><geometry><sphere radius=".00001"/></geometry></collision>
+        <inertial>
+            <origin xyz="0 0 0" rpy="0 0 0"/>
+            <mass value="0.0001"/>
+            <inertia ixx="0.1" ixy="0.0" ixz="0.0" iyy="0.1"  iyz="0.0" izz="0.1"/>
+        </inertial>
+    </link>
+    <joint name="table_joint_x" type="prismatic">
+      <parent link="table_surface_interface_y"/>
+      <child link="table_surface_interface_x"/>
+      <origin xyz="0 0.0 0.15" rpy="0 0 0"/>
+      <axis xyz="0 1 0"/>
+      <limit lower="-0.8" upper="1.0"
+             effort="10000" velocity="10000" />
+      <dynamics damping="0.5" friction = "0.1"/>
+    </joint>
+    <link name="table_surface_interface_x">
+        <visual><geometry><sphere radius=".00001"/></geometry></visual>
+        <collision><geometry><sphere radius=".00001"/></geometry></collision>
+        <inertial>
+            <origin xyz="0 0 0" rpy="0 0 0"/>
+            <mass value="0.0001"/>
+            <inertia ixx="0.1" ixy="0.0" ixz="0.0" iyy="0.1"  iyz="0.0" izz="0.1"/>
+        </inertial>
+    </link>
+    <joint name="table_joint_tilt_x" type="revolute">
+        <parent link="table_surface_interface_x"/>
+        <child link="table_surface"/>
+        <origin xyz="0 0 0" rpy="0 0 1.5707"/>
+        <axis xyz="0 1 0"/>
+        <limit lower="-0.8" upper="0.3"
+               effort="10000" velocity="10000" />
+        <dynamics damping="0.5" friction = "0.1"/>
+    </joint>
+<!--     <link name="table_surface_interface_tilt">
+        <visual><geometry><sphere radius=".00001"/></geometry></visual>
+        <collision><geometry><sphere radius=".00001"/></geometry></collision>
+        <inertial>
+            <origin xyz="0 0 0" rpy="0 0 0"/>
+            <mass value="0.0001"/>
+            <inertia ixx="0.1" ixy="0.0" ixz="0.0" iyy="0.1"  iyz="0.0" izz="0.1"/>
+        </inertial>
+    </link>
+    <joint name="table_joint_tilt_y" type="revolute">
+        <parent link="table_surface_interface_tilt"/>
+        <child link="table_surface"/>
+        <origin xyz="0 0 0" rpy="0 0 0"/>
+        <axis xyz="1 0 0"/>
+        <limit lower="-0.8" upper="0.3"
+               effort="10000" velocity="10000" />
+        <dynamics damping="0.5" friction = "0.1"/>
+    </joint>
+ -->
 <!--     <joint name="table_joint_tilt2" type="revolute">
       <parent link="table_surface_interface"/>

File: iiwa_description/urdf/kuka_fittings/kuka_fitting_base.xacro (robot description, xacro)
@@ -51,5 +51,5 @@
     <parent link="kuka_fitting_link"/>
     <child link="kuka_fitting_ee_"/>
-    <origin xyz="0 0 0.1" rpy="0 3.14 0"/>
+    <origin xyz="0 0 -0.13" rpy="0 -3.14 0"/>
     <limit lower="0" upper="0"
            effort="0" velocity="0" />
