Commit message: latest from thinkpad

File: iiwa_description/urdf/force_control_platform/iiwa14.xacro (robot description, xacro)
@@ -250,5 +250,5 @@
       </inertial>
       <visual>
-        <origin xyz="0 0 0" rpy="0 0 0"/>
+        <origin xyz="0 0 -0.13" rpy="0 0 0"/>
         <geometry>
           <mesh filename="package://iiwa_description/meshes/iiwa14/visual/link_7.stl"/>
@@ -257,5 +257,5 @@
       </visual>
       <collision>
-        <origin xyz="0 0 0" rpy="0 0 0"/>
+        <origin xyz="0 0 -0.13" rpy="0 0 0"/>
         <geometry>
           <mesh filename="package://iiwa_description/meshes/iiwa14/collision/link_7.stl"/>

File: iiwa_description/urdf/force_control_platform/pulsating_surface.xacro (robot description, xacro)
@@ -6,8 +6,8 @@
       <parent link="world"/>
       <child link="table_surface_interface"/>
-      <origin xyz="1.5 0.25 0.15" rpy="0 0 1.5707"/>
+      <origin xyz="1.5 0.25 0.0" rpy="0 0 0"/>
       <axis xyz="0 0 1"/>
       <limit lower="-0.8" upper="1.0"
-             effort="10000" velocity="10000" />
+             effort="100" velocity="10000" />
       <dynamics damping="0.5" friction = "0.1"/>
     </joint>

File: iiwa_description/urdf/iiwa14.xacro (robot description, xacro)
@@ -4,10 +4,10 @@
   <xacro:property name="safety_controller_k_pos" value="100" />
   <xacro:property name="safety_controller_k_vel" value="2" />
-  <xacro:property name="joint_damping" value="0.4" />
-  <xacro:property name="joint_friction" value="1.4"/>
+  <!-- <xacro:property name="joint_damping" value="0.4" /> -->
+  <!-- <xacro:property name="joint_friction" value="1.4"/> -->
   <xacro:property name="max_effort" value="5000"/>
-  <xacro:property name="max_velocity" value="100"/>
-  <xacro:property name="joint_friction" value="0.005" />
-  <xacro:property name="joint_damping" value="0.9" />
+  <xacro:property name="max_velocity" value="10"/>
+  <xacro:property name="joint_friction" value="0.05" />
+  <xacro:property name="joint_damping" value="10.8" />
   <xacro:property name="PIhalf" value="1.570796" />
   <xacro:property name="PI" value="3.141592" />
@@ -248,7 +248,7 @@
     <link name="${robot_name}_link_7">
       <inertial>
-        <origin xyz="0 0 0.02" rpy="0 0 0"/>
+        <origin xyz="0 0 -0.1" rpy="0 0 0"/>
         <mass value="0.3"/>
-        <inertia ixx="0.001"  ixy="0"  ixz="0" iyy="0.001" iyz="0" izz="0.001" />
+        <inertia ixx="0.1"  ixy="0"  ixz="0" iyy="0.1" iyz="0" izz="0.1" />
       </inertial>
       <visual>
