Commit message: Working simulation, controllers loaded

File: iiwa_description/urdf/dual_arm_system/dual_arm_left.xacro (robot description, xacro)
@@ -20,25 +20,26 @@
       xyz="0 0 1" />
     <limit
-      lower="-3.14"
-      upper="3.14"
-      effort="20000"
-      velocity="13" />
-    <dynamics damping="${joint_damping}" friction = "${joint_friction}"/>
-  </joint>
-  <link
+      lower="-${PI}"
+      upper="${PI}"
+      effort="20000"
+      velocity="13" />
+    <dynamics damping="${joint_damping}" friction = "${joint_friction}"/>
+  </joint>
+   <link
     name="Link_L1">
     <inertial>
       <origin
-        xyz="0.00302464836897415 0.00148467584367146 -0.0196712040191069"
-        rpy="0 0 0" />
-      <mass
-        value="0.523170961054133" />
-      <inertia
-        ixx="9.86315700006277E-05"
-        ixy="-1.83712585125958E-06"
-        ixz="1.50310533353745E-05"
-        iyy="0.000101226511355012"
-        iyz="6.90483440689725E-06"
-        izz="4.61898687854836E-06" />
+        xyz="0 -0.00002198 0.03386448"
+        rpy="0 0 0" />
+      <mass
+        value="0.34855237" />
+      <inertia
+        ixx="0.00041198"
+        ixy="0"
+        ixz="0"
+        iyy="0.00042179"
+        iyz="-0.00000013"
+        izy="-0.00000013"
+        izz="0.00045583" />
     </inertial>
     <visual>
@@ -49,5 +50,5 @@
         <mesh
           filename="package://iiwa_description/meshes/Dual_Arm_Manipulator/Arm/Link_1.STL" />
-      </geometry>
+      </geometry><!--iiwa14/collision/Dual_Arm/Link1.STL-->
       <material
         name="">
@@ -62,5 +63,5 @@
       <geometry>
         <mesh
-          filename="package://iiwa_description/meshes/Dual_Arm_Manipulator/Arm/Link_1.STL"  />
+          filename="package://iiwa_description/meshes/Dual_Arm_Manipulator/Arm/Link_1_collision.STL" />
       </geometry>
     </collision>
@@ -72,6 +73,5 @@
       xyz="0 0 0.098815"
       rpy="-${PIhalf} 0 0" />
-      <!-- xyz="0 0 -0.0635"
-      rpy="1.57079632679489 -0.380374098489847 0.317429885556193"-->
+      <!-- "1.57079632679489 -0.380374098489847 0.317429885556193"-->
     <parent
       link="Link_L1" />
@@ -81,25 +81,27 @@
       xyz="0 0 1" />
     <limit
-      lower="-1.57"
-      upper="1.57"
-      effort="20000"
-      velocity="13" />
-    <dynamics damping="${joint_damping}" friction = "${joint_friction}"/>
-  </joint>
-  <link
+      lower="-${PI}"
+      upper="${PI}"
+      effort="20000"
+      velocity="13" />
+    <dynamics damping="${joint_damping}" friction = "${joint_friction}"/>
+  </joint>
+<link
     name="Link_L2">
     <inertial>
       <origin
-        xyz="-0.0841816926424142 -9.94783774485586E-05 0.00119770428720625"
-        rpy="0 0 0" />
-      <mass
-        value="0.361073886022953" />
-      <inertia
-        ixx="1.38598083295319E-06"
-        ixy="-3.76180464461997E-07"
-        ixz="5.01830776658136E-09"
-        iyy="0.000417336089370728"
-        iyz="3.07943156555252E-09"
-        izz="0.000417240402620394" />
+        xyz="-0.00002616 -0.08182747 0.00586724"
+        rpy="0 0 0" />
+      <mass
+        value=" 0.14210191" />
+      <inertia
+        ixx="0.00061848"
+        ixy="0.00000018"
+        ixz="0"
+        iyx="0.00000018"
+        iyy="0.00003828"
+        iyz="-0.00005076"
+        izy="-0.00005076"
+        izz="0.00060901" />
     </inertial>
     <visual>
@@ -114,14 +116,14 @@
         name="">
         <color
-          rgba="1 1 1 1" />
-      </material>
-    </visual>
-    <collision>
-      <origin
-        xyz="0 0 0"
-        rpy="0 0 0" />
-      <geometry>
-        <mesh
-          filename="package://iiwa_description/meshes/Dual_Arm_Manipulator/Arm/Link_2.STL" />
+          rgba="0.898039215686275 0.898039215686275 0.898039215686275 1" />
+      </material>
+    </visual>
+    <collision>
+      <origin
+        xyz="0 0 0"
+        rpy="0 0 0" />
+      <geometry>
+        <mesh
+          filename="package://iiwa_description/meshes/Dual_Arm_Manipulator/Arm/Link_2_collision.STL" />
       </geometry>
     </collision>
@@ -142,26 +144,34 @@
       xyz="0 0 1" />
     <limit
-      lower="-3.14"
-      upper="3.14"
-      effort="20000"
-      velocity="13" />
-    <dynamics damping="${joint_damping}" friction = "${joint_friction}"/>
-  </joint>
-  <link name="Link_L3">
+      lower="-${PI}"
+      upper="${PI}"
+      effort="20000"
+      velocity="13" />
+    <dynamics damping="${joint_damping}" friction = "${joint_friction}"/>
+  </joint>
+  <link
+    name="Link_L3">
     <inertial>
-      <origin xyz="0.00289722994622221 0.00112305403125196 0.0290055866352336" rpy="0 0 0" />
-      <mass value="0.217746913814738" />
-      <inertia
-        ixx="9.95073774261661E-05"
-        ixy="-2.667473422779E-07"
-        ixz="-3.12070252262036E-06"
-        iyy="0.000106288781760734"
-        iyz="-2.88857039626312E-06"
-        izz="6.98820523527226E-06" />
-    </inertial>
-    <visual>
-      <origin xyz="0 0 0" rpy="0 0 0" />
-      <geometry>
-        <mesh filename="package://iiwa_description/meshes/Dual_Arm_Manipulator/Arm/Link_3.STL" />
+      <origin
+        xyz="0.00018087 0 0.11630050"
+        rpy="0 0 0" />
+      <mass
+        value="0.09637272" />
+      <inertia
+        ixx="0.00031529"
+        ixy="0"
+        ixz="0.00000077"
+        iyy="0.00031517"
+        iyz="0"
+        izx="0.00000077"
+        izz="0.00001827" />
+    </inertial>
+    <visual>
+      <origin
+        xyz="0 0 0"
+        rpy="0 0 0" />
+      <geometry>
+        <mesh
+          filename="package://iiwa_description/meshes/Dual_Arm_Manipulator/Arm/Link_3.STL" />
       </geometry>
       <material
@@ -177,5 +187,5 @@
       <geometry>
         <mesh
-          filename="package://iiwa_description/meshes/Dual_Arm_Manipulator/Arm/Link_3.STL" />
+          filename="package://iiwa_description/meshes/Dual_Arm_Manipulator/Arm/Link_3_collision.STL" />
       </geometry>
     </collision>
@@ -187,5 +197,5 @@
       xyz="-0.019005 0 0.1675"
       rpy="0 -${PIhalf} 0" />
-      <!-- xyz="0.0266700000000004 0.0019050000000066 0.0609600000000012"
+      <!--xyz="0.0266700000000004 0.0019050000000066 0.0609600000000012"
       rpy="-1.5707963267949 -0.824186362211141 -1.57079632679489"-->
     <parent
@@ -196,6 +206,6 @@
       xyz="0 0 1" />
     <limit
-      lower="-1.57"
-      upper="1.57"
+      lower="-${PI}"
+      upper="${PI}"
       effort="20000"
       velocity="13" />
@@ -206,15 +216,16 @@
       <inertial>
       <origin
-        xyz="-0.00106966507570738 -0.0713978397746767 -0.00106966507570611"
-        rpy="0 0 0" />
-      <mass
-        value="0.217746913814738" />
-      <inertia
-        ixx="9.95073774261661E-05"
-        ixy="-2.667473422779E-07"
-        ixz="-3.12070252262036E-06"
-        iyy="0.000106288781760734"
-        iyz="-2.88857039626312E-06"
-        izz="6.98820523527226E-06" />
+        xyz=" -0.01338844 0 0.00944589"
+        rpy="0 0 0" />
+      <mass
+        value="0.01812912" />
+      <inertia
+        ixx="0.00000196"
+        ixy="0"
+        ixz="-0.00000004"
+        iyy="0.00000943"
+        iyz="0"
+        izx="-0.00000004"
+        izz="0.00001043" />
     </inertial>
     <visual>
@@ -238,5 +249,5 @@
       <geometry>
         <mesh
-          filename="package://iiwa_description/meshes/Dual_Arm_Manipulator/Arm/Link_4.STL" />
+          filename="package://iiwa_description/meshes/Dual_Arm_Manipulator/Arm/Link_4_collision.STL" />
       </geometry>
     </collision>

File: iiwa_description/urdf/dual_arm_system/dual_arm_right.xacro (robot description, xacro)
@@ -19,6 +19,6 @@
       xyz="0 0 1" />
     <limit
-      lower="-3.14"
-      upper="3.14"
+      lower="-${PI}"
+      upper="${PI}"
       effort="20000"
       velocity="13" />
@@ -29,15 +29,16 @@
     <inertial>
       <origin
-        xyz="0.00302464836897415 0.00148467584367146 -0.0196712040191069"
-        rpy="0 0 0" />
-      <mass
-        value="0.523170961054133" />
-      <inertia
-        ixx="9.86315700006277E-05"
-        ixy="-1.83712585125958E-06"
-        ixz="1.50310533353745E-05"
-        iyy="0.000101226511355012"
-        iyz="6.90483440689725E-06"
-        izz="4.61898687854836E-06" />
+        xyz="0 -0.00002198 0.03386448"
+        rpy="0 0 0" />
+      <mass
+        value="0.34855237" />
+      <inertia
+        ixx="0.00041198"
+        ixy="0"
+        ixz="0"
+        iyy="0.00042179"
+        iyz="-0.00000013"
+        izy="-0.00000013"
+        izz="0.00045583" />
     </inertial>
     <visual>
@@ -61,5 +62,5 @@
       <geometry>
         <mesh
-          filename="package://iiwa_description/meshes/Dual_Arm_Manipulator/Arm/Link_1.STL" />
+          filename="package://iiwa_description/meshes/Dual_Arm_Manipulator/Arm/Link_1_collision.STL" />
       </geometry>
     </collision>
@@ -79,6 +80,6 @@
       xyz="0 0 1" />
     <limit
-      lower="-1.57"
-      upper="1.57"
+      lower="-${PI}"
+      upper="${PI}"
       effort="20000"
       velocity="13" />
@@ -89,15 +90,17 @@
     <inertial>
       <origin
-        xyz="-0.0841816926424142 -9.94783774485586E-05 0.00119770428720625"
-        rpy="0 0 0" />
-      <mass
-        value="0.361073886022953" />
-      <inertia
-        ixx="1.38598083295319E-06"
-        ixy="-3.76180464461997E-07"
-        ixz="5.01830776658136E-09"
-        iyy="0.000417336089370728"
-        iyz="3.07943156555252E-09"
-        izz="0.000417240402620394" />
+        xyz="-0.00002616 -0.08182747 0.00586724"
+        rpy="0 0 0" />
+      <mass
+        value=" 0.14210191" />
+      <inertia
+        ixx="0.00061848"
+        ixy="0.00000018"
+        ixz="0"
+        iyx="0.00000018"
+        iyy="0.00003828"
+        iyz="-0.00005076"
+        izy="-0.00005076"
+        izz="0.00060901" />
     </inertial>
     <visual>
@@ -121,5 +124,5 @@
       <geometry>
         <mesh
-          filename="package://iiwa_description/meshes/Dual_Arm_Manipulator/Arm/Link_2.STL" />
+          filename="package://iiwa_description/meshes/Dual_Arm_Manipulator/Arm/Link_2_collision.STL" />
       </geometry>
     </collision>
@@ -140,6 +143,6 @@
       xyz="0 0 1" />
     <limit
-      lower="-3.14"
-      upper="3.14"
+      lower="-${PI}"
+      upper="${PI}"
       effort="20000"
       velocity="13" />
@@ -150,15 +153,16 @@
     <inertial>
       <origin
-        xyz="0.00289722994622221 0.00112305403125196 0.0290055866352336"
-        rpy="0 0 0" />
-      <mass
-        value="0.217746913814738" />
-      <inertia
-        ixx="9.95073774261661E-05"
-        ixy="-2.667473422779E-07"
-        ixz="-3.12070252262036E-06"
-        iyy="0.000106288781760734"
-        iyz="-2.88857039626312E-06"
-        izz="6.98820523527226E-06" />
+        xyz="0.00018087 0 0.11630050"
+        rpy="0 0 0" />
+      <mass
+        value="0.09637272" />
+      <inertia
+        ixx="0.00031529"
+        ixy="0"
+        ixz="0.00000077"
+        iyy="0.00031517"
+        iyz="0"
+        izx="0.00000077"
+        izz="0.00001827" />
     </inertial>
     <visual>
@@ -182,5 +186,5 @@
       <geometry>
         <mesh
-          filename="package://iiwa_description/meshes/Dual_Arm_Manipulator/Arm/Link_3.STL" />
+          filename="package://iiwa_description/meshes/Dual_Arm_Manipulator/Arm/Link_3_collision.STL" />
       </geometry>
     </collision>
@@ -201,6 +205,6 @@
       xyz="0 0 1" />
     <limit
-      lower="-1.57"
-      upper="1.57"
+      lower="-${PI}"
+      upper="${PI}"
       effort="20000"
       velocity="13" />
@@ -211,15 +215,16 @@
       <inertial>
       <origin
-        xyz="-0.00106966507570738 -0.0713978397746767 -0.00106966507570611"
-        rpy="0 0 0" />
-      <mass
-        value="0.217746913814738" />
-      <inertia
-        ixx="9.95073774261661E-05"
-        ixy="-2.667473422779E-07"
-        ixz="-3.12070252262036E-06"
-        iyy="0.000106288781760734"
-        iyz="-2.88857039626312E-06"
-        izz="6.98820523527226E-06" />
+        xyz=" -0.01338844 0 0.00944589"
+        rpy="0 0 0" />
+      <mass
+        value="0.01812912" />
+      <inertia
+        ixx="0.00000196"
+        ixy="0"
+        ixz="-0.00000004"
+        iyy="0.00000943"
+        iyz="0"
+        izx="-0.00000004"
+        izz="0.00001043" />
     </inertial>
     <visual>
@@ -243,5 +248,5 @@
       <geometry>
         <mesh
-          filename="package://iiwa_description/meshes/Dual_Arm_Manipulator/Arm/Link_4.STL" />
+          filename="package://iiwa_description/meshes/Dual_Arm_Manipulator/Arm/Link_4_collision.STL" />
       </geometry>
     </collision>

File: iiwa_description/urdf/dual_arm_system/iiwa.gazebo.xacro (robot description, xacro)
@@ -153,4 +153,5 @@
       <selfCollide>0</selfCollide>
     </gazebo>
+<!--
     <gazebo reference="gripper_base_link">
       <material>Gazebo/White</material>
@@ -191,5 +192,5 @@
     <gazebo reference="${robot_name}_joint_7">
       <provideFeedback>true</provideFeedback>
-    </gazebo>
+    </gazebo>-->
     <!--EOAT-->
 <!--

File: iiwa_description/urdf/dual_arm_system/iiwa.transmission.xacro (robot description, xacro)
@@ -152,4 +152,5 @@
       </actuator>
     </transmission>
+<!--
   <transmission name="gripper_base_joint_tran">
       <robotNamespace>/${robot_name}</robotNamespace>
@@ -211,5 +212,5 @@
   <mechanicalReduction>1</mechanicalReduction>
       </actuator>
-    </transmission>
+    </transmission>-->
 <!--
   <transmission name="pulsating_surface_tran_1">
