Commit message: New arms added to gazebo model. Inertial properties need to be updated, collision meshes are needed and a solution to it being unstable is also needed

File: iiwa_description/urdf/dual_arm_system/Dual_Arm.xacro (robot description, xacro)
@@ -60,6 +60,6 @@
   <xacro:dual_arm_right robot_name="${robot_name}"/>
   <xacro:dual_arm_left robot_name="${robot_name}"/>
-  <xacro:gripper_R robot_name="$(arg robot_name)"/>
-  <xacro:gripper_L robot_name="$(arg robot_name)"/>
+  <!--<xacro:gripper_R robot_name="$(arg robot_name)"/>
+  <xacro:gripper_L robot_name="$(arg robot_name)"/>-->
   </xacro:macro>
 </robot>

File: iiwa_description/urdf/dual_arm_system/complete_chain.urdf.xacro (robot description, xacro)
@@ -7,9 +7,9 @@
 	<xacro:include filename="$(find iiwa_description)/urdf/pulsating_surface.transmission.xacro" />
 	<xacro:include filename="$(find iiwa_description)/urdf/dual_arm_system/iiwa.transmission.xacro" />
-	<xacro:pulsating_surface robot_name="$(arg robot_name)"/>
+	<!--<xacro:pulsating_surface robot_name="$(arg robot_name)"/>-->
 	<xacro:complete_chain robot_name="$(arg robot_name)"/>
 	<!-- <xacro:pulsating_surface_gazebo robot_name="$(arg robot_name)"/> -->
 	<xacro:iiwa_gazebo robot_name="$(arg robot_name)"/>
 	<xacro:iiwa_transmission hardware_interface="$(arg hardware_interface)" robot_name="$(arg robot_name)"/>
-	<xacro:pulsating_surface_transmission hardware_interface="$(arg hardware_interface)" robot_name="$(arg robot_name)"/>
+	<!--<xacro:pulsating_surface_transmission hardware_interface="$(arg hardware_interface)" robot_name="$(arg robot_name)"/>-->
 </robot>

File: iiwa_description/urdf/dual_arm_system/dual_arm_left.xacro (robot description, xacro)
@@ -11,5 +11,6 @@
     <origin
       xyz="-0.0744445637977397 0.152871273073736 -0.110435575211296"
-      rpy="-1.43251148060093 -0.775712981728982 2.94539473140516" />
+      rpy="-1.7091 0.7757 -0.1962" />
+      <!-- rpy="-1.43251148060093 -0.775712981728982 2.94539473140516"-->
     <parent
       link="base_link" />
@@ -47,19 +48,19 @@
       <geometry>
         <mesh
-          filename="package://iiwa_description/meshes/iiwa14/collision/Dual_Arm/Link1.STL" />
-      </geometry>
-      <material
-        name="">
-        <color
-          rgba="1 1 1 1" />
-      </material>
-    </visual>
-    <collision>
-      <origin
-        xyz="0 0 0"
-        rpy="0 0 0" />
-      <geometry>
-        <mesh
-          filename="package://iiwa_description/meshes/iiwa14/collision/Dual_Arm/Link1.STL" />
+          filename="package://iiwa_description/meshes/Dual_Arm_Manipulator/Arm/Link_1.STL" />
+      </geometry>
+      <material
+        name="">
+        <color
+          rgba="1 1 1 1" />
+      </material>
+    </visual>
+    <collision>
+      <origin
+        xyz="0 0 0"
+        rpy="0 0 0" />
+      <geometry>
+        <mesh
+          filename="package://iiwa_description/meshes/Dual_Arm_Manipulator/Arm/Link_1.STL"  />
       </geometry>
     </collision>
@@ -69,6 +70,8 @@
     type="revolute">
     <origin
-      xyz="0 0 -0.0635"
-      rpy="1.57079632679489 -0.380374098489847 0.317429885556193" />
+      xyz="0 0 0.098815"
+      rpy="-${PIhalf} 0 0" />
+      <!-- xyz="0 0 -0.0635"
+      rpy="1.57079632679489 -0.380374098489847 0.317429885556193"-->
     <parent
       link="Link_L1" />
@@ -106,19 +109,19 @@
       <geometry>
         <mesh
-          filename="package://iiwa_description/meshes/iiwa14/collision/Dual_Arm/Link2.STL" />
-      </geometry>
-      <material
-        name="">
-        <color
-          rgba="1 1 1 1" />
-      </material>
-    </visual>
-    <collision>
-      <origin
-        xyz="0 0 0"
-        rpy="0 0 0" />
-      <geometry>
-        <mesh
-          filename="package://iiwa_description/meshes/iiwa14/collision/Dual_Arm/Link2.STL" />
+          filename="package://iiwa_description/meshes/Dual_Arm_Manipulator/Arm/Link_2.STL" />
+      </geometry>
+      <material
+        name="">
+        <color
+          rgba="1 1 1 1" />
+      </material>
+    </visual>
+    <collision>
+      <origin
+        xyz="0 0 0"
+        rpy="0 0 0" />
+      <geometry>
+        <mesh
+          filename="package://iiwa_description/meshes/Dual_Arm_Manipulator/Arm/Link_2.STL" />
       </geometry>
     </collision>
@@ -128,6 +131,8 @@
     type="revolute">
     <origin
-      xyz="-0.178688999999999 -0.00012700000000021 0"
-      rpy="-1.57079632679489 -1.0547118733939E-15 1.5707963267949" />
+      xyz="0 -0.16645 0"
+      rpy="${PIhalf} 0 0" />
+      <!-- xyz="-0.178688999999999 -0.00012700000000021 0"
+      rpy="-1.57079632679489 -1.0547118733939E-15 1.5707963267949"-->
     <parent
       link="Link_L2" />
@@ -158,19 +163,19 @@
       <origin xyz="0 0 0" rpy="0 0 0" />
       <geometry>
-        <mesh filename="package://iiwa_description/meshes/iiwa14/collision/Dual_Arm/Link3.STL" />
-      </geometry>
-      <material
-        name="">
-        <color
-          rgba="1 1 1 1" />
-      </material>
-    </visual>
-    <collision>
-      <origin
-        xyz="0 0 0"
-        rpy="0 0 0" />
-      <geometry>
-        <mesh
-          filename="package://iiwa_description/meshes/iiwa14/collision/Dual_Arm/Link3.STL" />
+        <mesh filename="package://iiwa_description/meshes/Dual_Arm_Manipulator/Arm/Link_3.STL" />
+      </geometry>
+      <material
+        name="">
+        <color
+          rgba="1 1 1 1" />
+      </material>
+    </visual>
+    <collision>
+      <origin
+        xyz="0 0 0"
+        rpy="0 0 0" />
+      <geometry>
+        <mesh
+          filename="package://iiwa_description/meshes/Dual_Arm_Manipulator/Arm/Link_3.STL" />
       </geometry>
     </collision>
@@ -180,6 +185,8 @@
     type="revolute">
     <origin
-      xyz="0.0266700000000004 0.0019050000000066 0.0609600000000012"
-      rpy="-1.5707963267949 -0.824186362211141 -1.57079632679489" />
+      xyz="-0.019005 0 0.1675"
+      rpy="0 -${PIhalf} 0" />
+      <!-- xyz="0.0266700000000004 0.0019050000000066 0.0609600000000012"
+      rpy="-1.5707963267949 -0.824186362211141 -1.57079632679489"-->
     <parent
       link="Link_L3" />
@@ -217,19 +224,19 @@
       <geometry>
         <mesh
-          filename="package://iiwa_description/meshes/iiwa14/collision/Dual_Arm/Link4.STL" />
-      </geometry>
-      <material
-        name="">
-        <color
-          rgba="1 1 1 1" />
-      </material>
-    </visual>
-    <collision>
-      <origin
-        xyz="0 0 0"
-        rpy="0 0 0" />
-      <geometry>
-        <mesh
-          filename="package://iiwa_description/meshes/iiwa14/collision/Dual_Arm/Link4.STL" />
+          filename="package://iiwa_description/meshes/Dual_Arm_Manipulator/Arm/Link_4.STL" />
+      </geometry>
+      <material
+        name="">
+        <color
+          rgba="1 1 1 1" />
+      </material>
+    </visual>
+    <collision>
+      <origin
+        xyz="0 0 0"
+        rpy="0 0 0" />
+      <geometry>
+        <mesh
+          filename="package://iiwa_description/meshes/Dual_Arm_Manipulator/Arm/Link_4.STL" />
       </geometry>
     </collision>

File: iiwa_description/urdf/dual_arm_system/dual_arm_right.xacro (robot description, xacro)
@@ -11,5 +11,5 @@
     <origin
       xyz="-0.0744445637977397 -0.152871273073736 -0.110435575211296"
-      rpy="1.43251148060093 -0.775712981728982 -2.94539473140516" />
+      rpy="1.7091 0.7757 0.1962" /> <!-- "1.43251148060093 -0.775712981728982 -2.94539473140516" -->
     <parent
       link="base_link" />
@@ -47,6 +47,6 @@
       <geometry>
         <mesh
-          filename="package://iiwa_description/meshes/iiwa14/collision/Dual_Arm/Link1.STL" />
-      </geometry>
+          filename="package://iiwa_description/meshes/Dual_Arm_Manipulator/Arm/Link_1.STL" />
+      </geometry><!--iiwa14/collision/Dual_Arm/Link1.STL-->
       <material
         name="">
@@ -61,5 +61,5 @@
       <geometry>
         <mesh
-          filename="package://iiwa_description/meshes/iiwa14/collision/Dual_Arm/Link1.STL" />
+          filename="package://iiwa_description/meshes/Dual_Arm_Manipulator/Arm/Link_1.STL" />
       </geometry>
     </collision>
@@ -69,6 +69,7 @@
     type="revolute">
     <origin
-      xyz="0 0 -0.0635"
-      rpy="1.57079632679489 -0.380374098489847 0.317429885556193" />
+      xyz="0 0 0.098815"
+      rpy="-${PIhalf} 0 0" />
+      <!-- "1.57079632679489 -0.380374098489847 0.317429885556193"-->
     <parent
       link="Link_R1" />
@@ -106,5 +107,5 @@
       <geometry>
         <mesh
-          filename="package://iiwa_description/meshes/iiwa14/collision/Dual_Arm/Link2.STL" />
+          filename="package://iiwa_description/meshes/Dual_Arm_Manipulator/Arm/Link_2.STL" />
       </geometry>
       <material
@@ -120,5 +121,5 @@
       <geometry>
         <mesh
-          filename="package://iiwa_description/meshes/iiwa14/collision/Dual_Arm/Link2.STL" />
+          filename="package://iiwa_description/meshes/Dual_Arm_Manipulator/Arm/Link_2.STL" />
       </geometry>
     </collision>
@@ -128,6 +129,8 @@
     type="revolute">
     <origin
-      xyz="-0.178688999999999 -0.00012700000000021 0"
-      rpy="-1.57079632679489 -1.0547118733939E-15 1.5707963267949" />
+      xyz="0 -0.16645 0"
+      rpy="${PIhalf} 0 0" />
+      <!-- xyz="-0.178688999999999 -0.00012700000000021 0"
+      rpy="-1.57079632679489 -1.0547118733939E-15 1.5707963267949"-->
     <parent
       link="Link_R2" />
@@ -165,5 +168,5 @@
       <geometry>
         <mesh
-          filename="package://iiwa_description/meshes/iiwa14/collision/Dual_Arm/Link3.STL" />
+          filename="package://iiwa_description/meshes/Dual_Arm_Manipulator/Arm/Link_3.STL" />
       </geometry>
       <material
@@ -179,5 +182,5 @@
       <geometry>
         <mesh
-          filename="package://iiwa_description/meshes/iiwa14/collision/Dual_Arm/Link3.STL" />
+          filename="package://iiwa_description/meshes/Dual_Arm_Manipulator/Arm/Link_3.STL" />
       </geometry>
     </collision>
@@ -187,6 +190,8 @@
     type="revolute">
     <origin
-      xyz="0.0266700000000004 0.0019050000000066 0.0609600000000012"
-      rpy="-1.5707963267949 -0.824186362211141 -1.57079632679489" />
+      xyz="-0.019005 0 0.1675"
+      rpy="0 -${PIhalf} 0" />
+      <!--xyz="0.0266700000000004 0.0019050000000066 0.0609600000000012"
+      rpy="-1.5707963267949 -0.824186362211141 -1.57079632679489"-->
     <parent
       link="Link_R3" />
@@ -224,5 +229,5 @@
       <geometry>
         <mesh
-          filename="package://iiwa_description/meshes/iiwa14/collision/Dual_Arm/Link4.STL" />
+          filename="package://iiwa_description/meshes/Dual_Arm_Manipulator/Arm/Link_4.STL" />
       </geometry>
       <material
@@ -238,5 +243,5 @@
       <geometry>
         <mesh
-          filename="package://iiwa_description/meshes/iiwa14/collision/Dual_Arm/Link4.STL" />
+          filename="package://iiwa_description/meshes/Dual_Arm_Manipulator/Arm/Link_4.STL" />
       </geometry>
     </collision>

Commit message: Model with wrist. Instabilities when last link is added to the controller

File: iiwa_description/urdf/dual_arm_system/Dual_Arm.xacro (robot description, xacro)
@@ -5,4 +5,6 @@
   <xacro:include filename="$(find iiwa_description)/urdf/dual_arm_system/gripper_L.xacro" />
   <xacro:include filename="$(find iiwa_description)/urdf/dual_arm_system/gripper_R.xacro" />
+  <xacro:include filename="$(find iiwa_description)/urdf/dual_arm_system/miniwrist_right.xacro" />
+  <xacro:include filename="$(find iiwa_description)/urdf/dual_arm_system/miniwrist_left.xacro" />
   <xacro:macro name="dual_arm_manipulator" params="robot_name">
   <xacro:property name="joint_friction" value="0.005" />
@@ -58,6 +60,11 @@
     </collision>
   </link>
+  <!-- left arm -->
   <xacro:dual_arm_right robot_name="${robot_name}"/>
+  <!-- right arm -->
   <xacro:dual_arm_left robot_name="${robot_name}"/>
+  <!-- end-effectors -->
+  <xacro:miniwrist_right robot_name="${robot_name}"/>
+  <xacro:miniwrist_left robot_name="${robot_name}"/>
   <!--<xacro:gripper_R robot_name="$(arg robot_name)"/>
   <xacro:gripper_L robot_name="$(arg robot_name)"/>-->

File: iiwa_description/urdf/dual_arm_system/complete_chain.urdf.xacro (robot description, xacro)
@@ -3,5 +3,4 @@
 	<!-- Import all Gazebo-customization elements, including Gazebo colors -->
 	<xacro:include filename="$(find iiwa_description)/urdf/dual_arm_system/complete_chain.xacro" />
-	<xacro:include filename="$(find iiwa_description)/urdf/pulsating_surface.xacro" />
 	<xacro:include filename="$(find iiwa_description)/urdf/dual_arm_system/iiwa.gazebo.xacro" />
 	<xacro:include filename="$(find iiwa_description)/urdf/pulsating_surface.transmission.xacro" />
@@ -10,4 +9,5 @@
 	<xacro:complete_chain robot_name="$(arg robot_name)"/>
 	<!-- <xacro:pulsating_surface_gazebo robot_name="$(arg robot_name)"/> -->
+	<!-- Loads the manipulation environment -->
 	<xacro:iiwa_gazebo robot_name="$(arg robot_name)"/>
 	<xacro:iiwa_transmission hardware_interface="$(arg hardware_interface)" robot_name="$(arg robot_name)"/>

File: iiwa_description/urdf/dual_arm_system/complete_chain.xacro (robot description, xacro)
@@ -10,4 +10,5 @@
 	<xacro:include filename="$(find iiwa_description)/urdf/dual_arm_system/Dual_Arm.xacro" />
 	<xacro:include filename="$(find iiwa_description)/urdf/pulsating_surface.xacro" />
+	<xacro:include filename="$(find iiwa_description)/urdf/dual_arm_system/surgical_env.xacro" />
 	<!-- <xacro:include filename="$(find iiwa_description)/urdf/gripper_eoat.xacro" /> -->
 	<xacro:arg name="hardware_interface" default="EffortJointInterface"/>
@@ -16,4 +17,5 @@
 	<xacro:arg name="origin_rpy" default="0 0 0"/>
 	<xacro:kuka_base_frame robot_name="$(arg robot_name)"/>
+	<xacro:surgical_env robot_name="$(arg robot_name)"/>
 	<!-- <xacro:pulsating_surface robot_name="$(arg robot_name)"/> -->
 	<xacro:iiwa14 hardware_interface="$(arg hardware_interface)" robot_name="$(arg robot_name)" parent="world">

File: iiwa_description/urdf/dual_arm_system/dual_arm_left.xacro (robot description, xacro)
@@ -2,5 +2,5 @@
 <robot xmlns:xacro="http://www.ros.org/wiki/xacro">
   <xacro:property name="joint_friction" value="0.005" />
-  <xacro:property name="joint_damping" value="0.8" />
+  <xacro:property name="joint_damping" value="1.5" />
   <xacro:property name="PIhalf" value="1.570796" />
   <xacro:property name="PI" value="3.141592" />
@@ -195,5 +195,5 @@
     type="revolute">
     <origin
-      xyz="-0.019005 0 0.1675"
+      xyz="0.038005 0 0.1675"
       rpy="0 ${PIhalf} ${PI}" />
       <!--xyz="0.0266700000000004 0.0019050000000066 0.0609600000000012"

File: iiwa_description/urdf/dual_arm_system/dual_arm_right.xacro (robot description, xacro)
@@ -2,5 +2,5 @@
 <robot xmlns:xacro="http://www.ros.org/wiki/xacro">
   <xacro:property name="joint_friction" value="0.005" />
-  <xacro:property name="joint_damping" value="0.8" />
+  <xacro:property name="joint_damping" value="1.0" />
   <xacro:property name="PIhalf" value="1.570796" />
   <xacro:property name="PI" value="3.141592" />
@@ -10,5 +10,5 @@
     type="revolute">
     <origin
-      xyz="-0.0744445637977397 -0.152871273073736 -0.110435575211296"
+      xyz="-0.0744445637977397 -0.152871273073736 -0.080435575211296"
       rpy="1.7091 0.7757 0.1962" /> <!-- "1.43251148060093 -0.775712981728982 -2.94539473140516" -->
     <parent
@@ -102,5 +102,5 @@
         iyz="-0.00005076"
         izy="-0.00005076"
-        izz="0.00060901" />
+        izz="0.0060901" />
     </inertial>
     <visual>
@@ -164,5 +164,5 @@
         iyz="0"
         izx="0.00000077"
-        izz="0.00001827" />
+        izz="0.001827" />
     </inertial>
     <visual>
@@ -194,5 +194,5 @@
     type="revolute">
     <origin
-      xyz="-0.019005 0 0.1675"
+      xyz="0.038005 0 0.1675"
       rpy="0 ${PIhalf} ${PI}" />
       <!--xyz="0.0266700000000004 0.0019050000000066 0.0609600000000012"
@@ -209,5 +209,5 @@
       effort="20000"
       velocity="13" />
-    <dynamics damping="${joint_damping}" friction = "${joint_friction}"/>
+    <dynamics damping="0" friction = "${joint_friction}"/>
   </joint>
  <link
@@ -218,5 +218,5 @@
         rpy="0 0 0" />
       <mass
-        value="0.01812912" />
+        value="0.04812912" />
       <inertia
         ixx="0.00000196"
@@ -226,5 +226,5 @@
         iyz="0"
         izx="-0.00000004"
-        izz="0.00001043" />
+        izz="0.001043" />
     </inertial>
     <visual>

File: iiwa_description/urdf/dual_arm_system/iiwa.gazebo.xacro (robot description, xacro)
@@ -153,4 +153,22 @@
       <selfCollide>0</selfCollide>
     </gazebo>
+    <gazebo reference="object">
+      <material>Gazebo/Red</material>
+      <mu1>0.2</mu1>
+      <mu2>0.2</mu2>
+      <selfCollide>0</selfCollide>
+    </gazebo>
+    <gazebo reference="wristL2_R">
+      <material>Gazebo/Red</material>
+      <mu1>0.2</mu1>
+      <mu2>0.2</mu2>
+      <selfCollide>0</selfCollide>
+    </gazebo>
+    <gazebo reference="wristL2_L">
+      <material>Gazebo/Red</material>
+      <mu1>0.2</mu1>
+      <mu2>0.2</mu2>
+      <selfCollide>0</selfCollide>
+    </gazebo>
 <!--
     <gazebo reference="gripper_base_link">

File: iiwa_description/urdf/iiwa14.urdf.xacro (robot description, xacro)
@@ -8,4 +8,5 @@
   <xacro:include filename="$(find iiwa_description)/urdf/iiwa.gazebo.xacro" />
   <xacro:include filename="$(find iiwa_description)/urdf/materials.xacro" />
+  <xacro:include filename="$(find iiwa_description)/urdf/iiwa.transmission.xacro" />
   <!--Import the lbr iiwa macro -->
   <xacro:include filename="$(find iiwa_description)/urdf/iiwa14.xacro"/>
@@ -66,3 +67,4 @@
   </xacro:iiwa14>
   <xacro:iiwa_gazebo robot_name="$(arg robot_name)"/>
+  <xacro:iiwa_transmission hardware_interface="$(arg hardware_interface)" robot_name="$(arg robot_name)"/>
 </robot>

File: iiwa_description/urdf/iiwa14.xacro (robot description, xacro)
@@ -9,5 +9,5 @@
   <xacro:property name="max_velocity" value="100"/>
   <xacro:property name="joint_friction" value="0.005" />
-  <xacro:property name="joint_damping" value="0.5" />
+  <xacro:property name="joint_damping" value="0.9" />
   <xacro:property name="PIhalf" value="1.570796" />
   <xacro:property name="PI" value="3.141592" />
