Commit message: Stability check

File: iiwa_description/urdf/dual_arm_system/complete_chain.xacro (robot description, xacro)
@@ -17,5 +17,5 @@
 	<xacro:arg name="origin_rpy" default="0 0 0"/>
 	<xacro:kuka_base_frame robot_name="$(arg robot_name)"/>
-	<xacro:surgical_env robot_name="$(arg robot_name)"/>
+	<!-- <xacro:surgical_env robot_name="$(arg robot_name)"/> -->
 	<!-- <xacro:pulsating_surface robot_name="$(arg robot_name)"/> -->
 	<xacro:iiwa14 hardware_interface="$(arg hardware_interface)" robot_name="$(arg robot_name)" parent="world">

File: iiwa_description/urdf/dual_arm_system/dual_arm_left.xacro (robot description, xacro)
@@ -1,5 +1,5 @@
 <?xml version="1.0"?>
 <robot xmlns:xacro="http://www.ros.org/wiki/xacro">
-  <xacro:property name="joint_friction" value="0.005" />
+  <xacro:property name="joint_friction" value="0.00" />
   <xacro:property name="joint_damping" value="1.5" />
   <xacro:property name="PIhalf" value="1.570796" />
@@ -85,5 +85,5 @@
       effort="20000"
       velocity="13" />
-    <dynamics damping="${joint_damping}" friction = "${joint_friction}"/>
+    <dynamics damping="${joint_damping}" friction = "0"/>
   </joint>
 <link
@@ -157,5 +157,6 @@
         rpy="0 0 0" />
       <mass
-        value="0.09637272" />
+        value="0.2" />
+        <!-- 0.09637272 -->
       <inertia
         ixx="0.00031529"
@@ -219,5 +220,6 @@
         rpy="0 0 0" />
       <mass
-        value="0.01812912" />
+        value="0.1812912" />
+        <!-- original mass  0.01812912-->
       <inertia
         ixx="0.00000196"

File: iiwa_description/urdf/dual_arm_system/dual_arm_right.xacro (robot description, xacro)
@@ -1,6 +1,6 @@
 <?xml version="1.0"?>
 <robot xmlns:xacro="http://www.ros.org/wiki/xacro">
-  <xacro:property name="joint_friction" value="0.005" />
-  <xacro:property name="joint_damping" value="1.0" />
+  <xacro:property name="joint_friction" value="0.00" />
+  <xacro:property name="joint_damping" value="1.5" />
   <xacro:property name="PIhalf" value="1.570796" />
   <xacro:property name="PI" value="3.141592" />
@@ -84,5 +84,5 @@
       effort="20000"
       velocity="13" />
-    <dynamics damping="${joint_damping}" friction = "${joint_friction}"/>
+    <dynamics damping="${joint_damping}" friction = "0"/>
   </joint>
 <link
@@ -156,5 +156,6 @@
         rpy="0 0 0" />
       <mass
-        value="0.09637272" />
+        value="0.2" />
+        <!-- 0.09637272 -->
       <inertia
         ixx="0.00031529"
@@ -209,5 +210,5 @@
       effort="20000"
       velocity="13" />
-    <dynamics damping="0" friction = "${joint_friction}"/>
+    <dynamics damping="${joint_damping}" friction = "${joint_friction}"/>
   </joint>
  <link
@@ -218,5 +219,5 @@
         rpy="0 0 0" />
       <mass
-        value="0.04812912" />
+        value="0.1812912" />
       <inertia
         ixx="0.00000196"
