Commit message: added controls for the miniwrist

File: iiwa_description/urdf/dual_arm_system/iiwa.transmission.xacro (robot description, xacro)
@@ -152,4 +152,24 @@
       </actuator>
     </transmission>
+  <transmission name="wristJ1_R_tran">
+      <robotNamespace>/${robot_name}</robotNamespace>
+      <type>transmission_interface/SimpleTransmission</type>
+      <joint name="wristJ1_R">
+  <hardwareInterface>hardware_interface/${hardware_interface}</hardwareInterface>
+      </joint>
+      <actuator name="wristJ1_R_motor">
+  <mechanicalReduction>1</mechanicalReduction>
+      </actuator>
+  </transmission>
+  <transmission name="wristJ2_R_tran">
+      <robotNamespace>/${robot_name}</robotNamespace>
+      <type>transmission_interface/SimpleTransmission</type>
+      <joint name="wristJ2_R">
+  <hardwareInterface>hardware_interface/${hardware_interface}</hardwareInterface>
+      </joint>
+      <actuator name="wristJ2_R_motor">
+  <mechanicalReduction>1</mechanicalReduction>
+      </actuator>
+  </transmission>
 <!--
   <transmission name="gripper_base_joint_tran">

File: iiwa_description/urdf/dual_arm_system/miniwrist_left.xacro (robot description, xacro)
@@ -19,5 +19,5 @@
       <mass value="0.0253977949262739" />
       <inertia
-        ixx="3.49511160259362E-06" ixy="-8.03793468213869E-08" ixz="1.78582674691137E-08" iyy="5.98607693493441E-06" iyz="-6.25954886336517E-09" izz="2.86657161143928E-06" />
+        ixx="0.0349511160259362" ixy="-0.000803793468213869" ixz="0.00000178582674691137" iyy="0.0598607693493441E" iyz="-0.00000625954886336517" izz="0.0286657161143928" />
     </inertial>
     <visual>

File: iiwa_description/urdf/dual_arm_system/miniwrist_right.xacro (robot description, xacro)
@@ -19,5 +19,5 @@
       <mass value="0.0253977949262739" />
       <inertia
-        ixx="3.49511160259362E-06" ixy="-8.03793468213869E-08" ixz="1.78582674691137E-08" iyy="5.98607693493441E-06" iyz="-6.25954886336517E-09" izz="2.86657161143928E-06" />
+        ixx="0.0349511160259362" ixy="-0.000803793468213869" ixz="0.00000178582674691137" iyy="0.0598607693493441E" iyz="-0.00000625954886336517" izz="0.0286657161143928" />
     </inertial>
     <visual>
